Commit message: testing changes

File: wheelchair2_description/urdf/kangaroo_ros2_control.xacro (robot description, xacro)
@@ -1,27 +1,33 @@
-<?xml version="1.0"?>
+<?xml version="1.0" encoding="UTF-8"?>
 <robot xmlns:xacro="http://www.ros.org/wiki/xacro">
-  <xacro:macro name="kangaroo_x2_driver" params="name prefix">
-    <ros2_control name="${name}" type="system">
-      <hardware>
-        <plugin>wheelchair2_kangaroo_x2_driver/Kangaroo</plugin>
-        <param name="left_wheel_name">left_wheel_joint</param>
-        <param name="right_wheel_name">right_wheel_joint</param>
-        <param name="wheel_diameter">0.32</param>
-        <param name="wheel_center_distance">0.55</param>
-        <param name="encoder_lines_per_revolution">65536</param>
-        <param name="hz">50</param>
-        <param name="port">/dev/ttyACM0</param>
-      </hardware>
-      <joint name="${prefix}left_wheel_joint">
-        <command_interface name="velocity"/>
-        <state_interface name="position"/>
-        <state_interface name="velocity"/>
-      </joint>
-      <joint name="${prefix}right_wheel_joint">
-        <command_interface name="velocity"/>
-        <state_interface name="position"/>
-        <state_interface name="velocity"/>
-      </joint>
-    </ros2_control>
-  </xacro:macro>
+	<xacro:macro name="kangaroo_x2_driver" params="name prefix is_sim">
+		<ros2_control name="${name}" type="system">
+			<hardware>
+				<xacro:if value="${is_sim}">
+					<plugin>gazebo_ros2_control/GazeboSystem</plugin>
+				</xacro:if>
+				<xacro:unless value="${is_sim}">
+					<!-- <plugin>wheelchair2_kangaroo_x2_driver/Kangaroo</plugin> -->
+					<plugin>mock_components/GenericSystem</plugin>
+					<param name="left_wheel_name">chassis_to_left_wheel</param>
+					<param name="right_wheel_name">chassis_to_right_wheel</param>
+					<param name="wheel_diameter">0.32</param>
+					<param name="wheel_center_distance">0.55</param>
+					<param name="encoder_lines_per_revolution">65536</param>
+					<param name="hz">50</param>
+					<param name="port">/dev/ttyACM0</param>
+				</xacro:unless>
+			</hardware>
+			<joint name="${prefix}left_wheel_joint">
+				<command_interface name="velocity" />
+				<state_interface name="position" />
+				<state_interface name="velocity" />
+			</joint>
+			<joint name="${prefix}right_wheel_joint">
+				<command_interface name="velocity" />
+				<state_interface name="position" />
+				<state_interface name="velocity" />
+			</joint>
+		</ros2_control>
+	</xacro:macro>
 </robot>

File: wheelchair2_description/urdf/wheelchair2_livox.urdf.xacro (robot description, xacro)
@@ -6,5 +6,7 @@
 	<xacro:include filename="$(find wheelchair2_description)/urdf/wheelchair2_livox_gazebo.urdf.xacro" />
 	<xacro:include filename="$(find ros2_livox_simulation)/urdf/mid360.xacro" />
+	<xacro:include filename="$(find wheelchair2_description)/urdf/kangaroo_ros2_control.xacro" />
 	<xacro:arg name="use_nominal_extrinsics" default="false" />
+	<xacro:arg name="is_sim" default="true" />
 	<xacro:arg name="add_plug" default="false" />
 	<xacro:arg name="use_mesh" default="true" />
@@ -34,5 +36,6 @@
 			<origin xyz="0 0 0" rpy=" 0 0 3.14" />
 			<geometry>
-				<mesh filename="file://$(find wheelchair2_description)/meshes/wheelchair2.dae" scale="0.01 0.01 0.01" />
+				<mesh filename="file://$(find wheelchair2_description)/meshes/wheelchair2.dae"
+					scale="0.01 0.01 0.01" />
 			</geometry>
 			<material name="black" />
@@ -40,34 +43,64 @@
 	</link>
 	<!-- Left Wheel-->
-	<xacro:m1_link_cylinder name="left_wheel" origin_rpy="0 0 0" origin_xyz="0 0 0.027" mass="0.10441" ixx="0.1000000042" ixy="0" ixz="0" iyy="0.1000000042" iyz="0" izz="0.1000000040" radius="0.155" length="0.06" radius_2="0.0028" length_2="0.005" material="grey" />
+	<xacro:m1_link_cylinder name="left_wheel" origin_rpy="0 0 0" origin_xyz="0 0 0.027" mass="0.10441"
+		ixx="0.1000000042" ixy="0" ixz="0" iyy="0.1000000042" iyz="0" izz="0.1000000040" radius="0.155"
+		length="0.06" radius_2="0.0028" length_2="0.005" material="grey" />
 	<!-- joint between chassis and Left wheel-->
-	<xacro:w_joint name="chassis_to_left_wheel" type="continuous" axis_xyz="0 0 1" axis_rpy="0 0 0" limit_e="100" limit_v="20" damping="1.0" friction="200000.0" origin_rpy="-1.57 0 0" origin_xyz="-0.22 0.28 -0.285" parent="chassis" child="left_wheel" />
+	<xacro:w_joint name="chassis_to_left_wheel" type="continuous" axis_xyz="0 0 1" axis_rpy="0 0 0"
+		limit_e="100" limit_v="20" damping="1.0" friction="200000.0" origin_rpy="-1.57 0 0"
+		origin_xyz="-0.22 0.28 -0.285" parent="chassis" child="left_wheel" />
 	<!--  inertia values are added by 0.1 in both left and right wheel to avoid collapsing of model in
 	gazebo-->
 	<!-- joint between chassis and Right Wheel-->
 	<!-- Right Wheel-->
-	<xacro:m1_link_cylinder name="right_wheel" origin_rpy="0 0 0" origin_xyz="0 0 0.027" mass="0.10441" ixx="0.1000000042" ixy="0" ixz="0" iyy="0.1000000042" iyz="0" izz="0.1000000040" radius="0.155" length="0.06" radius_2="0.0028" length_2="0.005" material="grey" />
-	<xacro:w_joint name="chassis_to_right_wheel" type="continuous" axis_xyz="0 0 1" axis_rpy="0 0 0" limit_e="100" limit_v="20" damping="1.0" friction="200000.0" origin_rpy="-1.57 0 0" origin_xyz="-0.22 -0.32 -0.285" parent="chassis" child="right_wheel" />
+	<xacro:m1_link_cylinder name="right_wheel" origin_rpy="0 0 0" origin_xyz="0 0 0.027"
+		mass="0.10441" ixx="0.1000000042" ixy="0" ixz="0" iyy="0.1000000042" iyz="0" izz="0.1000000040"
+		radius="0.155" length="0.06" radius_2="0.0028" length_2="0.005" material="grey" />
+	<xacro:w_joint name="chassis_to_right_wheel" type="continuous" axis_xyz="0 0 1" axis_rpy="0 0 0"
+		limit_e="100" limit_v="20" damping="1.0" friction="200000.0" origin_rpy="-1.57 0 0"
+		origin_xyz="-0.22 -0.32 -0.285" parent="chassis" child="right_wheel" />
 	<!-- Caster 1,2 and there joints with Base Link-->
-	<xacro:m_link_sphere name="caster1" origin_rpy="0 0 0" origin_xyz="0 0 0" mass="0.45164" ixx="0.100000005621" ixy="0.100000001310" ixz="0.100000001649" iyy="0.100000004345" iyz="0.100000002360" izz="0.100000003315" material="black" radius="0.1" radius_2="0.001" />
-	<xacro:f_joint name="chassis_to_caster1" type="fixed" axis_xyz="0 0 0" origin_rpy="0 0 0" origin_xyz="0.2 -0.25 -0.33" parent="chassis" child="caster1" />
-	<xacro:m_link_sphere name="caster2" origin_rpy="0 0 0" origin_xyz="0 0 0" mass="0.45164" ixx="0.100000005621" ixy="0.100000001310" ixz="0.100000001649" iyy="0.100000004345" iyz="0.100000002360" izz="0.100000003315" material="black" radius="0.1" radius_2="0.001" />
-	<xacro:f_joint name="chassis_to_caster2" type="fixed" axis_xyz="0 0 0" origin_rpy="0 0 0" origin_xyz="0.2 0.25 -0.33" parent="chassis" child="caster2" />
-	<xacro:f_link_box name="rod1" origin_rpy="0 0 0" origin_xyz="0 0 0" mass="0.45164" ixx="0.100000005621" ixy="0.100000001310" ixz="0.100000001649" iyy="0.100000004345" iyz="0.100000002360" izz="0.100000003315" material="black" size="0.016 0.016 0.6" />
-	<xacro:f_joint name="chassis_to_rod1" type="fixed" axis_xyz="0 0 0" origin_rpy="0 0 0" origin_xyz="-0.23 0.24 0.65" parent="chassis" child="rod1" />
-	<xacro:f_link_box name="rod2" origin_rpy="0 0 0" origin_xyz="0 0 0" mass="0.45164" ixx="0.100000005621" ixy="0.100000001310" ixz="0.100000001649" iyy="0.100000004345" iyz="0.100000002360" izz="0.100000003315" material="black" size="0.016 0.016 0.6" />
-	<xacro:f_joint name="chassis_to_rod2" type="fixed" axis_xyz="0 0 0" origin_rpy="0 0 0" origin_xyz="-0.23 -0.24 0.65" parent="chassis" child="rod2" />
-	<xacro:f_link_box name="camera_base_rod" origin_rpy="0 0 0" origin_xyz="0 0 0" mass="0.45164" ixx="0.100000005621" ixy="0.100000001310" ixz="0.100000001649" iyy="0.100000004345" iyz="0.100000002360" izz="0.100000003315" material="black" size="0.016 0.48 0.016" />
-	<xacro:f_joint name="chassis_to_camera_base_rod" type="fixed" axis_xyz="0 0 0" origin_rpy="0 0 0" origin_xyz="-0.23 0 0.650" parent="chassis" child="camera_base_rod" />
-	<xacro:f_link_box name="lidar_base_rod" origin_rpy="0 0 0" origin_xyz="0 0 0" mass="0.45164" ixx="0.100000005621" ixy="0.100000001310" ixz="0.100000001649" iyy="0.100000004345" iyz="0.100000002360" izz="0.100000003315" material="black" size="0.016 0.48 0.016" />
-	<xacro:f_joint name="chassis_to_lidar_base_rod" type="fixed" axis_xyz="0 0 0" origin_rpy="0 0 0" origin_xyz="0.23 0 -0.15" parent="chassis" child="lidar_base_rod" />
+	<xacro:m_link_sphere name="caster1" origin_rpy="0 0 0" origin_xyz="0 0 0" mass="0.45164"
+		ixx="0.100000005621" ixy="0.100000001310" ixz="0.100000001649" iyy="0.100000004345"
+		iyz="0.100000002360" izz="0.100000003315" material="black" radius="0.1" radius_2="0.001" />
+	<xacro:f_joint name="chassis_to_caster1" type="fixed" axis_xyz="0 0 0" origin_rpy="0 0 0"
+		origin_xyz="0.2 -0.25 -0.33" parent="chassis" child="caster1" />
+	<xacro:m_link_sphere name="caster2" origin_rpy="0 0 0" origin_xyz="0 0 0" mass="0.45164"
+		ixx="0.100000005621" ixy="0.100000001310" ixz="0.100000001649" iyy="0.100000004345"
+		iyz="0.100000002360" izz="0.100000003315" material="black" radius="0.1" radius_2="0.001" />
+	<xacro:f_joint name="chassis_to_caster2" type="fixed" axis_xyz="0 0 0" origin_rpy="0 0 0"
+		origin_xyz="0.2 0.25 -0.33" parent="chassis" child="caster2" />
+	<xacro:f_link_box name="rod1" origin_rpy="0 0 0" origin_xyz="0 0 0" mass="0.45164"
+		ixx="0.100000005621" ixy="0.100000001310" ixz="0.100000001649" iyy="0.100000004345"
+		iyz="0.100000002360" izz="0.100000003315" material="black" size="0.016 0.016 0.6" />
+	<xacro:f_joint name="chassis_to_rod1" type="fixed" axis_xyz="0 0 0" origin_rpy="0 0 0"
+		origin_xyz="-0.23 0.24 0.65" parent="chassis" child="rod1" />
+	<xacro:f_link_box name="rod2" origin_rpy="0 0 0" origin_xyz="0 0 0" mass="0.45164"
+		ixx="0.100000005621" ixy="0.100000001310" ixz="0.100000001649" iyy="0.100000004345"
+		iyz="0.100000002360" izz="0.100000003315" material="black" size="0.016 0.016 0.6" />
+	<xacro:f_joint name="chassis_to_rod2" type="fixed" axis_xyz="0 0 0" origin_rpy="0 0 0"
+		origin_xyz="-0.23 -0.24 0.65" parent="chassis" child="rod2" />
+	<xacro:f_link_box name="camera_base_rod" origin_rpy="0 0 0" origin_xyz="0 0 0" mass="0.45164"
+		ixx="0.100000005621" ixy="0.100000001310" ixz="0.100000001649" iyy="0.100000004345"
+		iyz="0.100000002360" izz="0.100000003315" material="black" size="0.016 0.48 0.016" />
+	<xacro:f_joint name="chassis_to_camera_base_rod" type="fixed" axis_xyz="0 0 0" origin_rpy="0 0 0"
+		origin_xyz="-0.23 0 0.650" parent="chassis" child="camera_base_rod" />
+	<xacro:f_link_box name="lidar_base_rod" origin_rpy="0 0 0" origin_xyz="0 0 0" mass="0.45164"
+		ixx="0.100000005621" ixy="0.100000001310" ixz="0.100000001649" iyy="0.100000004345"
+		iyz="0.100000002360" izz="0.100000003315" material="black" size="0.016 0.48 0.016" />
+	<xacro:f_joint name="chassis_to_lidar_base_rod" type="fixed" axis_xyz="0 0 0" origin_rpy="0 0 0"
+		origin_xyz="0.23 0 -0.15" parent="chassis" child="lidar_base_rod" />
 	<!--Lidar-->
-	<xacro:m_link_cylinder name="rplidar" origin_rpy="0 0 0" origin_xyz="0 0 0" mass="0.10441" ixx="0.1000000042" ixy="0" ixz="0" iyy="0.1000000042" iyz="0" izz="0.1000000040" material="black" filename="file://$(find wheelchair2_description)/meshes/rplidar.dae" scale="1 1 1" />
+	<xacro:m_link_cylinder name="rplidar" origin_rpy="0 0 0" origin_xyz="0 0 0" mass="0.10441"
+		ixx="0.1000000042" ixy="0" ixz="0" iyy="0.1000000042" iyz="0" izz="0.1000000040"
+		material="black" filename="file://$(find wheelchair2_description)/meshes/rplidar.dae"
+		scale="1 1 1" />
 	<!-- joint between chassis and lidar -->
-	<xacro:f_joint name="chassis_to_rplidar" type="fixed" axis_xyz="0 0 0" origin_rpy="0 0 0" origin_xyz="0.53 0 -0.15" parent="chassis" child="rplidar" />
+	<xacro:f_joint name="chassis_to_rplidar" type="fixed" axis_xyz="0 0 0" origin_rpy="0 0 0"
+		origin_xyz="0.53 0 -0.15" parent="chassis" child="rplidar" />
 	<xacro:mid360 name="livox" parent="camera_base_rod" topic="mid360">
 		<origin xyz="0 0 0.1" rpy="0 0 0" />
 	</xacro:mid360>
-	<!-- Gazebo Plugin-->
+	<xacro:kangaroo_x2_driver name="kangaroo_ros2_control" prefix="" is_sim="$(arg is_sim)"></xacro:kangaroo_x2_driver>
 	<gazebo>
 		<plugin name="gazebo_ros2_control" filename="libgazebo_ros2_control.so">
