Commit message: minor changes

File: wheelchair2_description/urdf/links_joints.urdf.xacro (robot description, xacro)
@@ -6,5 +6,6 @@
 	<!--macro
 	for cylinder shaped links(r,lwheels and lidar)-->
-	<xacro:macro name="m_link_cylinder" params="name origin_xyz origin_rpy mass ixx ixy ixz iyy iyz izz filename scale material ">
+	<xacro:macro name="m_link_cylinder"
+		params="name origin_xyz origin_rpy mass ixx ixy ixz iyy iyz izz filename scale material ">
 		<link name="${name}">
 			<inertial>				<!--Inertial
@@ -34,5 +35,6 @@
 	<!--macro
 	for cylinder shaped links(r,lwheels and lidar)-->
-	<xacro:macro name="m1_link_cylinder" params="name origin_xyz origin_rpy mass radius length radius_2 length_2 ixx ixy ixz iyy iyz izz material ">
+	<xacro:macro name="m1_link_cylinder"
+		params="name origin_xyz origin_rpy mass radius length radius_2 length_2 ixx ixy ixz iyy iyz izz material ">
 		<link name="${name}">
 			<inertial>				<!--Inertial
@@ -63,5 +65,6 @@
 	<!--macro
 	for box shaped links(r,lwheels and lidar)-->
-	<xacro:macro name="m_link_box" params="name origin_xyz origin_rpy size mass ixx ixy ixz iyy iyz izz v_origin_xyz v_origin_rpy filename scale material ">
+	<xacro:macro name="m_link_box"
+		params="name origin_xyz origin_rpy size mass ixx ixy ixz iyy iyz izz v_origin_xyz v_origin_rpy filename scale material ">
 		<link name="${name}">
 			<inertial>				<!--Inertial
@@ -89,5 +92,6 @@
 		</link>
 	</xacro:macro>
-	<xacro:macro name="f_link_box" params="name origin_xyz origin_rpy size mass ixx ixy ixz iyy iyz izz material ">
+	<xacro:macro name="f_link_box"
+		params="name origin_xyz origin_rpy size mass ixx ixy ixz iyy iyz izz material ">
 		<link name="${name}">
 			<inertial>				<!--Inertial
@@ -115,5 +119,6 @@
 		</link>
 	</xacro:macro>
-	<xacro:macro name="m_link_sphere" params="name origin_xyz origin_rpy radius radius_2 mass ixx ixy ixz iyy iyz izz material">
+	<xacro:macro name="m_link_sphere"
+		params="name origin_xyz origin_rpy radius radius_2 mass ixx ixy ixz iyy iyz izz material">
 		<link name="${name}">
 			<inertial>				<!--Inertial
@@ -143,5 +148,6 @@
 	<!-- It includes parent link, child link, limits, axis, origin, dynamics and transmission of the
 	robot-->
-	<xacro:macro name="m_joint" params="name type axis_xyz axis_rpy origin_rpy origin_xyz parent limit_e limit_v lower upper child damping friction ">
+	<xacro:macro name="m_joint"
+		params="name type axis_xyz axis_rpy origin_rpy origin_xyz parent limit_e limit_v lower upper child damping friction ">
 		<joint name="${name}" type="${type}">
 			<axis xyz="${axis_xyz}" rpy="${axis_rpy}" />
@@ -152,16 +158,17 @@
 			<child link="${child}" />
 		</joint>
-		<transmission name="trans_${name}">
-			<type>transmission_interface/SimpleTransmission</type>
-			<joint name="${name}">
-				<hardwareInterface>hardware_interface/EffortJointInterface</hardwareInterface>
-			</joint>
-			<actuator name="motor_${name}">
-				<hardwareInterface>hardware_interface/EffortJointInterface</hardwareInterface>
-				<mechanicalReduction>1</mechanicalReduction>
-			</actuator>
-		</transmission>
-	</xacro:macro>
-	<xacro:macro name="w_joint" params="name type axis_xyz axis_rpy origin_rpy origin_xyz parent limit_e limit_v child damping friction ">
+		<!-- <transmission name="trans_${name}"> -->
+		<!-- 	<type>transmission_interface/SimpleTransmission</type> -->
+		<!-- 	<joint name="${name}"> -->
+		<!-- 		<hardwareInterface>hardware_interface/EffortJointInterface</hardwareInterface> -->
+		<!-- 	</joint> -->
+		<!-- 	<actuator name="motor_${name}"> -->
+		<!-- 		<hardwareInterface>hardware_interface/EffortJointInterface</hardwareInterface> -->
+		<!-- 		<mechanicalReduction>1</mechanicalReduction> -->
+		<!-- 	</actuator> -->
+		<!-- </transmission> -->
+	</xacro:macro>
+	<xacro:macro name="w_joint"
+		params="name type axis_xyz axis_rpy origin_rpy origin_xyz parent limit_e limit_v child damping friction ">
 		<joint name="${name}" type="${type}">
 			<axis xyz="${axis_xyz}" rpy="${axis_rpy}" />
@@ -172,16 +179,17 @@
 			<child link="${child}" />
 		</joint>
-		<transmission name="trans_${name}">
-			<type>transmission_interface/SimpleTransmission</type>
-			<joint name="${name}">
-				<hardwareInterface>hardware_interface/EffortJointInterface</hardwareInterface>
-			</joint>
-			<actuator name="motor_${name}">
-				<hardwareInterface>hardware_interface/EffortJointInterface</hardwareInterface>
-				<mechanicalReduction>1</mechanicalReduction>
-			</actuator>
-		</transmission>
-	</xacro:macro>
-	<xacro:macro name="m2_joint" params="name type axis_xyz axis_rpy origin_rpy origin_xyz parent limit_e limit_v lower upper child damping friction ">
+		<!-- <transmission name="trans_${name}"> -->
+		<!-- 	<type>transmission_interface/SimpleTransmission</type> -->
+		<!-- 	<joint name="${name}"> -->
+		<!-- 		<hardwareInterface>hardware_interface/EffortJointInterface</hardwareInterface> -->
+		<!-- 	</joint> -->
+		<!-- 	<actuator name="motor_${name}"> -->
+		<!-- 		<hardwareInterface>hardware_interface/EffortJointInterface</hardwareInterface> -->
+		<!-- 		<mechanicalReduction>1</mechanicalReduction> -->
+		<!-- 	</actuator> -->
+		<!-- </transmission> -->
+	</xacro:macro>
+	<xacro:macro name="m2_joint"
+		params="name type axis_xyz axis_rpy origin_rpy origin_xyz parent limit_e limit_v lower upper child damping friction ">
 		<joint name="${name}" type="${type}">
 			<axis xyz="${axis_xyz}" rpy="${axis_rpy}" />
@@ -193,5 +201,6 @@
 		</joint>
 	</xacro:macro>
-	<xacro:macro name="mimic_joint" params="name type axis_xyz axis_rpy origin_rpy origin_xyz parent joint multiplier offset limit_e limit_v lower upper child damping friction ">
+	<xacro:macro name="mimic_joint"
+		params="name type axis_xyz axis_rpy origin_rpy origin_xyz parent joint multiplier offset limit_e limit_v lower upper child damping friction ">
 		<joint name="${name}" type="${type}">
 			<axis xyz="${axis_xyz}" rpy="${axis_rpy}" />

File: wheelchair2_description/urdf/wheelchair2_livox.urdf.xacro (robot description, xacro)
@@ -5,10 +5,7 @@
 	<xacro:include filename="$(find wheelchair2_description)/urdf/links_joints.urdf.xacro" />
 	<xacro:include filename="$(find wheelchair2_description)/urdf/wheelchair2_livox_gazebo.urdf.xacro" />
-<xacro:include filename="$(find wheelchair2_description)/urdf/wheelchair2_livox_gazebo.urdf.xacro" />
+<!-- <xacro:include filename="$(find wheelchair2_description)/urdf/wheelchair2_livox_gazebo.urdf.xacro" /> -->
 <xacro:include filename="$(find wheelchair2_description)/urdf/kangaroo_ros2_control.urdf.xacro" />
 	<xacro:include filename="$(find ros2_livox_simulation)/urdf/mid360.xacro" />
-	<xacro:arg name="use_nominal_extrinsics" default="false" />
-	<xacro:arg name="add_plug" default="false" />
-	<xacro:arg name="use_mesh" default="true" />
 <xacro:arg name="is_sim" default="true" />
 <xacro:arg name="gazebo_controllers" default="$(find wheelchair2_bringup)/config/wheelchair2_controllers.yaml" />

File: wheelchair2_description/urdf/wheelchair2_livox_gazebo.urdf.xacro (robot description, xacro)
@@ -2,22 +2,19 @@
 <robot name="wheelchair2"
 	xmlns:xacro="http://www.ros.org/wiki/xacro">
-	<gazebo>
-		<plugin name='diff_drive' filename='libgazebo_ros_diff_drive.so'>
-			<!-- Wheel Information -->
-			<left_joint>chassis_to_left_wheel</left_joint>
-			<right_joint>chassis_to_right_wheel</right_joint>
-			<wheel_separation>0.48</wheel_separation>
-			<wheel_diameter>0.31</wheel_diameter>
-			<!-- Limits -->
-			<max_wheel_torque>40</max_wheel_torque>
-			<max_wheel_acceleration>1.0</max_wheel_acceleration>
-			<!-- Output -->
-			<odometry_frame>odom</odometry_frame>
-			<robot_base_frame>base_link</robot_base_frame>
-			<publish_odom>true</publish_odom>
-			<publish_odom_tf>true</publish_odom_tf>
-			<publish_wheel_tf>false</publish_wheel_tf>
-		</plugin>
-	</gazebo>
+	<!-- <gazebo> -->
+	<!-- 	<plugin name='diff_drive' filename='libgazebo_ros_diff_drive.so'> -->
+	<!-- 		<left_joint>chassis_to_left_wheel</left_joint> -->
+	<!-- 		<right_joint>chassis_to_right_wheel</right_joint> -->
+	<!-- 		<wheel_separation>0.48</wheel_separation> -->
+	<!-- 		<wheel_diameter>0.31</wheel_diameter> -->
+	<!-- 		<max_wheel_torque>40</max_wheel_torque> -->
+	<!-- 		<max_wheel_acceleration>1.0</max_wheel_acceleration> -->
+	<!-- 		<odometry_frame>odom</odometry_frame> -->
+	<!-- 		<robot_base_frame>base_link</robot_base_frame> -->
+	<!-- 		<publish_odom>true</publish_odom> -->
+	<!-- 		<publish_odom_tf>true</publish_odom_tf> -->
+	<!-- 		<publish_wheel_tf>false</publish_wheel_tf> -->
+	<!-- 	</plugin> -->
+	<!-- </gazebo> -->
 	<!--Gazebo
 	related physics values of left wheel joint-->
