Commit message: modified camera_lidar urdf to make it work with ros2_control

File: wheelchair2_description/urdf/wheelchair2_camera_lidar.urdf.xacro (robot description, xacro)
@@ -4,9 +4,13 @@
 	<!-- Include Files-->
 	<xacro:include filename="$(find wheelchair2_description)/urdf/links_joints.urdf.xacro" />
-	<xacro:include filename="$(find wheelchair2_description)/urdf/wheelchair2_camera_lidar_gazebo.urdf.xacro" />
+	<xacro:include
+		filename="$(find wheelchair2_description)/urdf/wheelchair2_camera_lidar_gazebo.urdf.xacro" />
 	<xacro:include filename="$(find wheelchair2_description)/urdf/realsense.urdf.xacro" />
 	<xacro:arg name="use_nominal_extrinsics" default="false" />
 	<xacro:arg name="add_plug" default="false" />
 	<xacro:arg name="use_mesh" default="true" />
+	<xacro:arg name="is_sim" default="true" />
+	<xacro:arg name="gazebo_controllers"
+		default="$(find wheelchair2_bringup)/config/wheelchair2_controllers.yaml" />
 	<link name="base_link" />
 	<joint name="base_joint" type="fixed">
@@ -34,5 +38,6 @@
 			<origin xyz="0 0 0" rpy=" 0 0 3.14" />
 			<geometry>
-				<mesh filename="file://$(find wheelchair2_description)/meshes/wheelchair2.dae" scale="0.01 0.01 0.01" />
+				<mesh filename="file://$(find wheelchair2_description)/meshes/wheelchair2.dae"
+					scale="0.01 0.01 0.01" />
 			</geometry>
 			<material name="black" />
@@ -40,39 +45,74 @@
 	</link>
 	<!-- Left Wheel-->
-	<xacro:m1_link_cylinder name="left_wheel" origin_rpy="0 0 0" origin_xyz="0 0 0.027" mass="0.10441" ixx="0.1000000042" ixy="0" ixz="0" iyy="0.1000000042" iyz="0" izz="0.1000000040" radius="0.155" length="0.06" radius_2="0.0028" length_2="0.005" material="grey" />
+	<xacro:m1_link_cylinder name="left_wheel" origin_rpy="0 0 0" origin_xyz="0 0 0.027" mass="0.10441"
+		ixx="0.1000000042" ixy="0" ixz="0" iyy="0.1000000042" iyz="0" izz="0.1000000040" radius="0.155"
+		length="0.06" radius_2="0.0028" length_2="0.005" material="grey" />
 	<!-- joint between chassis and Left wheel-->
-	<xacro:w_joint name="chassis_to_left_wheel" type="continuous" axis_xyz="0 0 1" axis_rpy="0 0 0" limit_e="100" limit_v="20" damping="1.0" friction="200000.0" origin_rpy="-1.57 0 0" origin_xyz="-0.22 0.28 -0.285" parent="chassis" child="left_wheel" />
+	<xacro:w_joint name="chassis_to_left_wheel" type="continuous" axis_xyz="0 0 1" axis_rpy="0 0 0"
+		limit_e="100" limit_v="20" damping="1.0" friction="200000.0" origin_rpy="-1.57 0 0"
+		origin_xyz="-0.22 0.28 -0.285" parent="chassis" child="left_wheel" />
 	<!--  inertia values are added by 0.1 in both left and right wheel to avoid collapsing of model in
 	gazebo-->
 	<!-- joint between chassis and Right Wheel-->
 	<!-- Right Wheel-->
-	<xacro:m1_link_cylinder name="right_wheel" origin_rpy="0 0 0" origin_xyz="0 0 0.027" mass="0.10441" ixx="0.1000000042" ixy="0" ixz="0" iyy="0.1000000042" iyz="0" izz="0.1000000040" radius="0.155" length="0.06" radius_2="0.0028" length_2="0.005" material="grey" />
-	<xacro:w_joint name="chassis_to_right_wheel" type="continuous" axis_xyz="0 0 1" axis_rpy="0 0 0" limit_e="100" limit_v="20" damping="1.0" friction="200000.0" origin_rpy="-1.57 0 0" origin_xyz="-0.22 -0.32 -0.285" parent="chassis" child="right_wheel" />
+	<xacro:m1_link_cylinder name="right_wheel" origin_rpy="0 0 0" origin_xyz="0 0 0.027"
+		mass="0.10441" ixx="0.1000000042" ixy="0" ixz="0" iyy="0.1000000042" iyz="0" izz="0.1000000040"
+		radius="0.155" length="0.06" radius_2="0.0028" length_2="0.005" material="grey" />
+	<xacro:w_joint name="chassis_to_right_wheel" type="continuous" axis_xyz="0 0 1" axis_rpy="0 0 0"
+		limit_e="100" limit_v="20" damping="1.0" friction="200000.0" origin_rpy="-1.57 0 0"
+		origin_xyz="-0.22 -0.32 -0.285" parent="chassis" child="right_wheel" />
 	<!-- Caster 1,2 and there joints with Base Link-->
-	<xacro:m_link_sphere name="caster1" origin_rpy="0 0 0" origin_xyz="0 0 0" mass="0.45164" ixx="0.100000005621" ixy="0.100000001310" ixz="0.100000001649" iyy="0.100000004345" iyz="0.100000002360" izz="0.100000003315" material="black" radius="0.1" radius_2="0.001" />
-	<xacro:f_joint name="chassis_to_caster1" type="fixed" axis_xyz="0 0 0" origin_rpy="0 0 0" origin_xyz="0.2 -0.25 -0.33" parent="chassis" child="caster1" />
-	<xacro:m_link_sphere name="caster2" origin_rpy="0 0 0" origin_xyz="0 0 0" mass="0.45164" ixx="0.100000005621" ixy="0.100000001310" ixz="0.100000001649" iyy="0.100000004345" iyz="0.100000002360" izz="0.100000003315" material="black" radius="0.1" radius_2="0.001" />
-	<xacro:f_joint name="chassis_to_caster2" type="fixed" axis_xyz="0 0 0" origin_rpy="0 0 0" origin_xyz="0.2 0.25 -0.33" parent="chassis" child="caster2" />
-	<xacro:f_link_box name="rod1" origin_rpy="0 0 0" origin_xyz="0 0 0" mass="0.45164" ixx="0.100000005621" ixy="0.100000001310" ixz="0.100000001649" iyy="0.100000004345" iyz="0.100000002360" izz="0.100000003315" material="black" size="0.016 0.016 0.6" />
-	<xacro:f_joint name="chassis_to_rod1" type="fixed" axis_xyz="0 0 0" origin_rpy="0 0 0" origin_xyz="-0.23 0.24 0.65" parent="chassis" child="rod1" />
-	<xacro:f_link_box name="rod2" origin_rpy="0 0 0" origin_xyz="0 0 0" mass="0.45164" ixx="0.100000005621" ixy="0.100000001310" ixz="0.100000001649" iyy="0.100000004345" iyz="0.100000002360" izz="0.100000003315" material="black" size="0.016 0.016 0.6" />
-	<xacro:f_joint name="chassis_to_rod2" type="fixed" axis_xyz="0 0 0" origin_rpy="0 0 0" origin_xyz="-0.23 -0.24 0.65" parent="chassis" child="rod2" />
-	<xacro:f_link_box name="camera_base_rod" origin_rpy="0 0 0" origin_xyz="0 0 0" mass="0.45164" ixx="0.100000005621" ixy="0.100000001310" ixz="0.100000001649" iyy="0.100000004345" iyz="0.100000002360" izz="0.100000003315" material="black" size="0.016 0.48 0.016" />
-	<xacro:f_joint name="chassis_to_camera_base_rod" type="fixed" axis_xyz="0 0 0" origin_rpy="0 0 0" origin_xyz="-0.23 0 0.650" parent="chassis" child="camera_base_rod" />
-	<xacro:f_link_box name="lidar_base_rod" origin_rpy="0 0 0" origin_xyz="0 0 0" mass="0.45164" ixx="0.100000005621" ixy="0.100000001310" ixz="0.100000001649" iyy="0.100000004345" iyz="0.100000002360" izz="0.100000003315" material="black" size="0.016 0.48 0.016" />
-	<xacro:f_joint name="chassis_to_lidar_base_rod" type="fixed" axis_xyz="0 0 0" origin_rpy="0 0 0" origin_xyz="0.23 0 -0.15" parent="chassis" child="lidar_base_rod" />
+	<xacro:m_link_sphere name="caster1" origin_rpy="0 0 0" origin_xyz="0 0 0" mass="0.45164"
+		ixx="0.100000005621" ixy="0.100000001310" ixz="0.100000001649" iyy="0.100000004345"
+		iyz="0.100000002360" izz="0.100000003315" material="black" radius="0.1" radius_2="0.001" />
+	<xacro:f_joint name="chassis_to_caster1" type="fixed" axis_xyz="0 0 0" origin_rpy="0 0 0"
+		origin_xyz="0.2 -0.25 -0.33" parent="chassis" child="caster1" />
+	<xacro:m_link_sphere name="caster2" origin_rpy="0 0 0" origin_xyz="0 0 0" mass="0.45164"
+		ixx="0.100000005621" ixy="0.100000001310" ixz="0.100000001649" iyy="0.100000004345"
+		iyz="0.100000002360" izz="0.100000003315" material="black" radius="0.1" radius_2="0.001" />
+	<xacro:f_joint name="chassis_to_caster2" type="fixed" axis_xyz="0 0 0" origin_rpy="0 0 0"
+		origin_xyz="0.2 0.25 -0.33" parent="chassis" child="caster2" />
+	<xacro:f_link_box name="rod1" origin_rpy="0 0 0" origin_xyz="0 0 0" mass="0.45164"
+		ixx="0.100000005621" ixy="0.100000001310" ixz="0.100000001649" iyy="0.100000004345"
+		iyz="0.100000002360" izz="0.100000003315" material="black" size="0.016 0.016 0.6" />
+	<xacro:f_joint name="chassis_to_rod1" type="fixed" axis_xyz="0 0 0" origin_rpy="0 0 0"
+		origin_xyz="-0.23 0.24 0.65" parent="chassis" child="rod1" />
+	<xacro:f_link_box name="rod2" origin_rpy="0 0 0" origin_xyz="0 0 0" mass="0.45164"
+		ixx="0.100000005621" ixy="0.100000001310" ixz="0.100000001649" iyy="0.100000004345"
+		iyz="0.100000002360" izz="0.100000003315" material="black" size="0.016 0.016 0.6" />
+	<xacro:f_joint name="chassis_to_rod2" type="fixed" axis_xyz="0 0 0" origin_rpy="0 0 0"
+		origin_xyz="-0.23 -0.24 0.65" parent="chassis" child="rod2" />
+	<xacro:f_link_box name="camera_base_rod" origin_rpy="0 0 0" origin_xyz="0 0 0" mass="0.45164"
+		ixx="0.100000005621" ixy="0.100000001310" ixz="0.100000001649" iyy="0.100000004345"
+		iyz="0.100000002360" izz="0.100000003315" material="black" size="0.016 0.48 0.016" />
+	<xacro:f_joint name="chassis_to_camera_base_rod" type="fixed" axis_xyz="0 0 0" origin_rpy="0 0 0"
+		origin_xyz="-0.23 0 0.650" parent="chassis" child="camera_base_rod" />
+	<xacro:f_link_box name="lidar_base_rod" origin_rpy="0 0 0" origin_xyz="0 0 0" mass="0.45164"
+		ixx="0.100000005621" ixy="0.100000001310" ixz="0.100000001649" iyy="0.100000004345"
+		iyz="0.100000002360" izz="0.100000003315" material="black" size="0.016 0.48 0.016" />
+	<xacro:f_joint name="chassis_to_lidar_base_rod" type="fixed" axis_xyz="0 0 0" origin_rpy="0 0 0"
+		origin_xyz="0.23 0 -0.15" parent="chassis" child="lidar_base_rod" />
 	<!--Lidar-->
-	<xacro:m_link_cylinder name="rplidar" origin_rpy="0 0 0" origin_xyz="0 0 0" mass="0.10441" ixx="0.1000000042" ixy="0" ixz="0" iyy="0.1000000042" iyz="0" izz="0.1000000040" material="black" filename="file://$(find wheelchair2_description)/meshes/rplidar.dae" scale="1 1 1" />
+	<xacro:m_link_cylinder name="rplidar" origin_rpy="0 0 0" origin_xyz="0 0 0" mass="0.10441"
+		ixx="0.1000000042" ixy="0" ixz="0" iyy="0.1000000042" iyz="0" izz="0.1000000040"
+		material="black" filename="file://$(find wheelchair2_description)/meshes/rplidar.dae"
+		scale="1 1 1" />
 	<!-- joint between chassis and lidar -->
-	<xacro:f_joint name="chassis_to_rplidar" type="fixed" axis_xyz="0 0 0" origin_rpy="0 0 0" origin_xyz="0.53 0 -0.15" parent="chassis" child="rplidar" />
+	<xacro:f_joint name="chassis_to_rplidar" type="fixed" axis_xyz="0 0 0" origin_rpy="0 0 0"
+		origin_xyz="0.53 0 -0.15" parent="chassis" child="rplidar" />
 	<xacro:realsense parent="base_link" name="camera">
 		<origin xyz="0.20 -0.24 0.50" rpy="0 -0.01 0" />
 	</xacro:realsense>
 	<!-- Gazebo Plugin-->
-	<gazebo>
-		<plugin name="gazebo_ros2_control" filename="libgazebo_ros2_control.so">
-			<!-- <robotNamespace>/wheelchair2</robotNamespace> -->
-			<legacyModeNS>true</legacyModeNS>
-		</plugin>
-	</gazebo>
+	<xacro:if value="$(arg is_sim)">
+		<gazebo>
+			<plugin name="gazebo_ros2_control" filename="libgazebo_ros2_control.so">
+				<parameters>$(arg gazebo_controllers)</parameters>
+				<ros>
+					<remapping>/wheelchair2_base_controller/cmd_vel_unstamped:=/cmd_vel</remapping>
+					<remapping>/wheelchair2_base_controller/odom:=/odom</remapping>
+				</ros>
+			</plugin>
+		</gazebo>
+	</xacro:if>
 </robot>

File: wheelchair2_description/urdf/wheelchair2_camera_lidar_gazebo.urdf.xacro (robot description, xacro)
@@ -2,22 +2,20 @@
 <robot name="wheelchair2"
 	xmlns:xacro="http://www.ros.org/wiki/xacro">
-	<gazebo>
-		<plugin name='diff_drive' filename='libgazebo_ros_diff_drive.so'>
-			<!-- Wheel Information -->
-			<left_joint>chassis_to_left_wheel</left_joint>
-			<right_joint>chassis_to_right_wheel</right_joint>
-			<wheel_separation>0.48</wheel_separation>
-			<wheel_diameter>0.31</wheel_diameter>
-			<!-- Limits -->
-			<max_wheel_torque>40</max_wheel_torque>
-			<max_wheel_acceleration>1.0</max_wheel_acceleration>
-			<!-- Output -->
-			<odometry_frame>odom</odometry_frame>
-			<robot_base_frame>base_link</robot_base_frame>
-			<publish_odom>true</publish_odom>
-			<publish_odom_tf>true</publish_odom_tf>
-			<publish_wheel_tf>false</publish_wheel_tf>
-		</plugin>
-	</gazebo>
+	<!-- <gazebo> -->
+	<!-- 	<plugin name='diff_drive' filename='libgazebo_ros_diff_drive.so'> -->
+	<!-- 		<left_joint>chassis_to_left_wheel</left_joint> -->
+	<!-- 		<right_joint>chassis_to_right_wheel</right_joint> -->
+	<!-- 		<wheel_separation>0.48</wheel_separation> -->
+	<!-- 		<wheel_diameter>0.31</wheel_diameter> -->
+	<!-- 		<max_wheel_torque>40</max_wheel_torque> -->
+	<!-- 		<max_wheel_acceleration>1.0</max_wheel_acceleration> -->
+	<!-- 		<odometry_frame>odom</odometry_frame> -->
+	<!-- 		<robot_base_frame>base_link</robot_base_frame> -->
+	<!-- 		<publish_odom>true</publish_odom> -->
+	<!-- 		<publish_odom_tf>true</publish_odom_tf> -->
+	<!-- 		<publish_wheel_tf>false</publish_wheel_tf> -->
+	<!-- 	</plugin> -->
+	<!-- </gazebo> -->
+	<!---->
 	<!--Gazebo
 	related physics values of left wheel joint-->

File: wheelchair2_description/urdf/wheelchair2_livox.urdf.xacro (robot description, xacro)
@@ -8,5 +8,6 @@
 	<xacro:include filename="$(find ros2_livox_simulation)/urdf/mid360.xacro" />
 	<xacro:arg name="is_sim" default="true" />
-	<xacro:arg name="gazebo_controllers" default="$(find wheelchair2_bringup)/config/wheelchair2_controllers.yaml" />
+	<xacro:arg name="gazebo_controllers"
+		default="$(find wheelchair2_bringup)/config/wheelchair2_controllers.yaml" />
 	<link name="base_link" />
 	<joint name="base_joint" type="fixed">

Commit message: added param files and world files

File: wheelchair2_description/urdf/wheelchair2_camera_lidar.urdf.xacro (robot description, xacro)
@@ -6,4 +6,5 @@
 	<xacro:include
 		filename="$(find wheelchair2_description)/urdf/wheelchair2_camera_lidar_gazebo.urdf.xacro" />
+	<xacro:include filename="$(find wheelchair2_description)/urdf/kangaroo_ros2_control.urdf.xacro" />
 	<xacro:include filename="$(find wheelchair2_description)/urdf/realsense.urdf.xacro" />
 	<xacro:arg name="use_nominal_extrinsics" default="false" />
@@ -14,4 +15,11 @@
 		default="$(find wheelchair2_bringup)/config/wheelchair2_controllers.yaml" />
 	<link name="base_link" />
+	<!-- Add Base Footprint -->
+	<!-- <joint name="base_footprint_joint" type="fixed"> -->
+	<!-- 	<parent link="base_link" /> -->
+	<!-- 	<child link="base_footprint" /> -->
+	<!-- 	<origin xyz="0 0 0" rpy="0 0 0" /> -->
+	<!-- </joint> -->
+	<!-- <link name="base_footprint" /> -->
 	<joint name="base_joint" type="fixed">
 		<parent link="base_link" />
@@ -50,5 +58,5 @@
 	<!-- joint between chassis and Left wheel-->
 	<xacro:w_joint name="chassis_to_left_wheel" type="continuous" axis_xyz="0 0 1" axis_rpy="0 0 0"
-		limit_e="100" limit_v="20" damping="1.0" friction="200000.0" origin_rpy="-1.57 0 0"
+		limit_e="100" limit_v="20" damping="1.0" friction="0.01" origin_rpy="-1.57 0 0"
 		origin_xyz="-0.22 0.28 -0.285" parent="chassis" child="left_wheel" />
 	<!--  inertia values are added by 0.1 in both left and right wheel to avoid collapsing of model in
@@ -60,5 +68,5 @@
 		radius="0.155" length="0.06" radius_2="0.0028" length_2="0.005" material="grey" />
 	<xacro:w_joint name="chassis_to_right_wheel" type="continuous" axis_xyz="0 0 1" axis_rpy="0 0 0"
-		limit_e="100" limit_v="20" damping="1.0" friction="200000.0" origin_rpy="-1.57 0 0"
+		limit_e="100" limit_v="20" damping="1.0" friction="0.01" origin_rpy="-1.57 0 0"
 		origin_xyz="-0.22 -0.32 -0.285" parent="chassis" child="right_wheel" />
 	<!-- Caster 1,2 and there joints with Base Link-->
@@ -104,4 +112,5 @@
 		<origin xyz="0.20 -0.24 0.50" rpy="0 -0.01 0" />
 	</xacro:realsense>
+	<xacro:kangaroo_x2_driver name="kangaroo_ros2_control" prefix="" is_sim="$(arg is_sim)"></xacro:kangaroo_x2_driver>
 	<!-- Gazebo Plugin-->
 	<xacro:if value="$(arg is_sim)">

File: wheelchair2_description/urdf/wheelchair2_camera_lidar_gazebo.urdf.xacro (robot description, xacro)
@@ -82,5 +82,5 @@
 			<pose> 0 0 0 0 0 0 </pose>
 			<visualize>false</visualize>
-			<update_rate>15</update_rate>
+			<update_rate>30</update_rate>
 			<ray>
 				<scan>
@@ -108,5 +108,5 @@
 				<ros>
 					<!-- <namespace>/gpu_ray</namespace> -->
-					<argument>~/out:=scan_raw</argument>
+					<argument>~/out:=scan</argument>
 				</ros>
 				<output_type>sensor_msgs/LaserScan</output_type>

File: wheelchair2_description/urdf/wheelchair2_livox.urdf.xacro (robot description, xacro)
@@ -11,4 +11,11 @@
 		default="$(find wheelchair2_bringup)/config/wheelchair2_controllers.yaml" />
 	<link name="base_link" />
+	<!-- <joint name="base_footprint_joint" type="fixed"> -->
+	<!-- 	<parent link="base_link" /> -->
+	<!-- 	<child link="base_footprint" /> -->
+	<!-- 	<origin xyz="0 0 0" rpy="0 0 0" /> -->
+	<!-- </joint> -->
+	<!---->
+	<!-- <link name="base_footprint" /> -->
 	<joint name="base_joint" type="fixed">
 		<parent link="base_link" />

Commit message: fixed bug with nav2 substitutions. Nav2 now starts.

File: wheelchair2_description/urdf/wheelchair2_camera_lidar.urdf.xacro (robot description, xacro)
@@ -16,10 +16,10 @@
 	<link name="base_link" />
 	<!-- Add Base Footprint -->
-	<!-- <joint name="base_footprint_joint" type="fixed"> -->
-	<!-- 	<parent link="base_link" /> -->
-	<!-- 	<child link="base_footprint" /> -->
-	<!-- 	<origin xyz="0 0 0" rpy="0 0 0" /> -->
-	<!-- </joint> -->
-	<!-- <link name="base_footprint" /> -->
+	<joint name="base_footprint_joint" type="fixed">
+		<parent link="base_link" />
+		<child link="base_footprint" />
+		<origin xyz="0 0 0" rpy="0 0 0" />
+	</joint>
+	<link name="base_footprint" />
 	<joint name="base_joint" type="fixed">
 		<parent link="base_link" />

File: wheelchair2_description/urdf/wheelchair2_livox.urdf.xacro (robot description, xacro)
@@ -11,11 +11,10 @@
 		default="$(find wheelchair2_bringup)/config/wheelchair2_controllers.yaml" />
 	<link name="base_link" />
-	<!-- <joint name="base_footprint_joint" type="fixed"> -->
-	<!-- 	<parent link="base_link" /> -->
-	<!-- 	<child link="base_footprint" /> -->
-	<!-- 	<origin xyz="0 0 0" rpy="0 0 0" /> -->
-	<!-- </joint> -->
-	<!---->
-	<!-- <link name="base_footprint" /> -->
+	<joint name="base_footprint_joint" type="fixed">
+		<parent link="base_link" />
+		<child link="base_footprint" />
+		<origin xyz="0 0 0" rpy="0 0 0" />
+	</joint>
+	<link name="base_footprint" />
 	<joint name="base_joint" type="fixed">
 		<parent link="base_link" />
