Commit message: 2d lidar working

File: wheelchair2_description/urdf/mid360.xacro (robot description, xacro)
@@ -20,12 +20,12 @@
   </xacro:macro>
   <xacro:macro name="mid360" params="name:='' parent:= 'base_link' topic:='mid360' *origin ">
-<link name="${name}">
-<xacro:box_inertia m="${length}" w="${width}" d="${length}" h="${height}"/>
-  <visual>
+    <link name="${name}">
+      <xacro:box_inertia m="${length}" w="${width}" d="${length}" h="${height}"/>
+      <visual>
         <geometry>
-            <box size="${length} ${width} ${height}"/>
+          <box size="${length} ${width} ${height}"/>
         </geometry>
-  </visual>
-</link>
+      </visual>
+    </link>
     <joint name="${name}_joint" type="fixed">
       <parent link="${parent}"/>
@@ -33,45 +33,4 @@
       <xacro:insert_block name="origin"/>
     </joint>
-    <gazebo reference="${name}">
-      <sensor type="ray" name="${name}">
-        <pose>0 0 0 0 0 0</pose>
-        <visualize>true</visualize>
-        <update_rate>10</update_rate>
-        <!-- This ray plgin is only for visualization. -->
-        <plugin name="${name}_plugin" filename="libros2_livox.so">
-			<ray>
-			  <scan>
-				<horizontal>
-				<samples>100</samples>
-				<resolution>1</resolution>
-				<min_angle>${0}</min_angle>
-				<max_angle>${2*M_PI}</max_angle>
-				</horizontal>
-				<vertical>
-				<samples>360</samples>
-				<resolution>1</resolution>
-				<min_angle>${-7.22/180*M_PI}</min_angle>
-				<max_angle>${55.22/180*M_PI}</max_angle>
-				</vertical>
-			  </scan>
-			  <range>
-				<min>${laser_min_range}</min>
-				<max>${laser_max_range}</max>
-				<resolution>${resolution}</resolution>
-			  </range>
-			  <noise>
-				<type>gaussian</type>
-				<mean>${noise_mean}</mean>
-				<stddev>${noise_stddev}</stddev>
-			  </noise>
-			</ray>
-          <visualize>false</visualize>
-		  <samples>${samples}</samples>
-		  <downsample>1</downsample>
-		  <csv_file_name>$(find wheelchair2_description)/urdf/mid360.csv</csv_file_name>
-		  <topic>${topic}</topic>
-        </plugin>
-      </sensor>
-    </gazebo>
   </xacro:macro>
 </robot>

File: wheelchair2_gazebo/urdf/wheelchair2_camera_livox_gazebo.urdf.xacro (robot description, xacro)
@@ -9,4 +9,5 @@
     <xacro:include filename="$(find wheelchair2_gazebo)/urdf/ros2_control.urdf.xacro" />
     <xacro:include filename="$(find wheelchair2_gazebo)/urdf/wheelchair2_gazebo.urdf.xacro" />
+    <xacro:include filename="$(find wheelchair2_gazebo)/urdf/livox.urdf.xacro" />
     <xacro:arg name="use_nominal_extrinsics" default="false" />
     <xacro:arg name="add_plug" default="false" />
@@ -35,5 +36,5 @@
             <material name="black" />
         </collision>
-        <visual>
+        <!-- <visual>
             <origin xyz="0 0 0" rpy=" 0 0 3.14" />
             <geometry>
@@ -41,5 +42,5 @@
             </geometry>
             <material name="black" />
-        </visual>
+        </visual> -->
     </link>
     <!-- Left Wheel-->
@@ -67,8 +68,8 @@
     <xacro:f_joint name="base_link_to_lidar_base_rod" type="fixed" axis_xyz="0 0 0" origin_rpy="0 0 0" origin_xyz="0.23 0 -0.15" parent="base_link" child="lidar_base_rod" />
     <!--Lidar-->
-    <!-- <xacro:m_link_cylinder name="laser_frame" origin_rpy="0 0 0" origin_xyz="0 0 0" mass="0.10441" ixx="0.1000000042" ixy="0" ixz="0" iyy="0.1000000042" iyz="0" izz="0.1000000040" material="black" filename="file://$(find wheelchair2_description)/meshes/rplidar.dae" scale="1 1 1" /> -->
+    <xacro:m_link_cylinder name="laser_frame" origin_rpy="0 0 0" origin_xyz="0 0 0" mass="0.10441" ixx="0.1000000042" ixy="0" ixz="0" iyy="0.1000000042" iyz="0" izz="0.1000000040" material="black" filename="file://$(find wheelchair2_description)/meshes/rplidar.dae" scale="1 1 1" />
     <!-- joint between base_link and lidar -->
-    <!-- <xacro:f_joint name="base_link_to_laser" type="fixed" axis_xyz="0 0 0" origin_rpy="0 0 0" origin_xyz="0.53 0 -0.15" parent="base_link" child="laser_frame" />
-    <xacro:realsense parent="base_link" name="camera">
+    <xacro:f_joint name="base_link_to_laser" type="fixed" axis_xyz="0 0 0" origin_rpy="0 0 0" origin_xyz="0.53 0 -0.15" parent="base_link" child="laser_frame" />
+    <!-- <xacro:realsense parent="base_link" name="camera">
         <origin xyz="0 0 1.25" rpy="0 0 0" />
     </xacro:realsense> -->
