Commit message: simulation seems to work now

File: wheelchair2_description/urdf/kangaroo_ros2_control.urdf.xacro (robot description, xacro)
@@ -1,33 +1,39 @@
 <?xml version="1.0" encoding="UTF-8"?>
 <robot xmlns:xacro="http://www.ros.org/wiki/xacro">
-  <xacro:macro name="kangaroo_x2_driver" params="name prefix is_sim">
-    <ros2_control name="${name}" type="system">
-      <hardware>
-        <xacro:if value="${is_sim}">
-          <plugin>gazebo_ros2_control/GazeboSystem</plugin>
-        </xacro:if>
-        <xacro:unless value="${is_sim}">
-          <!-- <plugin>wheelchair2_kangaroo_x2_driver/Kangaroo</plugin> -->
-          <plugin>mock_components/GenericSystem</plugin>
-          <param name="left_wheel_name">chassis_to_left_wheel</param>
-          <param name="right_wheel_name">chassis_to_right_wheel</param>
-          <param name="wheel_diameter">0.32</param>
-          <param name="wheel_center_distance">0.55</param>
-          <param name="encoder_lines_per_revolution">65536</param>
-          <param name="hz">50</param>
-          <param name="port">/dev/ttyACM0</param>
-        </xacro:unless>
-      </hardware>
-      <joint name="${prefix}chassis_to_left_wheel">
-        <command_interface name="velocity" />
-        <state_interface name="position" />
-        <state_interface name="velocity" />
-      </joint>
-      <joint name="${prefix}chassis_to_right_wheel">
-        <command_interface name="velocity" />
-        <state_interface name="position" />
-        <state_interface name="velocity" />
-      </joint>
-    </ros2_control>
-  </xacro:macro>
+	<xacro:macro name="kangaroo_x2_driver" params="name prefix is_sim">
+		<ros2_control name="${name}" type="system">
+			<hardware>
+				<xacro:if value="${is_sim}">
+					<plugin>gazebo_ros2_control/GazeboSystem</plugin>
+				</xacro:if>
+				<xacro:unless value="${is_sim}">
+					<!-- <plugin>wheelchair2_kangaroo_x2_driver/Kangaroo</plugin> -->
+					<plugin>mock_components/GenericSystem</plugin>
+					<param name="left_wheel_name">chassis_to_left_wheel</param>
+					<param name="right_wheel_name">chassis_to_right_wheel</param>
+					<param name="wheel_diameter">0.32</param>
+					<param name="wheel_center_distance">0.55</param>
+					<param name="encoder_lines_per_revolution">65536</param>
+					<param name="hz">50</param>
+					<param name="port">/dev/ttyACM0</param>
+				</xacro:unless>
+			</hardware>
+			<joint name="${prefix}chassis_to_left_wheel">
+				<command_interface name="velocity">
+					<param name="min">-1</param>
+					<param name="max">1</param>
+				</command_interface>
+				<state_interface name="position" />
+				<state_interface name="velocity" />
+			</joint>
+			<joint name="${prefix}chassis_to_right_wheel">
+				<command_interface name="velocity">
+					<param name="min">-1</param>
+					<param name="max">1</param>
+				</command_interface>
+				<state_interface name="position" />
+				<state_interface name="velocity" />
+			</joint>
+		</ros2_control>
+	</xacro:macro>
 </robot>

File: wheelchair2_description/urdf/wheelchair2_livox.urdf.xacro (robot description, xacro)
@@ -5,9 +5,11 @@
 	<xacro:include filename="$(find wheelchair2_description)/urdf/links_joints.urdf.xacro" />
 	<xacro:include filename="$(find wheelchair2_description)/urdf/wheelchair2_livox_gazebo.urdf.xacro" />
-<!-- <xacro:include filename="$(find wheelchair2_description)/urdf/wheelchair2_livox_gazebo.urdf.xacro" /> -->
-<xacro:include filename="$(find wheelchair2_description)/urdf/kangaroo_ros2_control.urdf.xacro" />
+	<!-- <xacro:include filename="$(find
+	wheelchair2_description)/urdf/wheelchair2_livox_gazebo.urdf.xacro" /> -->
+	<xacro:include filename="$(find wheelchair2_description)/urdf/kangaroo_ros2_control.urdf.xacro" />
 	<xacro:include filename="$(find ros2_livox_simulation)/urdf/mid360.xacro" />
-<xacro:arg name="is_sim" default="true" />
-<xacro:arg name="gazebo_controllers" default="$(find wheelchair2_bringup)/config/wheelchair2_controllers.yaml" />
+	<xacro:arg name="is_sim" default="true" />
+	<xacro:arg name="gazebo_controllers"
+		default="$(find wheelchair2_bringup)/config/wheelchair2_controllers.yaml" />
 	<link name="base_link" />
 	<joint name="base_joint" type="fixed">
@@ -35,5 +37,6 @@
 			<origin xyz="0 0 0" rpy=" 0 0 3.14" />
 			<geometry>
-<mesh filename="file://$(find wheelchair2_description)/meshes/wheelchair2.dae" scale="0.01 0.01 0.01" />
+				<mesh filename="file://$(find wheelchair2_description)/meshes/wheelchair2.dae"
+					scale="0.01 0.01 0.01" />
 			</geometry>
 			<material name="black" />
@@ -41,41 +44,71 @@
 	</link>
 	<!-- Left Wheel-->
-<xacro:m1_link_cylinder name="left_wheel" origin_rpy="0 0 0" origin_xyz="0 0 0.027" mass="0.10441" ixx="0.1000000042" ixy="0" ixz="0" iyy="0.1000000042" iyz="0" izz="0.1000000040" radius="0.155" length="0.06" radius_2="0.0028" length_2="0.005" material="grey" />
+	<xacro:m1_link_cylinder name="left_wheel" origin_rpy="0 0 0" origin_xyz="0 0 0.027" mass="0.10441"
+		ixx="0.1000000042" ixy="0" ixz="0" iyy="0.1000000042" iyz="0" izz="0.1000000040" radius="0.155"
+		length="0.06" radius_2="0.0028" length_2="0.005" material="grey" />
 	<!-- joint between chassis and Left wheel-->
-<xacro:w_joint name="chassis_to_left_wheel" type="continuous" axis_xyz="0 0 1" axis_rpy="0 0 0" limit_e="100" limit_v="20" damping="1.0" friction="200000.0" origin_rpy="-1.57 0 0" origin_xyz="-0.22 0.28 -0.285" parent="chassis" child="left_wheel" />
+	<xacro:w_joint name="chassis_to_left_wheel" type="continuous" axis_xyz="0 0 1" axis_rpy="0 0 0"
+		limit_e="100" limit_v="20" damping="1.0" friction="2.0" origin_rpy="-1.57 0 0"
+		origin_xyz="-0.22 0.28 -0.285" parent="chassis" child="left_wheel" />
 	<!--  inertia values are added by 0.1 in both left and right wheel to avoid collapsing of model in
 	gazebo-->
 	<!-- joint between chassis and Right Wheel-->
 	<!-- Right Wheel-->
-<xacro:m1_link_cylinder name="right_wheel" origin_rpy="0 0 0" origin_xyz="0 0 0.027" mass="0.10441" ixx="0.1000000042" ixy="0" ixz="0" iyy="0.1000000042" iyz="0" izz="0.1000000040" radius="0.155" length="0.06" radius_2="0.0028" length_2="0.005" material="grey" />
-<xacro:w_joint name="chassis_to_right_wheel" type="continuous" axis_xyz="0 0 1" axis_rpy="0 0 0" limit_e="100" limit_v="20" damping="1.0" friction="200000.0" origin_rpy="-1.57 0 0" origin_xyz="-0.22 -0.32 -0.285" parent="chassis" child="right_wheel" />
+	<xacro:m1_link_cylinder name="right_wheel" origin_rpy="0 0 0" origin_xyz="0 0 0.027"
+		mass="0.10441" ixx="0.1000000042" ixy="0" ixz="0" iyy="0.1000000042" iyz="0" izz="0.1000000040"
+		radius="0.155" length="0.06" radius_2="0.0028" length_2="0.005" material="grey" />
+	<xacro:w_joint name="chassis_to_right_wheel" type="continuous" axis_xyz="0 0 1" axis_rpy="0 0 0"
+		limit_e="100" limit_v="20" damping="1.0" friction="2.0" origin_rpy="-1.57 0 0"
+		origin_xyz="-0.22 -0.32 -0.285" parent="chassis" child="right_wheel" />
 	<!-- Caster 1,2 and there joints with Base Link-->
-<xacro:m_link_sphere name="caster1" origin_rpy="0 0 0" origin_xyz="0 0 0" mass="0.45164" ixx="0.100000005621" ixy="0.100000001310" ixz="0.100000001649" iyy="0.100000004345" iyz="0.100000002360" izz="0.100000003315" material="black" radius="0.1" radius_2="0.001" />
-<xacro:f_joint name="chassis_to_caster1" type="fixed" axis_xyz="0 0 0" origin_rpy="0 0 0" origin_xyz="0.2 -0.25 -0.33" parent="chassis" child="caster1" />
-<xacro:m_link_sphere name="caster2" origin_rpy="0 0 0" origin_xyz="0 0 0" mass="0.45164" ixx="0.100000005621" ixy="0.100000001310" ixz="0.100000001649" iyy="0.100000004345" iyz="0.100000002360" izz="0.100000003315" material="black" radius="0.1" radius_2="0.001" />
-<xacro:f_joint name="chassis_to_caster2" type="fixed" axis_xyz="0 0 0" origin_rpy="0 0 0" origin_xyz="0.2 0.25 -0.33" parent="chassis" child="caster2" />
-<xacro:f_link_box name="rod1" origin_rpy="0 0 0" origin_xyz="0 0 0" mass="0.45164" ixx="0.100000005621" ixy="0.100000001310" ixz="0.100000001649" iyy="0.100000004345" iyz="0.100000002360" izz="0.100000003315" material="black" size="0.016 0.016 0.6" />
-<xacro:f_joint name="chassis_to_rod1" type="fixed" axis_xyz="0 0 0" origin_rpy="0 0 0" origin_xyz="-0.23 0.24 0.65" parent="chassis" child="rod1" />
-<xacro:f_link_box name="rod2" origin_rpy="0 0 0" origin_xyz="0 0 0" mass="0.45164" ixx="0.100000005621" ixy="0.100000001310" ixz="0.100000001649" iyy="0.100000004345" iyz="0.100000002360" izz="0.100000003315" material="black" size="0.016 0.016 0.6" />
-<xacro:f_joint name="chassis_to_rod2" type="fixed" axis_xyz="0 0 0" origin_rpy="0 0 0" origin_xyz="-0.23 -0.24 0.65" parent="chassis" child="rod2" />
-<xacro:f_link_box name="camera_base_rod" origin_rpy="0 0 0" origin_xyz="0 0 0" mass="0.45164" ixx="0.100000005621" ixy="0.100000001310" ixz="0.100000001649" iyy="0.100000004345" iyz="0.100000002360" izz="0.100000003315" material="black" size="0.016 0.48 0.016" />
-<xacro:f_joint name="chassis_to_camera_base_rod" type="fixed" axis_xyz="0 0 0" origin_rpy="0 0 0" origin_xyz="-0.23 0 0.650" parent="chassis" child="camera_base_rod" />
-<xacro:f_link_box name="lidar_base_rod" origin_rpy="0 0 0" origin_xyz="0 0 0" mass="0.45164" ixx="0.100000005621" ixy="0.100000001310" ixz="0.100000001649" iyy="0.100000004345" iyz="0.100000002360" izz="0.100000003315" material="black" size="0.016 0.48 0.016" />
-<xacro:f_joint name="chassis_to_lidar_base_rod" type="fixed" axis_xyz="0 0 0" origin_rpy="0 0 0" origin_xyz="0.23 0 -0.15" parent="chassis" child="lidar_base_rod" />
+	<xacro:m_link_sphere name="caster1" origin_rpy="0 0 0" origin_xyz="0 0 0" mass="0.45164"
+		ixx="0.100000005621" ixy="0.100000001310" ixz="0.100000001649" iyy="0.100000004345"
+		iyz="0.100000002360" izz="0.100000003315" material="black" radius="0.1" radius_2="0.001" />
+	<xacro:f_joint name="chassis_to_caster1" type="fixed" axis_xyz="0 0 0" origin_rpy="0 0 0"
+		origin_xyz="0.2 -0.25 -0.33" parent="chassis" child="caster1" />
+	<xacro:m_link_sphere name="caster2" origin_rpy="0 0 0" origin_xyz="0 0 0" mass="0.45164"
+		ixx="0.100000005621" ixy="0.100000001310" ixz="0.100000001649" iyy="0.100000004345"
+		iyz="0.100000002360" izz="0.100000003315" material="black" radius="0.1" radius_2="0.001" />
+	<xacro:f_joint name="chassis_to_caster2" type="fixed" axis_xyz="0 0 0" origin_rpy="0 0 0"
+		origin_xyz="0.2 0.25 -0.33" parent="chassis" child="caster2" />
+	<xacro:f_link_box name="rod1" origin_rpy="0 0 0" origin_xyz="0 0 0" mass="0.45164"
+		ixx="0.100000005621" ixy="0.100000001310" ixz="0.100000001649" iyy="0.100000004345"
+		iyz="0.100000002360" izz="0.100000003315" material="black" size="0.016 0.016 0.6" />
+	<xacro:f_joint name="chassis_to_rod1" type="fixed" axis_xyz="0 0 0" origin_rpy="0 0 0"
+		origin_xyz="-0.23 0.24 0.65" parent="chassis" child="rod1" />
+	<xacro:f_link_box name="rod2" origin_rpy="0 0 0" origin_xyz="0 0 0" mass="0.45164"
+		ixx="0.100000005621" ixy="0.100000001310" ixz="0.100000001649" iyy="0.100000004345"
+		iyz="0.100000002360" izz="0.100000003315" material="black" size="0.016 0.016 0.6" />
+	<xacro:f_joint name="chassis_to_rod2" type="fixed" axis_xyz="0 0 0" origin_rpy="0 0 0"
+		origin_xyz="-0.23 -0.24 0.65" parent="chassis" child="rod2" />
+	<xacro:f_link_box name="camera_base_rod" origin_rpy="0 0 0" origin_xyz="0 0 0" mass="0.45164"
+		ixx="0.100000005621" ixy="0.100000001310" ixz="0.100000001649" iyy="0.100000004345"
+		iyz="0.100000002360" izz="0.100000003315" material="black" size="0.016 0.48 0.016" />
+	<xacro:f_joint name="chassis_to_camera_base_rod" type="fixed" axis_xyz="0 0 0" origin_rpy="0 0 0"
+		origin_xyz="-0.23 0 0.650" parent="chassis" child="camera_base_rod" />
+	<xacro:f_link_box name="lidar_base_rod" origin_rpy="0 0 0" origin_xyz="0 0 0" mass="0.45164"
+		ixx="0.100000005621" ixy="0.100000001310" ixz="0.100000001649" iyy="0.100000004345"
+		iyz="0.100000002360" izz="0.100000003315" material="black" size="0.016 0.48 0.016" />
+	<xacro:f_joint name="chassis_to_lidar_base_rod" type="fixed" axis_xyz="0 0 0" origin_rpy="0 0 0"
+		origin_xyz="0.23 0 -0.15" parent="chassis" child="lidar_base_rod" />
 	<!--Lidar-->
-<xacro:m_link_cylinder name="rplidar" origin_rpy="0 0 0" origin_xyz="0 0 0" mass="0.10441" ixx="0.1000000042" ixy="0" ixz="0" iyy="0.1000000042" iyz="0" izz="0.1000000040" material="black" filename="file://$(find wheelchair2_description)/meshes/rplidar.dae" scale="1 1 1" />
+	<xacro:m_link_cylinder name="rplidar" origin_rpy="0 0 0" origin_xyz="0 0 0" mass="0.10441"
+		ixx="0.1000000042" ixy="0" ixz="0" iyy="0.1000000042" iyz="0" izz="0.1000000040"
+		material="black" filename="file://$(find wheelchair2_description)/meshes/rplidar.dae"
+		scale="1 1 1" />
 	<!-- joint between chassis and lidar -->
-<xacro:f_joint name="chassis_to_rplidar" type="fixed" axis_xyz="0 0 0" origin_rpy="0 0 0" origin_xyz="0.53 0 -0.15" parent="chassis" child="rplidar" />
+	<xacro:f_joint name="chassis_to_rplidar" type="fixed" axis_xyz="0 0 0" origin_rpy="0 0 0"
+		origin_xyz="0.53 0 -0.15" parent="chassis" child="rplidar" />
 	<xacro:mid360 name="livox" parent="camera_base_rod" topic="mid360">
 		<origin xyz="0 0 0.1" rpy="0 0 0" />
 	</xacro:mid360>
-<xacro:kangaroo_x2_driver name="kangaroo_ros2_control" prefix="" is_sim="$(arg is_sim)"></xacro:kangaroo_x2_driver>
+	<xacro:kangaroo_x2_driver name="kangaroo_ros2_control" prefix="" is_sim="$(arg is_sim)"></xacro:kangaroo_x2_driver>
 	<!-- Gazebo Plugin-->
-<xacro:if value="$(arg is_sim)">
-	<gazebo>
-		<plugin name="gazebo_ros2_control" filename="libgazebo_ros2_control.so">
-<parameters>$(arg gazebo_controllers)</parameters>
-</plugin>
-</gazebo>
-</xacro:if>
+	<xacro:if value="$(arg is_sim)">
+		<gazebo>
+			<plugin name="gazebo_ros2_control" filename="libgazebo_ros2_control.so">
+				<parameters>$(arg gazebo_controllers)</parameters>
+			</plugin>
+		</gazebo>
+	</xacro:if>
 </robot>

File: wheelchair2_description/urdf/wheelchair2_livox_gazebo.urdf.xacro (robot description, xacro)
@@ -19,27 +19,25 @@
 	<!--Gazebo
 	related physics values of left wheel joint-->
-	<gazebo reference="chassis_to_left_wheel">
-		<mu1 value="10000.0" />
-		<mu2 value="10000.0" />
-		<fdir1 value="0 0 1" />
-		<kp value="300" />
-		<!--500000-->
-		<kd value="10" />
-		<!--10-->
-		<ki value="200" />
-		<maxVel value="2.0" />
-		<minDepth value="0.0001" />
-	</gazebo>
-	<!-- Gazebo related physics values of right wheel joint-->
-	<gazebo reference="chassis_to_right_wheel">
-		<mu1 value="10000.0" />
-		<mu2 value="10000.0" />
-		<fdir1 value="0 0 1" />
-		<kp value="300" />
-		<kd value="10" />
-		<ki value="200" />
-		<maxVel value="2.0" />
-		<minDepth value="0.0001" />
-	</gazebo>
+	<!-- <gazebo reference="chassis_to_left_wheel"> -->
+	<!-- 	<mu1 value="10000.0" /> -->
+	<!-- 	<mu2 value="10000.0" /> -->
+	<!-- 	<fdir1 value="0 0 1" /> -->
+	<!-- 	<kp value="300" /> -->
+	<!-- 	<kd value="10" /> -->
+	<!-- 	<ki value="200" /> -->
+	<!-- 	<maxVel value="2.0" /> -->
+	<!-- 	<minDepth value="0.0001" /> -->
+	<!-- </gazebo> -->
+	<!-- <gazebo reference="chassis_to_right_wheel"> -->
+	<!-- 	<mu1 value="10000.0" /> -->
+	<!-- 	<mu2 value="10000.0" /> -->
+	<!-- 	<fdir1 value="0 0 1" /> -->
+	<!-- 	<kp value="300" /> -->
+	<!-- 	<kd value="10" /> -->
+	<!-- 	<ki value="200" /> -->
+	<!-- 	<maxVel value="2.0" /> -->
+	<!-- 	<minDepth value="0.0001" /> -->
+	<!-- </gazebo> -->
+	<!---->
 	<gazebo reference="chassis">
 		<material>Gazebo/FlatBlack</material>
@@ -76,42 +74,3 @@
 		<material>Gazebo/Grey</material>
 	</gazebo>
-	<!-- <gazebo reference="rplidar"> -->
-	<!-- 	<material>Gazebo/DarkGrey</material> -->
-	<!---->
-	<!-- 	<sensor name="laser" type="ray"> -->
-	<!-- 		<pose> 0 0 0 0 0 0 </pose> -->
-	<!-- 		<visualize>false</visualize> -->
-	<!-- 		<update_rate>15</update_rate> -->
-	<!-- 		<ray> -->
-	<!-- 			<scan> -->
-	<!-- 				<horizontal> -->
-	<!-- 					<samples>720</samples> -->
-	<!-- 					<min_angle>-1.57</min_angle> -->
-	<!-- 					<max_angle>1.57</max_angle> -->
-	<!-- 				</horizontal> -->
-	<!-- 			</scan> -->
-	<!-- 			<range> -->
-	<!-- 				<min>0.1</min> -->
-	<!-- 				<max>25</max> -->
-	<!-- 			</range> -->
-	<!-- 			<noise> -->
-	<!-- 				<type>gaussian</type> -->
-	<!-- Noise parameters based on published spec for Hokuyo laser -->
-	<!--               achieving "+-30mm" accuracy at range < 10m.  A mean of 0.0m and -->
-	<!--               stddev of 0.01m will put 99.7% of samples within 0.03m of the true -->
-	<!--               reading. -->
-	<!-- 				<mean>0.0</mean> -->
-	<!-- 				<stddev>0.01</stddev> -->
-	<!-- 			</noise> -->
-	<!-- 		</ray> -->
-	<!-- 		<plugin name="laser_controller" filename="libgazebo_ros_ray_sensor.so"> -->
-	<!-- 			<ros> -->
-	<!-- <namespace>/gpu_ray</namespace> -->
-	<!-- 				<argument>~/out:=scan_raw</argument> -->
-	<!-- 			</ros> -->
-	<!-- 			<output_type>sensor_msgs/LaserScan</output_type> -->
-	<!-- 			<frame_name>rplidar</frame_name> -->
-	<!-- 		</plugin> -->
-	<!-- 	</sensor> -->
-	<!-- </gazebo> -->
 </robot>
