Commit message: added changes to urdf to make it work better with nav2

File: wheelchair2_description/urdf/kangaroo_ros2_control.urdf.xacro (robot description, xacro)
@@ -10,6 +10,6 @@
 					<plugin>wheelchair2_kangaroo_x2_driver/Kangaroo</plugin>
 					<!-- <plugin>mock_components/GenericSystem</plugin> -->
-					<param name="left_wheel_name">chassis_to_left_wheel</param>
-					<param name="right_wheel_name">chassis_to_right_wheel</param>
+					<param name="left_wheel_name">base_link_to_left_wheel</param>
+					<param name="right_wheel_name">base_link_to_right_wheel</param>
 					<param name="wheel_diameter">0.32</param>
 					<param name="wheel_center_distance">0.55</param>
@@ -20,5 +20,5 @@
 				</xacro:unless>
 			</hardware>
-			<joint name="${prefix}chassis_to_left_wheel">
+			<joint name="${prefix}base_link_to_left_wheel">
 				<command_interface name="velocity">
 					<param name="min">-1</param>
@@ -28,5 +28,5 @@
 				<state_interface name="velocity" />
 			</joint>
-			<joint name="${prefix}chassis_to_right_wheel">
+			<joint name="${prefix}base_link_to_right_wheel">
 				<command_interface name="velocity">
 					<param name="min">-1</param>

File: wheelchair2_description/urdf/wheelchair2.urdf.xacro (robot description, xacro)
@@ -7,6 +7,8 @@
 	<xacro:include filename="$(find wheelchair2_description)/urdf/wheelchair2_gazebo.urdf.xacro" />
 	<xacro:include filename="$(find wheelchair2_description)/urdf/_d435.urdf.xacro" />
-	<!--xacro:include filename="$(find wheelchair2_description)/urdf/_d455.urdf.xacro" /-->
-	<!--xacro:arg name="use_nominal_extrinsics" default="false"/>
+	<!--xacro:include
+	filename="$(find wheelchair2_description)/urdf/_d455.urdf.xacro" /-->
+	<!--xacro:arg
+	name="use_nominal_extrinsics" default="false"/>
   <xacro:arg name="add_plug" default="false" />
   <xacro:arg name="use_mesh" default="true" /-->
@@ -14,8 +16,8 @@
 	<joint name="base_joint" type="fixed">
 		<parent link="base_link" />
-		<child link="chassis" />
+		<child link="base_link" />
 		<origin xyz="0 0 0.2" rpy="0 0 0" />
 	</joint>
-	<link name='chassis'>
+	<link name='base_link'>
 		<pose>0 0 0.1 0 0 0</pose>
 		<inertial>
@@ -38,5 +40,6 @@
 			<origin xyz="0 0 0" rpy=" 0 0 3.14" />
 			<geometry>
-				<mesh filename="file://$(find wheelchair2_description)/wheelchair2.dae" scale="0.01 0.01 0.01" />
+				<mesh filename="file://$(find wheelchair2_description)/wheelchair2.dae"
+					scale="0.01 0.01 0.01" />
 			</geometry>
 			<material name="black" />
@@ -45,34 +48,66 @@
 	<!--Left
 	Wheel-->
-	<xacro:m1_link_cylinder name="left_wheel" origin_rpy="0 0 0" origin_xyz="0 0 0.027" mass="0.10441" ixx="0.1000000042" ixy="0" ixz="0" iyy="0.1000000042" iyz="0" izz="0.1000000040" radius="0.155" length="0.06" radius_2="0.0028" length_2="0.005" material="grey" />
+	<xacro:m1_link_cylinder name="left_wheel" origin_rpy="0 0 0" origin_xyz="0 0 0.027" mass="0.10441"
+		ixx="0.1000000042" ixy="0" ixz="0" iyy="0.1000000042" iyz="0" izz="0.1000000040" radius="0.155"
+		length="0.06" radius_2="0.0028" length_2="0.005" material="grey" />
 	<!--joint
-	between chassis and Left wheel-->
-	<xacro:w_joint name="chassis_to_left_wheel" type="continuous" axis_xyz="0 0 1" axis_rpy="0 0 0" limit_e="100" limit_v="20" damping="1.0" friction="200000.0" origin_rpy="-1.57 0 0" origin_xyz="-0.22 0.28 -0.285" parent="chassis" child="left_wheel" />
+	between base_link and Left wheel-->
+	<xacro:w_joint name="base_link_to_left_wheel" type="continuous" axis_xyz="0 0 1" axis_rpy="0 0 0"
+		limit_e="100" limit_v="20" damping="1.0" friction="200000.0" origin_rpy="-1.57 0 0"
+		origin_xyz="-0.22 0.28 -0.285" parent="base_link" child="left_wheel" />
 	<!-- inertia values are added by 0.1 in both left and right wheel to avoid collapsing of model in
 	gazebo-->
 	<!--joint
-	between chassis and Right Wheel-->
+	between base_link and Right Wheel-->
 	<!--Right
 	Wheel-->
-	<xacro:m1_link_cylinder name="right_wheel" origin_rpy="0 0 0" origin_xyz="0 0 0.027" mass="0.10441" ixx="0.1000000042" ixy="0" ixz="0" iyy="0.1000000042" iyz="0" izz="0.1000000040" radius="0.155" length="0.06" radius_2="0.0028" length_2="0.005" material="grey" />
-	<xacro:w_joint name="chassis_to_right_wheel" type="continuous" axis_xyz="0 0 1" axis_rpy="0 0 0" limit_e="100" limit_v="20" damping="1.0" friction="200000.0" origin_rpy="-1.57 0 0" origin_xyz="-0.22 -0.32 -0.285" parent="chassis" child="right_wheel" />
+	<xacro:m1_link_cylinder name="right_wheel" origin_rpy="0 0 0" origin_xyz="0 0 0.027"
+		mass="0.10441" ixx="0.1000000042" ixy="0" ixz="0" iyy="0.1000000042" iyz="0" izz="0.1000000040"
+		radius="0.155" length="0.06" radius_2="0.0028" length_2="0.005" material="grey" />
+	<xacro:w_joint name="base_link_to_right_wheel" type="continuous" axis_xyz="0 0 1" axis_rpy="0 0 0"
+		limit_e="100" limit_v="20" damping="1.0" friction="200000.0" origin_rpy="-1.57 0 0"
+		origin_xyz="-0.22 -0.32 -0.285" parent="base_link" child="right_wheel" />
 	<!--Caster
 	1,2 and there joints with Base Link-->
-	<xacro:m_link_sphere name="caster1" origin_rpy="0 0 0" origin_xyz="0 0 0" mass="0.45164" ixx="0.100000005621" ixy="0.100000001310" ixz="0.100000001649" iyy="0.100000004345" iyz="0.100000002360" izz="0.100000003315" material="black" radius="0.1" radius_2="0.001" />
-	<xacro:f_joint name="chassis_to_caster1" type="fixed" axis_xyz="0 0 0" origin_rpy="0 0 0" origin_xyz="0.2 -0.25 -0.33" parent="chassis" child="caster1" />
-	<xacro:m_link_sphere name="caster2" origin_rpy="0 0 0" origin_xyz="0 0 0" mass="0.45164" ixx="0.100000005621" ixy="0.100000001310" ixz="0.100000001649" iyy="0.100000004345" iyz="0.100000002360" izz="0.100000003315" material="black" radius="0.1" radius_2="0.001" />
-	<xacro:f_joint name="chassis_to_caster2" type="fixed" axis_xyz="0 0 0" origin_rpy="0 0 0" origin_xyz="0.2 0.25 -0.33" parent="chassis" child="caster2" />
-	<xacro:f_link_box name="rod1" origin_rpy="0 0 0" origin_xyz="0 0 0" mass="0.45164" ixx="0.100000005621" ixy="0.100000001310" ixz="0.100000001649" iyy="0.100000004345" iyz="0.100000002360" izz="0.100000003315" material="black" size="0.016 0.016 0.6" />
-	<xacro:f_joint name="chassis_to_rod1" type="fixed" axis_xyz="0 0 0" origin_rpy="0 0 0" origin_xyz="-0.23 0.24 0.65" parent="chassis" child="rod1" />
-	<xacro:f_link_box name="rod2" origin_rpy="0 0 0" origin_xyz="0 0 0" mass="0.45164" ixx="0.100000005621" ixy="0.100000001310" ixz="0.100000001649" iyy="0.100000004345" iyz="0.100000002360" izz="0.100000003315" material="black" size="0.016 0.016 0.6" />
-	<xacro:f_joint name="chassis_to_rod2" type="fixed" axis_xyz="0 0 0" origin_rpy="0 0 0" origin_xyz="-0.23 -0.24 0.65" parent="chassis" child="rod2" />
-	<xacro:f_link_box name="camera_base_rod" origin_rpy="0 0 0" origin_xyz="0 0 0" mass="0.45164" ixx="0.100000005621" ixy="0.100000001310" ixz="0.100000001649" iyy="0.100000004345" iyz="0.100000002360" izz="0.100000003315" material="black" size="0.016 0.48 0.016" />
-	<xacro:f_joint name="chassis_to_camera_base_rod" type="fixed" axis_xyz="0 0 0" origin_rpy="0 0 0" origin_xyz="-0.23 0 0.650" parent="chassis" child="camera_base_rod" />
-	<!--xacro:f_link_box name="lidar_base_rod" origin_rpy="0 0 0" origin_xyz="0 0 0" mass="0.45164" ixx="0.100000005621" ixy="0.100000001310" ixz="0.100000001649" iyy="0.100000004345" iyz="0.100000002360" izz="0.100000003315" material="black" size="0.016 0.48 0.016"/>
-    <xacro:f_joint name="chassis_to_lidar_base_rod" type="fixed" axis_xyz="0 0 0" origin_rpy="0 0 0" origin_xyz="0.23 0 -0.15" parent="chassis" child="lidar_base_rod" /-->
+	<xacro:m_link_sphere name="caster1" origin_rpy="0 0 0" origin_xyz="0 0 0" mass="0.45164"
+		ixx="0.100000005621" ixy="0.100000001310" ixz="0.100000001649" iyy="0.100000004345"
+		iyz="0.100000002360" izz="0.100000003315" material="black" radius="0.1" radius_2="0.001" />
+	<xacro:f_joint name="base_link_to_caster1" type="fixed" axis_xyz="0 0 0" origin_rpy="0 0 0"
+		origin_xyz="0.2 -0.25 -0.33" parent="base_link" child="caster1" />
+	<xacro:m_link_sphere name="caster2" origin_rpy="0 0 0" origin_xyz="0 0 0" mass="0.45164"
+		ixx="0.100000005621" ixy="0.100000001310" ixz="0.100000001649" iyy="0.100000004345"
+		iyz="0.100000002360" izz="0.100000003315" material="black" radius="0.1" radius_2="0.001" />
+	<xacro:f_joint name="base_link_to_caster2" type="fixed" axis_xyz="0 0 0" origin_rpy="0 0 0"
+		origin_xyz="0.2 0.25 -0.33" parent="base_link" child="caster2" />
+	<xacro:f_link_box name="rod1" origin_rpy="0 0 0" origin_xyz="0 0 0" mass="0.45164"
+		ixx="0.100000005621" ixy="0.100000001310" ixz="0.100000001649" iyy="0.100000004345"
+		iyz="0.100000002360" izz="0.100000003315" material="black" size="0.016 0.016 0.6" />
+	<xacro:f_joint name="base_link_to_rod1" type="fixed" axis_xyz="0 0 0" origin_rpy="0 0 0"
+		origin_xyz="-0.23 0.24 0.65" parent="base_link" child="rod1" />
+	<xacro:f_link_box name="rod2" origin_rpy="0 0 0" origin_xyz="0 0 0" mass="0.45164"
+		ixx="0.100000005621" ixy="0.100000001310" ixz="0.100000001649" iyy="0.100000004345"
+		iyz="0.100000002360" izz="0.100000003315" material="black" size="0.016 0.016 0.6" />
+	<xacro:f_joint name="base_link_to_rod2" type="fixed" axis_xyz="0 0 0" origin_rpy="0 0 0"
+		origin_xyz="-0.23 -0.24 0.65" parent="base_link" child="rod2" />
+	<xacro:f_link_box name="camera_base_rod" origin_rpy="0 0 0" origin_xyz="0 0 0" mass="0.45164"
+		ixx="0.100000005621" ixy="0.100000001310" ixz="0.100000001649" iyy="0.100000004345"
+		iyz="0.100000002360" izz="0.100000003315" material="black" size="0.016 0.48 0.016" />
+	<xacro:f_joint name="base_link_to_camera_base_rod" type="fixed" axis_xyz="0 0 0"
+		origin_rpy="0 0 0" origin_xyz="-0.23 0 0.650" parent="base_link" child="camera_base_rod" />
+	<!--xacro:f_link_box
+	name="lidar_base_rod" origin_rpy="0 0 0" origin_xyz="0 0 0" mass="0.45164" ixx="0.100000005621"
+	ixy="0.100000001310" ixz="0.100000001649" iyy="0.100000004345" iyz="0.100000002360"
+	izz="0.100000003315" material="black" size="0.016 0.48 0.016"/>
+    <xacro:f_joint name="base_link_to_lidar_base_rod" type="fixed" axis_xyz="0 0 0" origin_rpy="0 0 0"
+	origin_xyz="0.23 0 -0.15" parent="base_link" child="lidar_base_rod" /-->
 	<!--Lidar-->
-	<!--xacro:m_link_cylinder name="rplidar" origin_rpy="0 0 0" origin_xyz="0 0 0" mass="0.10441" ixx="0.1000000042" ixy="0" ixz="0" iyy="0.1000000042" iyz="0" izz="0.1000000040" material="black" filename="package://wheelchair2_description/meshes/rplidar.dae" scale="1 1 1"/-->
-	<!-- joint between chassis and lidar -->
-	<!--xacro:f_joint name="chassis_to_rplidar" type="fixed" axis_xyz="0 0 0" origin_rpy="0 0 3.14" origin_xyz="0.23 0 -0.15" parent="chassis" child="rplidar" /-->
+	<!--xacro:m_link_cylinder
+	name="rplidar" origin_rpy="0 0 0" origin_xyz="0 0 0" mass="0.10441" ixx="0.1000000042" ixy="0"
+	ixz="0" iyy="0.1000000042" iyz="0" izz="0.1000000040" material="black"
+	filename="package://wheelchair2_description/meshes/rplidar.dae" scale="1 1 1"/-->
+	<!-- joint between base_link and lidar -->
+	<!--xacro:f_joint
+	name="base_link_to_rplidar" type="fixed" axis_xyz="0 0 0" origin_rpy="0 0 3.14" origin_xyz="0.23 0
+	-0.15" parent="base_link" child="rplidar" /-->
 	<!--Real_Sense-->
 	<xacro:sensor_d435 parent="base_link" name="camera2" topics_ns="camera2" pointcloud="true">

File: wheelchair2_description/urdf/wheelchair2_camera_lidar.urdf.xacro (robot description, xacro)
@@ -14,18 +14,17 @@
 	<xacro:arg name="gazebo_controllers"
 		default="$(find wheelchair2_bringup)/config/wheelchair2_controllers.yaml" />
-	<link name="base_link" />
+	<link name="base_footprint" />
 	<!-- Add Base Footprint -->
 	<joint name="base_footprint_joint" type="fixed">
-		<parent link="base_link" />
-		<child link="base_footprint" />
-		<origin xyz="0 0 0" rpy="0 0 0" />
+		<parent link="base_footprint" />
+		<child link="base_link" />
+		<origin xyz="0.22 0 0.2" rpy="0 0 0" />
 	</joint>
-	<link name="base_footprint" />
-	<joint name="base_joint" type="fixed">
-		<parent link="base_link" />
-		<child link="chassis" />
-		<origin xyz="0.22 0.0 0.2" rpy="0 0 0" />
-	</joint>
-	<link name='chassis'>
+	<!-- <joint name="base_joint" type="fixed"> -->
+	<!-- 	<parent link="base_link" /> -->
+	<!-- 	<child link="chassis" /> -->
+	<!-- 	<origin xyz="0.22 0.0 0.2" rpy="0 0 0" /> -->
+	<!-- </joint> -->
+	<link name='base_link'>
 		<pose>0 0 0.1 0 0 0</pose>
 		<inertial>
@@ -56,49 +55,50 @@
 		ixx="0.1000000042" ixy="0" ixz="0" iyy="0.1000000042" iyz="0" izz="0.1000000040" radius="0.155"
 		length="0.06" radius_2="0.0028" length_2="0.005" material="grey" />
-	<!-- joint between chassis and Left wheel-->
-	<xacro:w_joint name="chassis_to_left_wheel" type="continuous" axis_xyz="0 0 1" axis_rpy="0 0 0"
+	<!-- joint between base_link and Left wheel-->
+	<xacro:w_joint name="base_link_to_left_wheel" type="continuous" axis_xyz="0 0 1" axis_rpy="0 0 0"
 		limit_e="100" limit_v="20" damping="1.0" friction="0.01" origin_rpy="-1.57 0 0"
-		origin_xyz="-0.22 0.28 -0.285" parent="chassis" child="left_wheel" />
+		origin_xyz="-0.22 0.28 -0.285" parent="base_link" child="left_wheel" />
 	<!--  inertia values are added by 0.1 in both left and right wheel to avoid collapsing of model in
 	gazebo-->
-	<!-- joint between chassis and Right Wheel-->
+	<!-- joint between base_link and Right Wheel-->
 	<!-- Right Wheel-->
 	<xacro:m1_link_cylinder name="right_wheel" origin_rpy="0 0 0" origin_xyz="0 0 0.027"
 		mass="0.10441" ixx="0.1000000042" ixy="0" ixz="0" iyy="0.1000000042" iyz="0" izz="0.1000000040"
 		radius="0.155" length="0.06" radius_2="0.0028" length_2="0.005" material="grey" />
-	<xacro:w_joint name="chassis_to_right_wheel" type="continuous" axis_xyz="0 0 1" axis_rpy="0 0 0"
+	<xacro:w_joint name="base_link_to_right_wheel" type="continuous" axis_xyz="0 0 1" axis_rpy="0 0 0"
 		limit_e="100" limit_v="20" damping="1.0" friction="0.01" origin_rpy="-1.57 0 0"
-		origin_xyz="-0.22 -0.32 -0.285" parent="chassis" child="right_wheel" />
+		origin_xyz="-0.22 -0.32 -0.285" parent="base_link" child="right_wheel" />
 	<!-- Caster 1,2 and there joints with Base Link-->
 	<xacro:m_link_sphere name="caster1" origin_rpy="0 0 0" origin_xyz="0 0 0" mass="0.45164"
 		ixx="0.100000005621" ixy="0.100000001310" ixz="0.100000001649" iyy="0.100000004345"
 		iyz="0.100000002360" izz="0.100000003315" material="black" radius="0.1" radius_2="0.001" />
-	<xacro:f_joint name="chassis_to_caster1" type="fixed" axis_xyz="0 0 0" origin_rpy="0 0 0"
-		origin_xyz="0.2 -0.25 -0.33" parent="chassis" child="caster1" />
+	<xacro:f_joint name="base_link_to_caster1" type="fixed" axis_xyz="0 0 0" origin_rpy="0 0 0"
+		origin_xyz="0.2 -0.25 -0.33" parent="base_link" child="caster1" />
 	<xacro:m_link_sphere name="caster2" origin_rpy="0 0 0" origin_xyz="0 0 0" mass="0.45164"
 		ixx="0.100000005621" ixy="0.100000001310" ixz="0.100000001649" iyy="0.100000004345"
 		iyz="0.100000002360" izz="0.100000003315" material="black" radius="0.1" radius_2="0.001" />
-	<xacro:f_joint name="chassis_to_caster2" type="fixed" axis_xyz="0 0 0" origin_rpy="0 0 0"
-		origin_xyz="0.2 0.25 -0.33" parent="chassis" child="caster2" />
+	<xacro:f_joint name="base_link_to_caster2" type="fixed" axis_xyz="0 0 0" origin_rpy="0 0 0"
+		origin_xyz="0.2 0.25 -0.33" parent="base_link" child="caster2" />
 	<xacro:f_link_box name="rod1" origin_rpy="0 0 0" origin_xyz="0 0 0" mass="0.45164"
 		ixx="0.100000005621" ixy="0.100000001310" ixz="0.100000001649" iyy="0.100000004345"
 		iyz="0.100000002360" izz="0.100000003315" material="black" size="0.016 0.016 0.6" />
-	<xacro:f_joint name="chassis_to_rod1" type="fixed" axis_xyz="0 0 0" origin_rpy="0 0 0"
-		origin_xyz="-0.23 0.24 0.65" parent="chassis" child="rod1" />
+	<xacro:f_joint name="base_link_to_rod1" type="fixed" axis_xyz="0 0 0" origin_rpy="0 0 0"
+		origin_xyz="-0.23 0.24 0.65" parent="base_link" child="rod1" />
 	<xacro:f_link_box name="rod2" origin_rpy="0 0 0" origin_xyz="0 0 0" mass="0.45164"
 		ixx="0.100000005621" ixy="0.100000001310" ixz="0.100000001649" iyy="0.100000004345"
 		iyz="0.100000002360" izz="0.100000003315" material="black" size="0.016 0.016 0.6" />
-	<xacro:f_joint name="chassis_to_rod2" type="fixed" axis_xyz="0 0 0" origin_rpy="0 0 0"
-		origin_xyz="-0.23 -0.24 0.65" parent="chassis" child="rod2" />
+	<xacro:f_joint name="base_link_to_rod2" type="fixed" axis_xyz="0 0 0" origin_rpy="0 0 0"
+		origin_xyz="-0.23 -0.24 0.65" parent="base_link" child="rod2" />
 	<xacro:f_link_box name="camera_base_rod" origin_rpy="0 0 0" origin_xyz="0 0 0" mass="0.45164"
 		ixx="0.100000005621" ixy="0.100000001310" ixz="0.100000001649" iyy="0.100000004345"
 		iyz="0.100000002360" izz="0.100000003315" material="black" size="0.016 0.48 0.016" />
-	<xacro:f_joint name="chassis_to_camera_base_rod" type="fixed" axis_xyz="0 0 0" origin_rpy="0 0 0"
-		origin_xyz="-0.23 0 0.650" parent="chassis" child="camera_base_rod" />
+	<xacro:f_joint name="base_link_to_camera_base_rod" type="fixed" axis_xyz="0 0 0"
+		origin_rpy="0 0 0"
+		origin_xyz="-0.23 0 0.650" parent="base_link" child="camera_base_rod" />
 	<xacro:f_link_box name="lidar_base_rod" origin_rpy="0 0 0" origin_xyz="0 0 0" mass="0.45164"
 		ixx="0.100000005621" ixy="0.100000001310" ixz="0.100000001649" iyy="0.100000004345"
 		iyz="0.100000002360" izz="0.100000003315" material="black" size="0.016 0.48 0.016" />
-	<xacro:f_joint name="chassis_to_lidar_base_rod" type="fixed" axis_xyz="0 0 0" origin_rpy="0 0 0"
-		origin_xyz="0.23 0 -0.15" parent="chassis" child="lidar_base_rod" />
+	<xacro:f_joint name="base_link_to_lidar_base_rod" type="fixed" axis_xyz="0 0 0" origin_rpy="0 0 0"
+		origin_xyz="0.23 0 -0.15" parent="base_link" child="lidar_base_rod" />
 	<!--Lidar-->
 	<xacro:m_link_cylinder name="laser" origin_rpy="0 0 0" origin_xyz="0 0 0" mass="0.10441"
@@ -106,7 +106,7 @@
 		material="black" filename="file://$(find wheelchair2_description)/meshes/rplidar.dae"
 		scale="1 1 1" />
-	<!-- joint between chassis and lidar -->
-	<xacro:f_joint name="chassis_to_rplidar" type="fixed" axis_xyz="0 0 0" origin_rpy="0 0 0"
-		origin_xyz="0.53 0 -0.15" parent="chassis" child="laser" />
+	<!-- joint between base_link and lidar -->
+	<xacro:f_joint name="base_link_to_rplidar" type="fixed" axis_xyz="0 0 0" origin_rpy="0 0 0"
+		origin_xyz="0.53 0 -0.15" parent="base_link" child="laser" />
 	<xacro:realsense parent="base_link" name="camera">
 		<origin xyz="0.20 -0.24 0.50" rpy="0 -0.01 0" />

File: wheelchair2_description/urdf/wheelchair2_camera_lidar_gazebo.urdf.xacro (robot description, xacro)
@@ -20,5 +20,5 @@
 	<!--Gazebo
 	related physics values of left wheel joint-->
-	<gazebo reference="chassis_to_left_wheel">
+	<gazebo reference="base_link_to_left_wheel">
 		<mu1 value="10000.0" />
 		<mu2 value="10000.0" />
@@ -33,5 +33,5 @@
 	</gazebo>
 	<!-- Gazebo related physics values of right wheel joint-->
-	<gazebo reference="chassis_to_right_wheel">
+	<gazebo reference="base_link_to_right_wheel">
 		<mu1 value="10000.0" />
 		<mu2 value="10000.0" />
@@ -43,5 +43,5 @@
 		<minDepth value="0.0001" />
 	</gazebo>
-	<gazebo reference="chassis">
+	<gazebo reference="base_link">
 		<material>Gazebo/FlatBlack</material>
 	</gazebo>
