Commit message: removed simulation parts

File: wheelchair2_description/urdf/kangaroo_ros2_control.urdf.xacro (robot description, xacro)
@@ -1,24 +1,18 @@
 <?xml version="1.0" encoding="UTF-8"?>
 <robot xmlns:xacro="http://www.ros.org/wiki/xacro">
-	<xacro:macro name="kangaroo_x2_driver" params="name prefix is_sim">
-		<ros2_control name="${name}" type="system">
+	<xacro:macro name="kangaroo_x2_driver">
+		<ros2_control name="kangaroo_ros2_control" type="system">
 			<hardware>
-				<xacro:if value="${is_sim}">
-					<plugin>gazebo_ros2_control/GazeboSystem</plugin>
-				</xacro:if>
-				<xacro:unless value="${is_sim}">
-					<plugin>wheelchair2_kangaroo_x2_driver/Kangaroo</plugin>
-					<!-- <plugin>mock_components/GenericSystem</plugin> -->
-					<param name="left_wheel_name">base_link_to_left_wheel</param>
-					<param name="right_wheel_name">base_link_to_right_wheel</param>
-					<param name="wheel_diameter">0.32</param>
-					<param name="wheel_center_distance">0.55</param>
-					<param name="encoder_lines_per_revolution">65536</param>
-					<param name="hz">50</param>
-					<param name="port">/dev/ttyACM0</param>
-					<param name="mixed_mode">true</param>
-				</xacro:unless>
+				<plugin>wheelchair2_kangaroo_x2_driver/Kangaroo</plugin>
+				<param name="left_wheel_name">base_link_to_left_wheel</param>
+				<param name="right_wheel_name">base_link_to_right_wheel</param>
+				<param name="wheel_diameter">0.32</param>
+				<param name="wheel_center_distance">0.55</param>
+				<param name="encoder_lines_per_revolution">65536</param>
+				<param name="hz">50</param>
+				<param name="port">/dev/ttyACM0</param>
+				<param name="mixed_mode">true</param>
 			</hardware>
-			<joint name="${prefix}base_link_to_left_wheel">
+			<joint name="base_link_to_left_wheel">
 				<command_interface name="velocity">
 					<param name="min">-1</param>
@@ -28,5 +22,5 @@
 				<state_interface name="velocity" />
 			</joint>
-			<joint name="${prefix}base_link_to_right_wheel">
+			<joint name="base_link_to_right_wheel">
 				<command_interface name="velocity">
 					<param name="min">-1</param>

File: wheelchair2_description/urdf/wheelchair2_camera_livox.urdf.xacro (robot description, xacro)
@@ -4,16 +4,10 @@
 	<!-- Include Files-->
 	<xacro:include filename="$(find wheelchair2_description)/urdf/links_joints.urdf.xacro" />
-	<!-- <xacro:include -->
-		<!-- filename="$(find wheelchair2_description)/urdf/wheelchair2_camera_lidar_gazebo.urdf.xacro" /> -->
 	<xacro:include filename="$(find wheelchair2_description)/urdf/kangaroo_ros2_control.urdf.xacro" />
 	<xacro:include filename="$(find wheelchair2_description)/urdf/realsense.urdf.xacro" />
 	<xacro:include filename="$(find wheelchair2_description)/urdf/mid360.xacro" />
-	<!-- <xacro:include filename="$(find wheelchair2_description)/urdf/wheelchair2_livox_gazebo.urdf.xacro" /> -->
 	<xacro:arg name="use_nominal_extrinsics" default="false" />
 	<xacro:arg name="add_plug" default="false" />
 	<xacro:arg name="use_mesh" default="true" />
-	<xacro:arg name="is_sim" default="true" />
-	<xacro:arg name="gazebo_controllers"
-		default="$(find wheelchair2_bringup)/config/wheelchair2_controllers.yaml" />
 	<link name="base_footprint" />
 	<!-- Add Base Footprint -->
@@ -23,9 +17,4 @@
 		<origin xyz="0.22 0 0.2" rpy="0 0 0" />
 	</joint>
-	<!-- <joint name="base_joint" type="fixed"> -->
-	<!-- 	<parent link="base_link" /> -->
-	<!-- 	<child link="chassis" /> -->
-	<!-- 	<origin xyz="0.22 0.0 0.2" rpy="0 0 0" /> -->
-	<!-- </joint> -->
 	<link name='base_link'>
 		<pose>0 0 0.1 0 0 0</pose>
@@ -118,17 +107,4 @@
 		<origin xyz="-0.05 0 -0.05" rpy="3.14 0 0" />
 	</xacro:mid360>
-	<xacro:kangaroo_x2_driver name="kangaroo_ros2_control" prefix="" is_sim="$(arg is_sim)"></xacro:kangaroo_x2_driver>
-	<!-- Gazebo Plugin-->
-	<xacro:if value="$(arg is_sim)">
-		<gazebo>
-			<plugin name="gazebo_ros2_control" filename="libgazebo_ros2_control.so">
-				<parameters>$(arg gazebo_controllers)</parameters>
-				<parameters>$(find wheelchair2_bringup)/config/gazebo_ros2_control.yaml</parameters>
-				<ros>
-					<remapping>/wheelchair2_base_controller/cmd_vel_unstamped:=/cmd_vel</remapping>
-					<remapping>/wheelchair2_base_controller/odom:=/odom</remapping>
-				</ros>
-			</plugin>
-		</gazebo>
-	</xacro:if>
+	<xacro:kangaroo_x2_driver/>
 </robot>

Commit message: included gazebo parts to the motor driver

File: wheelchair2_description/urdf/kangaroo_ros2_control.urdf.xacro (robot description, xacro)
@@ -1,18 +1,24 @@
 <?xml version="1.0" encoding="UTF-8"?>
 <robot xmlns:xacro="http://www.ros.org/wiki/xacro">
-	<xacro:macro name="kangaroo_x2_driver">
-		<ros2_control name="kangaroo_ros2_control" type="system">
+	<xacro:macro name="kangaroo_x2_driver" params="name prefix is_sim">
+		<ros2_control name="${name}" type="system">
 			<hardware>
-				<plugin>wheelchair2_kangaroo_x2_driver/Kangaroo</plugin>
-				<param name="left_wheel_name">base_link_to_left_wheel</param>
-				<param name="right_wheel_name">base_link_to_right_wheel</param>
-				<param name="wheel_diameter">0.32</param>
-				<param name="wheel_center_distance">0.55</param>
-				<param name="encoder_lines_per_revolution">65536</param>
-				<param name="hz">50</param>
-				<param name="port">/dev/ttyACM0</param>
-				<param name="mixed_mode">true</param>
+				<xacro:if value="${is_sim}">
+					<plugin>gz_ros2_control/GazeboSimSystem</plugin>
+				</xacro:if>
+				<xacro:unless value="${is_sim}">
+					<plugin>wheelchair2_kangaroo_x2_driver/Kangaroo</plugin>
+					<!-- <plugin>mock_components/GenericSystem</plugin> -->
+					<param name="left_wheel_name">base_link_to_left_wheel</param>
+					<param name="right_wheel_name">base_link_to_right_wheel</param>
+					<param name="wheel_diameter">0.32</param>
+					<param name="wheel_center_distance">0.55</param>
+					<param name="encoder_lines_per_revolution">65536</param>
+					<param name="hz">50</param>
+					<param name="port">/dev/ttyACM0</param>
+					<param name="mixed_mode">true</param>
+				</xacro:unless>
 			</hardware>
-			<joint name="base_link_to_left_wheel">
+			<joint name="${prefix}base_link_to_left_wheel">
 				<command_interface name="velocity">
 					<param name="min">-1</param>
@@ -22,5 +28,5 @@
 				<state_interface name="velocity" />
 			</joint>
-			<joint name="base_link_to_right_wheel">
+			<joint name="${prefix}base_link_to_right_wheel">
 				<command_interface name="velocity">
 					<param name="min">-1</param>

Commit message: moved unused urdf

File: wheelchair2_description/urdf/kangaroo_ros2_control.urdf.xacro (robot description, xacro)
@@ -1,11 +1,11 @@
 <?xml version="1.0" encoding="UTF-8"?>
 <robot xmlns:xacro="http://www.ros.org/wiki/xacro">
-	<xacro:macro name="kangaroo_x2_driver" params="name prefix is_sim">
+	<xacro:macro name="kangaroo_x2_driver" params="name prefix use_sim_time">
 		<ros2_control name="${name}" type="system">
 			<hardware>
-				<xacro:if value="${is_sim}">
+				<xacro:if value="${use_sim_time}">
 					<plugin>gz_ros2_control/GazeboSimSystem</plugin>
 				</xacro:if>
-				<xacro:unless value="${is_sim}">
+				<xacro:unless value="${use_sim_time}">
 					<plugin>wheelchair2_kangaroo_x2_driver/Kangaroo</plugin>
 					<!-- <plugin>mock_components/GenericSystem</plugin> -->
@@ -25,6 +25,6 @@
 					<param name="max">1</param>
 				</command_interface>
-				<state_interface name="position" />
-				<state_interface name="velocity" />
+				<state_interface name="position"/>
+				<state_interface name="velocity"/>
 			</joint>
 			<joint name="${prefix}base_link_to_right_wheel">
@@ -33,6 +33,6 @@
 					<param name="max">1</param>
 				</command_interface>
-				<state_interface name="position" />
-				<state_interface name="velocity" />
+				<state_interface name="position"/>
+				<state_interface name="velocity"/>
 			</joint>
 		</ros2_control>
