Commit message: added dual camera support

File: wheelchair2_description/urdf/realsense.urdf.xacro (robot description, xacro)
@@ -111,13 +111,11 @@
 		<link name="${name}_color_optical_frame" />
 		<xacro:if value="${use_sim_time}">
-			<!-- Realsense Gazebo Plugin -->
-			<gazebo reference="camera_link">
+			<gazebo reference="${name}_link">
 				<material>Gazebo/Black</material>
-				<sensor name="camera" type="camera">
-					<pose> 0 0 0 0 0 0 </pose>
+				<sensor name="${name}_camera_sensor" type="camera"> <pose> 0 0 0 0 0 0 </pose>
 					<visualize>true</visualize>
 					<update_rate>10</update_rate>
 					<camera>
-						<camera_info_topic>camera/camera_info</camera_info_topic>
+						<camera_info_topic>${topics_ns}/color/camera_info</camera_info_topic>
 						<horizontal_fov>1.089</horizontal_fov>
 						<image>
@@ -131,6 +129,13 @@
 						</clip>
 					</camera>
-					<topic>camera/image_raw</topic>
-					<gz_frame_id>camera_link</gz_frame_id>
+					<plugin name="camera_controller" filename="libgazebo_ros_camera.so">
+						<ros>
+							<namespace>${topics_ns}</namespace>
+							<remapping>image_raw:=color/image_raw</remapping>
+							<remapping>camera_info:=color/camera_info</remapping>
+						</ros>
+						<camera_name>${name}_color</camera_name>
+						<frame_name>${name}_color_optical_frame</frame_name>
+					</plugin>
 				</sensor>
 			</gazebo>

File: wheelchair2_description/urdf/wheelchair2_core.urdf.xacro (robot description, xacro)
@@ -1,5 +1,5 @@
 <?xml version="1.0" encoding="UTF-8"?>
-<robot name="wheelchair2"
-    xmlns:xacro="http://www.ros.org/wiki/xacro">
+<robot name="wheelchair2" xmlns:xacro="http://www.ros.org/wiki/xacro">
+    <!-- <xacro:property name="pi" value="3.1415926535897931" /> -->
     <xacro:arg name="use_sim_time" default="false" />
     <xacro:arg name="use_nominal_extrinsics" default="false" />
@@ -30,5 +30,5 @@
         </collision>
         <visual>
-            <origin xyz="0 0 0" rpy="0 0 3.14"/>
+            <origin xyz="0 0 0" rpy="0 0 ${pi}"/>
             <geometry>
                 <mesh filename="file://$(find wheelchair2_description)/meshes/wheelchair2.dae" scale="0.01 0.01 0.01"/>
@@ -37,15 +37,8 @@
         </visual>
     </link>
-    <!-- Left Wheel-->
     <xacro:m1_link_cylinder name="left_wheel" origin_rpy="0 0 0" origin_xyz="0 0 0.027" mass="0.10441" ixx="0.1000000042" ixy="0" ixz="0" iyy="0.1000000042" iyz="0" izz="0.1000000040" radius="0.155" length="0.06" radius_2="0.0028" length_2="0.005" material="grey" />
-    <!-- joint between base_link and Left wheel-->
-    <xacro:w_joint name="base_link_to_left_wheel" type="continuous" axis_xyz="0 0 1" axis_rpy="0 0 0" limit_e="100" limit_v="20" damping="1.0" friction="0.01" origin_rpy="-1.57 0 0" origin_xyz="-0.22 0.28 -0.285" parent="base_link" child="left_wheel" />
-    <!--  inertia values are added by 0.1 in both left and right wheel to avoid collapsing of model in
-	gazebo-->
-    <!-- joint between base_link and Right Wheel-->
-    <!-- Right Wheel-->
+    <xacro:w_joint name="base_link_to_left_wheel" type="continuous" axis_xyz="0 0 1" axis_rpy="0 0 0" limit_e="100" limit_v="20" damping="1.0" friction="0.01" origin_rpy="-${pi/2} 0 0" origin_xyz="-0.22 0.28 -0.285" parent="base_link" child="left_wheel" />
     <xacro:m1_link_cylinder name="right_wheel" origin_rpy="0 0 0" origin_xyz="0 0 0.027" mass="0.10441" ixx="0.1000000042" ixy="0" ixz="0" iyy="0.1000000042" iyz="0" izz="0.1000000040" radius="0.155" length="0.06" radius_2="0.0028" length_2="0.005" material="grey" />
-    <xacro:w_joint name="base_link_to_right_wheel" type="continuous" axis_xyz="0 0 1" axis_rpy="0 0 0" limit_e="100" limit_v="20" damping="1.0" friction="0.01" origin_rpy="-1.57 0 0" origin_xyz="-0.22 -0.28 -0.285" parent="base_link" child="right_wheel" />
-    <!-- Caster 1,2 and there joints with Base Link-->
+    <xacro:w_joint name="base_link_to_right_wheel" type="continuous" axis_xyz="0 0 1" axis_rpy="0 0 0" limit_e="100" limit_v="20" damping="1.0" friction="0.01" origin_rpy="-${pi/2} 0 0" origin_xyz="-0.22 -0.28 -0.285" parent="base_link" child="right_wheel" />
     <xacro:m_link_sphere name="caster1" origin_rpy="0 0 0" origin_xyz="0 0 0" mass="0.45164" ixx="0.100000005621" ixy="0.100000001310" ixz="0.100000001649" iyy="0.100000004345" iyz="0.100000002360" izz="0.100000003315" material="black" radius="0.1" radius_2="0.001" />
     <xacro:f_joint name="base_link_to_caster1" type="fixed" axis_xyz="0 0 0" origin_rpy="0 0 0" origin_xyz="0.2 -0.25 -0.33" parent="base_link" child="caster1" />
@@ -58,25 +51,24 @@
     <xacro:f_link_box name="camera_base_rod" origin_rpy="0 0 0" origin_xyz="0 0 0" mass="0.45164" ixx="0.100000005621" ixy="0.100000001310" ixz="0.100000001649" iyy="0.100000004345" iyz="0.100000002360" izz="0.100000003315" material="black" size="0.016 0.48 0.016" />
     <xacro:f_joint name="base_link_to_camera_base_rod" type="fixed" axis_xyz="0 0 0" origin_rpy="0 0 0" origin_xyz="-0.23 0 0.650" parent="base_link" child="camera_base_rod" />
-    <!-- 3D Printed Mount -->
     <link name="camera_mount_link"/>
     <joint name="base_to_camera_mount" type="fixed">
-        <origin xyz="-0.19159 0 1.2144" rpy="0 0 0" />
         <parent link="base_link"/>
         <child link="camera_mount_link"/>
+        <origin xyz="-0.19159 0 1.2144" rpy="0 0 0" />
     </joint>
-    <!-- Realsense mounted to 3D printed mount -->
-    <xacro:realsense name="camera" parent="camera_mount_link" use_sim_time="$(arg use_sim_time)">
+    <xacro:realsense name="camera1" topics_ns="camera1" parent="camera_mount_link" use_sim_time="$(arg use_sim_time)">
         <origin xyz="0 0 0" rpy="0 0 0"/>
     </xacro:realsense>
-    <!-- livox link w.r.t camera_link -->
+    <xacro:realsense name="camera2" topics_ns="camera2" parent="camera_mount_link" use_sim_time="$(arg use_sim_time)">
+        <origin xyz="-0.13 0 0" rpy="0 0 -${pi}"/>
+    </xacro:realsense>
     <link name="livox_frame"/>
     <joint name="camera_link_to_livox_frame" type="fixed">
-        <origin xyz="-0.064156 0 -0.064846" rpy="-3.1416 -0.0131 0" />
-        <parent link="camera_link" />
+        <parent link="camera1_link" />
         <child link="livox_frame" />
+        <origin xyz="-0.064156 0 -0.064846" rpy="-${pi} -0.0131 0" />
         <axis xyz="0 0 0" />
     </joint>
     <xacro:kangaroo_x2_driver name="kangaroo_ros2_control" prefix="" use_sim_time="$(arg use_sim_time)"></xacro:kangaroo_x2_driver>
-    <!-- Gazebo Plugin-->
     <xacro:if value="$(arg use_sim_time)">
         <gazebo>
