Commit message: Added gui

File: wheelchair2_description/urdf/wheelchair2_core.urdf.xacro (robot description, xacro)
@@ -1,86 +1,108 @@
 <?xml version="1.0" encoding="UTF-8"?>
 <robot name="wheelchair2" xmlns:xacro="http://www.ros.org/wiki/xacro">
+    <!-- <xacro:property name="pi" value="3.1415926535897931" /> -->
+    <xacro:arg name="use_sim_time" default="false" />
+    <xacro:arg name="use_nominal_extrinsics" default="false" />
+    <xacro:arg name="add_plug" default="false" />
+    <xacro:arg name="use_mesh" default="true" />
+    <xacro:include filename="$(find wheelchair2_description)/urdf/links_joints.urdf.xacro" />
     <xacro:include filename="$(find wheelchair2_description)/urdf/kangaroo_ros2_control.urdf.xacro" />
+    <xacro:include filename="$(find wheelchair2_description)/urdf/realsense.urdf.xacro" />
     <link name="base_footprint" />
     <joint name="base_footprint_joint" type="fixed">
         <parent link="base_footprint" />
         <child link="base_link" />
-        <origin xyz="0 0 0.16" rpy="0 0 0" />
+        <origin xyz="0.22 0 0.2" rpy="0 0 0" />
     </joint>
     <link name="base_link">
+        <pose>0 0 0.1 0 0 0</pose>
+        <inertial>
+            <mass value="8.96"/>
+            <origin xyz="0 0 0" rpy="0 0 0"/>
+            <inertia ixx="2.83" ixy="-0.12" ixz="-1.17" iyy="3.47" iyz="0.29" izz="0.73"/>
+        </inertial>
+        <collision>
+            <origin xyz="0.1 0 0" rpy="0 0 0"/>
+            <geometry>
+                <box size="0.75 0.60 0.60"/>
+            </geometry>
+            <material name="black"/>
+        </collision>
         <visual>
-            <origin xyz="0.215 0 0.2" rpy="0 0 0"/>
+            <origin xyz="0 0 0" rpy="0 0 ${pi}"/>
             <geometry>
-                <box size="1.13 0.66 0.5"/>
+                <mesh filename="file://$(find wheelchair2_description)/meshes/wheelchair2.dae" scale="0.01 0.01 0.01"/>
             </geometry>
-            <material name="blue">
-                <color rgba="0 0 0.8 0.5"/>
-            </material>
+            <material name="black"/>
         </visual>
     </link>
-    <link name="left_wheel">
-        <visual>
-            <geometry><cylinder radius="0.16" length="0.05"/></geometry>
-            <material name="black"><color rgba="0 0 0 1"/></material>
-        </visual>
+    <xacro:m1_link_cylinder name="left_wheel" origin_rpy="0 0 0" origin_xyz="0 0 0.027" mass="0.10441" ixx="0.1000000042" ixy="0" ixz="0" iyy="0.1000000042" iyz="0" izz="0.1000000040" radius="0.155" length="0.06" radius_2="0.0028" length_2="0.005" material="grey" />
+    <xacro:w_joint name="base_link_to_left_wheel" type="continuous" axis_xyz="0 0 1" axis_rpy="0 0 0" limit_e="100" limit_v="20" damping="1.0" friction="0.01" origin_rpy="-${pi/2} 0 0" origin_xyz="-0.22 0.28 -0.285" parent="base_link" child="left_wheel" />
+    <xacro:m1_link_cylinder name="right_wheel" origin_rpy="0 0 0" origin_xyz="0 0 0.027" mass="0.10441" ixx="0.1000000042" ixy="0" ixz="0" iyy="0.1000000042" iyz="0" izz="0.1000000040" radius="0.155" length="0.06" radius_2="0.0028" length_2="0.005" material="grey" />
+    <xacro:w_joint name="base_link_to_right_wheel" type="continuous" axis_xyz="0 0 1" axis_rpy="0 0 0" limit_e="100" limit_v="20" damping="1.0" friction="0.01" origin_rpy="-${pi/2} 0 0" origin_xyz="-0.22 -0.28 -0.285" parent="base_link" child="right_wheel" />
+    <xacro:m_link_sphere name="caster1" origin_rpy="0 0 0" origin_xyz="0 0 0" mass="0.45164" ixx="0.100000005621" ixy="0.100000001310" ixz="0.100000001649" iyy="0.100000004345" iyz="0.100000002360" izz="0.100000003315" material="black" radius="0.1" radius_2="0.001" />
+    <xacro:f_joint name="base_link_to_caster1" type="fixed" axis_xyz="0 0 0" origin_rpy="0 0 0" origin_xyz="0.2 -0.25 -0.33" parent="base_link" child="caster1" />
+    <xacro:m_link_sphere name="caster2" origin_rpy="0 0 0" origin_xyz="0 0 0" mass="0.45164" ixx="0.100000005621" ixy="0.100000001310" ixz="0.100000001649" iyy="0.100000004345" iyz="0.100000002360" izz="0.100000003315" material="black" radius="0.1" radius_2="0.001" />
+    <xacro:f_joint name="base_link_to_caster2" type="fixed" axis_xyz="0 0 0" origin_rpy="0 0 0" origin_xyz="0.2 0.25 -0.33" parent="base_link" child="caster2" />
+    <xacro:f_link_box name="rod1" origin_rpy="0 0 0" origin_xyz="0 0 0" mass="0.45164" ixx="0.100000005621" ixy="0.100000001310" ixz="0.100000001649" iyy="0.100000004345" iyz="0.100000002360" izz="0.100000003315" material="black" size="0.016 0.016 0.6" />
+    <xacro:f_joint name="base_link_to_rod1" type="fixed" axis_xyz="0 0 0" origin_rpy="0 0 0" origin_xyz="-0.23 0.24 0.65" parent="base_link" child="rod1" />
+    <xacro:f_link_box name="rod2" origin_rpy="0 0 0" origin_xyz="0 0 0" mass="0.45164" ixx="0.100000005621" ixy="0.100000001310" ixz="0.100000001649" iyy="0.100000004345" iyz="0.100000002360" izz="0.100000003315" material="black" size="0.016 0.016 0.6" />
+    <xacro:f_joint name="base_link_to_rod2" type="fixed" axis_xyz="0 0 0" origin_rpy="0 0 0" origin_xyz="-0.23 -0.24 0.65" parent="base_link" child="rod2" />
+    <xacro:f_link_box name="camera_base_rod" origin_rpy="0 0 0" origin_xyz="0 0 0" mass="0.45164" ixx="0.100000005621" ixy="0.100000001310" ixz="0.100000001649" iyy="0.100000004345" iyz="0.100000002360" izz="0.100000003315" material="black" size="0.016 0.48 0.016" />
+    <xacro:f_joint name="base_link_to_camera_base_rod" type="fixed" axis_xyz="0 0 0" origin_rpy="0 0 0" origin_xyz="-0.23 0 0.650" parent="base_link" child="camera_base_rod" />
+    <link name="camera_mount_link"/>
+    <joint name="base_to_camera_mount" type="fixed">
+        <parent link="base_link"/>
+        <child link="camera_mount_link"/>
+        <origin xyz="-0.19159 0 1.2144" rpy="0 0 0" />
+    </joint>
+    <xacro:realsense name="camera1" topics_ns="camera1" parent="camera_mount_link" use_sim_time="$(arg use_sim_time)">
+        <origin xyz="0 0 0" rpy="0 0 0"/>
+    </xacro:realsense>
+    <xacro:realsense name="camera2" topics_ns="camera2" parent="camera_mount_link" use_sim_time="$(arg use_sim_time)">
+        <origin xyz="-0.13 0 0" rpy="0 0 -${pi}"/>
+    </xacro:realsense>
+    <link name="livox_frame"/>
+    <joint name="camera_link_to_livox_frame" type="fixed">
+        <parent link="camera1_link" />
+        <child link="livox_frame" />
+        <origin xyz="-0.064156 0 -0.064846" rpy="-${pi} -0.0131 0" />
+        <axis xyz="0 0 0" />
+    </joint>
+         <joint name="base_footprint_imu_joint" type="fixed">
+        <parent link="base_footprint" />
+        <child link="imu_link" />
+        <origin xyz="0.22 0 0.2" rpy="0 0 0" />
+    </joint>
+    <link name="imu_link">
+        <pose>0 0 0.1 0 0 0</pose>
+        <inertial>
+            <mass value="8.96"/>
+            <origin xyz="0 0 0" rpy="0 0 0"/>
+            <inertia ixx="2.83" ixy="-0.12" ixz="-1.17" iyy="3.47" iyz="0.29" izz="0.73"/>
+        </inertial>
+        <collision>
+            <origin xyz="0.1 0 0" rpy="0 0 0"/>
+            <geometry>
+                <box size="0.75 0.60 0.60"/>
+            </geometry>
+            <material name="black"/>
+        </collision>
     </link>
-    <joint name="base_link_to_left_wheel" type="continuous">
-        <parent link="base_link"/>
-        <child link="left_wheel"/>
-        <origin xyz="0 0.2775 0" rpy="-1.570796 0 0"/>
-        <axis xyz="0 0 1"/>
-    </joint>
-    <link name="right_wheel">
-        <visual>
-            <geometry><cylinder radius="0.16" length="0.05"/></geometry>
-            <material name="black"><color rgba="0 0 0 1"/></material>
-        </visual>
-    </link>
-    <joint name="base_link_to_right_wheel" type="continuous">
-        <parent link="base_link"/>
-        <child link="right_wheel"/>
-        <origin xyz="0 -0.2775 0" rpy="-1.570796 0 0"/>
-        <axis xyz="0 0 1"/>
-    </joint>
-    <link name="caster_left">
-        <visual>
-            <geometry><sphere radius="0.1"/></geometry>
-            <material name="grey"><color rgba="0.5 0.5 0.5 1"/></material>
-        </visual>
-    </link>
-    <joint name="caster_left_joint" type="fixed">
-        <parent link="base_link"/>
-        <child link="caster_left"/>
-        <origin xyz="0.49 0.2775 -0.06" rpy="0 0 0"/>
-    </joint>
-    <link name="caster_right">
-        <visual>
-            <geometry><sphere radius="0.1"/></geometry>
-            <material name="grey"><color rgba="0.5 0.5 0.5 1"/></material>
-        </visual>
-    </link>
-    <joint name="caster_right_joint" type="fixed">
-        <parent link="base_link"/>
-        <child link="caster_right"/>
-        <origin xyz="0.49 -0.2775 -0.06" rpy="0 0 0"/>
-    </joint>
     <link name="laser"/>
     <joint name="base_to_laser" type="fixed">
         <parent link="base_link" />
         <child link="laser" />
-        <origin xyz="0.23 0.0057 0.68" rpy="3.14159 0 0" />
+        <origin xyz="0.21 0 -0.095" rpy="0 3.14 0" />
     </joint>
-    <link name="livox_frame"/>
-    <joint name="base_to_livox" type="fixed">
-        <parent link="base_link" />
-        <child link="livox_frame" />
-        <origin xyz="0 0 1.44" rpy="3.14159 0 0" />
-    </joint>
-    <link name="imu_link"/>
-    <joint name="base_to_imu" type="fixed">
-        <parent link="base_link" />
-        <child link="imu_link" />
-        <origin xyz="0.37 0 0" rpy="0 0 0" />
-    </joint>
-    <xacro:kangaroo_x2_driver name="kangaroo_ros2_control" prefix="" use_sim_time="false"/>
+    <xacro:kangaroo_x2_driver name="kangaroo_ros2_control" prefix="" use_sim_time="$(arg use_sim_time)"></xacro:kangaroo_x2_driver>
+    <xacro:if value="$(arg use_sim_time)">
+        <gazebo>
+            <plugin name="gz_ros2_control::GazeboSimROS2ControlPlugin" filename="libgz_ros2_control-system.so">
+                <parameters>$(find wheelchair2_control)/config/wheelchair2_controllers.yaml</parameters>
+            </plugin>
+        </gazebo>
+        <xacro:include filename="$(find wheelchair2_gazebo)/urdf/wheelchair2_gazebo.urdf.xacro" />
+        <xacro:include filename="$(find wheelchair2_gazebo)/urdf/livox.urdf.xacro" />
+    </xacro:if>
 </robot>

Commit message: Restructured urdf

File: wheelchair2_description/urdf/wheelchair2_core.urdf.xacro (robot description, xacro)
@@ -1,108 +1,86 @@
 <?xml version="1.0" encoding="UTF-8"?>
 <robot name="wheelchair2" xmlns:xacro="http://www.ros.org/wiki/xacro">
-    <!-- <xacro:property name="pi" value="3.1415926535897931" /> -->
-    <xacro:arg name="use_sim_time" default="false" />
-    <xacro:arg name="use_nominal_extrinsics" default="false" />
-    <xacro:arg name="add_plug" default="false" />
-    <xacro:arg name="use_mesh" default="true" />
-    <xacro:include filename="$(find wheelchair2_description)/urdf/links_joints.urdf.xacro" />
     <xacro:include filename="$(find wheelchair2_description)/urdf/kangaroo_ros2_control.urdf.xacro" />
-    <xacro:include filename="$(find wheelchair2_description)/urdf/realsense.urdf.xacro" />
     <link name="base_footprint" />
     <joint name="base_footprint_joint" type="fixed">
         <parent link="base_footprint" />
         <child link="base_link" />
-        <origin xyz="0.22 0 0.2" rpy="0 0 0" />
+        <origin xyz="0 0 0.16" rpy="0 0 0" />
     </joint>
     <link name="base_link">
-        <pose>0 0 0.1 0 0 0</pose>
-        <inertial>
-            <mass value="8.96"/>
-            <origin xyz="0 0 0" rpy="0 0 0"/>
-            <inertia ixx="2.83" ixy="-0.12" ixz="-1.17" iyy="3.47" iyz="0.29" izz="0.73"/>
-        </inertial>
-        <collision>
-            <origin xyz="0.1 0 0" rpy="0 0 0"/>
+        <visual>
+            <origin xyz="0.215 0 0.2" rpy="0 0 0"/>
             <geometry>
-                <box size="0.75 0.60 0.60"/>
+                <box size="1.13 0.66 0.5"/>
             </geometry>
-            <material name="black"/>
-        </collision>
-        <visual>
-            <origin xyz="0 0 0" rpy="0 0 ${pi}"/>
-            <geometry>
-                <mesh filename="file://$(find wheelchair2_description)/meshes/wheelchair2.dae" scale="0.01 0.01 0.01"/>
-            </geometry>
-            <material name="black"/>
+            <material name="blue">
+                <color rgba="0 0 0.8 0.5"/>
+            </material>
         </visual>
     </link>
-    <xacro:m1_link_cylinder name="left_wheel" origin_rpy="0 0 0" origin_xyz="0 0 0.027" mass="0.10441" ixx="0.1000000042" ixy="0" ixz="0" iyy="0.1000000042" iyz="0" izz="0.1000000040" radius="0.155" length="0.06" radius_2="0.0028" length_2="0.005" material="grey" />
-    <xacro:w_joint name="base_link_to_left_wheel" type="continuous" axis_xyz="0 0 1" axis_rpy="0 0 0" limit_e="100" limit_v="20" damping="1.0" friction="0.01" origin_rpy="-${pi/2} 0 0" origin_xyz="-0.22 0.28 -0.285" parent="base_link" child="left_wheel" />
-    <xacro:m1_link_cylinder name="right_wheel" origin_rpy="0 0 0" origin_xyz="0 0 0.027" mass="0.10441" ixx="0.1000000042" ixy="0" ixz="0" iyy="0.1000000042" iyz="0" izz="0.1000000040" radius="0.155" length="0.06" radius_2="0.0028" length_2="0.005" material="grey" />
-    <xacro:w_joint name="base_link_to_right_wheel" type="continuous" axis_xyz="0 0 1" axis_rpy="0 0 0" limit_e="100" limit_v="20" damping="1.0" friction="0.01" origin_rpy="-${pi/2} 0 0" origin_xyz="-0.22 -0.28 -0.285" parent="base_link" child="right_wheel" />
-    <xacro:m_link_sphere name="caster1" origin_rpy="0 0 0" origin_xyz="0 0 0" mass="0.45164" ixx="0.100000005621" ixy="0.100000001310" ixz="0.100000001649" iyy="0.100000004345" iyz="0.100000002360" izz="0.100000003315" material="black" radius="0.1" radius_2="0.001" />
-    <xacro:f_joint name="base_link_to_caster1" type="fixed" axis_xyz="0 0 0" origin_rpy="0 0 0" origin_xyz="0.2 -0.25 -0.33" parent="base_link" child="caster1" />
-    <xacro:m_link_sphere name="caster2" origin_rpy="0 0 0" origin_xyz="0 0 0" mass="0.45164" ixx="0.100000005621" ixy="0.100000001310" ixz="0.100000001649" iyy="0.100000004345" iyz="0.100000002360" izz="0.100000003315" material="black" radius="0.1" radius_2="0.001" />
-    <xacro:f_joint name="base_link_to_caster2" type="fixed" axis_xyz="0 0 0" origin_rpy="0 0 0" origin_xyz="0.2 0.25 -0.33" parent="base_link" child="caster2" />
-    <xacro:f_link_box name="rod1" origin_rpy="0 0 0" origin_xyz="0 0 0" mass="0.45164" ixx="0.100000005621" ixy="0.100000001310" ixz="0.100000001649" iyy="0.100000004345" iyz="0.100000002360" izz="0.100000003315" material="black" size="0.016 0.016 0.6" />
-    <xacro:f_joint name="base_link_to_rod1" type="fixed" axis_xyz="0 0 0" origin_rpy="0 0 0" origin_xyz="-0.23 0.24 0.65" parent="base_link" child="rod1" />
-    <xacro:f_link_box name="rod2" origin_rpy="0 0 0" origin_xyz="0 0 0" mass="0.45164" ixx="0.100000005621" ixy="0.100000001310" ixz="0.100000001649" iyy="0.100000004345" iyz="0.100000002360" izz="0.100000003315" material="black" size="0.016 0.016 0.6" />
-    <xacro:f_joint name="base_link_to_rod2" type="fixed" axis_xyz="0 0 0" origin_rpy="0 0 0" origin_xyz="-0.23 -0.24 0.65" parent="base_link" child="rod2" />
-    <xacro:f_link_box name="camera_base_rod" origin_rpy="0 0 0" origin_xyz="0 0 0" mass="0.45164" ixx="0.100000005621" ixy="0.100000001310" ixz="0.100000001649" iyy="0.100000004345" iyz="0.100000002360" izz="0.100000003315" material="black" size="0.016 0.48 0.016" />
-    <xacro:f_joint name="base_link_to_camera_base_rod" type="fixed" axis_xyz="0 0 0" origin_rpy="0 0 0" origin_xyz="-0.23 0 0.650" parent="base_link" child="camera_base_rod" />
-    <link name="camera_mount_link"/>
-    <joint name="base_to_camera_mount" type="fixed">
+    <link name="left_wheel">
+        <visual>
+            <geometry><cylinder radius="0.16" length="0.05"/></geometry>
+            <material name="black"><color rgba="0 0 0 1"/></material>
+        </visual>
+    </link>
+    <joint name="base_link_to_left_wheel" type="continuous">
         <parent link="base_link"/>
-        <child link="camera_mount_link"/>
-        <origin xyz="-0.19159 0 1.2144" rpy="0 0 0" />
+        <child link="left_wheel"/>
+        <origin xyz="0 0.2775 0" rpy="-1.570796 0 0"/>
+        <axis xyz="0 0 1"/>
     </joint>
-    <xacro:realsense name="camera1" topics_ns="camera1" parent="camera_mount_link" use_sim_time="$(arg use_sim_time)">
-        <origin xyz="0 0 0" rpy="0 0 0"/>
-    </xacro:realsense>
-    <xacro:realsense name="camera2" topics_ns="camera2" parent="camera_mount_link" use_sim_time="$(arg use_sim_time)">
-        <origin xyz="-0.13 0 0" rpy="0 0 -${pi}"/>
-    </xacro:realsense>
-    <link name="livox_frame"/>
-    <joint name="camera_link_to_livox_frame" type="fixed">
-        <parent link="camera1_link" />
-        <child link="livox_frame" />
-        <origin xyz="-0.064156 0 -0.064846" rpy="-${pi} -0.0131 0" />
-        <axis xyz="0 0 0" />
+    <link name="right_wheel">
+        <visual>
+            <geometry><cylinder radius="0.16" length="0.05"/></geometry>
+            <material name="black"><color rgba="0 0 0 1"/></material>
+        </visual>
+    </link>
+    <joint name="base_link_to_right_wheel" type="continuous">
+        <parent link="base_link"/>
+        <child link="right_wheel"/>
+        <origin xyz="0 -0.2775 0" rpy="-1.570796 0 0"/>
+        <axis xyz="0 0 1"/>
     </joint>
-         <joint name="base_footprint_imu_joint" type="fixed">
-        <parent link="base_footprint" />
-        <child link="imu_link" />
-        <origin xyz="0.22 0 0.2" rpy="0 0 0" />
+    <link name="caster_left">
+        <visual>
+            <geometry><sphere radius="0.1"/></geometry>
+            <material name="grey"><color rgba="0.5 0.5 0.5 1"/></material>
+        </visual>
+    </link>
+    <joint name="caster_left_joint" type="fixed">
+        <parent link="base_link"/>
+        <child link="caster_left"/>
+        <origin xyz="0.49 0.2775 -0.06" rpy="0 0 0"/>
     </joint>
-    <link name="imu_link">
-        <pose>0 0 0.1 0 0 0</pose>
-        <inertial>
-            <mass value="8.96"/>
-            <origin xyz="0 0 0" rpy="0 0 0"/>
-            <inertia ixx="2.83" ixy="-0.12" ixz="-1.17" iyy="3.47" iyz="0.29" izz="0.73"/>
-        </inertial>
-        <collision>
-            <origin xyz="0.1 0 0" rpy="0 0 0"/>
-            <geometry>
-                <box size="0.75 0.60 0.60"/>
-            </geometry>
-            <material name="black"/>
-        </collision>
+    <link name="caster_right">
+        <visual>
+            <geometry><sphere radius="0.1"/></geometry>
+            <material name="grey"><color rgba="0.5 0.5 0.5 1"/></material>
+        </visual>
     </link>
+    <joint name="caster_right_joint" type="fixed">
+        <parent link="base_link"/>
+        <child link="caster_right"/>
+        <origin xyz="0.49 -0.2775 -0.06" rpy="0 0 0"/>
+    </joint>
     <link name="laser"/>
     <joint name="base_to_laser" type="fixed">
         <parent link="base_link" />
         <child link="laser" />
-        <origin xyz="0.21 0 -0.095" rpy="0 3.14 0" />
+        <origin xyz="0.23 0.0057 -0.068" rpy="0 3.14 0" />
     </joint>
-    <xacro:kangaroo_x2_driver name="kangaroo_ros2_control" prefix="" use_sim_time="$(arg use_sim_time)"></xacro:kangaroo_x2_driver>
-    <xacro:if value="$(arg use_sim_time)">
-        <gazebo>
-            <plugin name="gz_ros2_control::GazeboSimROS2ControlPlugin" filename="libgz_ros2_control-system.so">
-                <parameters>$(find wheelchair2_control)/config/wheelchair2_controllers.yaml</parameters>
-            </plugin>
-        </gazebo>
-        <xacro:include filename="$(find wheelchair2_gazebo)/urdf/wheelchair2_gazebo.urdf.xacro" />
-        <xacro:include filename="$(find wheelchair2_gazebo)/urdf/livox.urdf.xacro" />
-    </xacro:if>
+    <link name="livox_frame"/>
+    <joint name="base_to_livox" type="fixed">
+        <parent link="base_link" />
+        <child link="livox_frame" />
+        <origin xyz="0 0 1.44" rpy="3.14159 0 0" />
+    </joint>
+    <link name="imu_link"/>
+    <joint name="base_to_imu" type="fixed">
+        <parent link="base_link" />
+        <child link="imu_link" />
+        <origin xyz="0.37 0 0" rpy="0 0 0" />
+    </joint>
+    <xacro:kangaroo_x2_driver name="kangaroo_ros2_control" prefix="" use_sim_time="false"/>
 </robot>

Commit message: up with wi

File: wheelchair2_description/urdf/wheelchair2_core.urdf.xacro (robot description, xacro)
@@ -69,5 +69,5 @@
         <parent link="base_link" />
         <child link="laser" />
-        <origin xyz="0.23 0.0057 -0.068" rpy="0 3.14 0" />
+        <origin xyz="0.21 0.0057 -0.068" rpy="0 3.14 0" />
     </joint>
     <link name="livox_frame"/>
