Commit message: camera seems to work

File: wheelchair2_description/urdf/gz_sim/wheelchair2_camera_lidar.urdf.xacro (robot description, xacro)
@@ -8,5 +8,4 @@
 	<xacro:include filename="$(find wheelchair2_description)/urdf/gz_sim/realsense.urdf.xacro" />
 	<xacro:arg name="use_nominal_extrinsics" default="false" />
-	<xacro:arg name="add_plug" default="false" />
 	<xacro:arg name="use_mesh" default="true" />
 	<link name="base_link" />
@@ -23,5 +22,6 @@
 			<origin xyz="0 0 0" rpy=" 0 0 0" />
 			<!-- ALL INERTIA VALUES IN KILOGRAM PER SQUARE METER-->
-			<inertia ixx="2.83" ixy="-0.12" ixz="-1.17" iyy="3.47" iyz="0.29" izz="0.73" />
+			<!-- NOTE: z=c x=b y=a -->
+			<inertia ixx="6.47" ixy="-0.12" ixz="-1.17" iyy="8.54" iyz="0.29" izz="8.54" />
 		</inertial>
 		<collision>

File: wheelchair2_description/urdf/gz_sim/wheelchair2_camera_lidar_gz.urdf.xacro (robot description, xacro)
@@ -100,5 +100,5 @@
 		<sensor name="laser" type="gpu_lidar">
 			<pose> 0 0 0 0 0 0 </pose>
-			<visualize>false</visualize>
+			<visualize>true</visualize>
 			<update_rate>15</update_rate>
 			<topic>scan</topic>

File: wheelchair2_description/urdf/realsense.urdf.xacro (robot description, xacro)
@@ -8,5 +8,6 @@
 <robot name="realsense"
 	xmlns:xacro="http://ros.org/wiki/xacro">
-	<xacro:macro name="realsense" params="name:=camera topics_ns:=camera pointcloud:=false parent *origin">
+	<xacro:macro name="realsense"
+		params="name:=camera topics_ns:=camera pointcloud:=false parent *origin">
 		<xacro:property name="M_PI" value="3.1415926535897931" />
 		<!-- The following values are approximate, and the camera node
@@ -44,9 +45,11 @@
 		<link name="${name}_link">
 			<visual>
-				<origin xyz="${d435_cam_mount_from_center_offset} ${-d435_cam_depth_py} 0" rpy="${M_PI/2} 0 ${M_PI/2}" />
+				<origin xyz="${d435_cam_mount_from_center_offset} ${-d435_cam_depth_py} 0"
+					rpy="${M_PI/2} 0 ${M_PI/2}" />
 				<geometry>
 					<!-- <box size="${d435_cam_width} ${d435_cam_height} ${d435_cam_depth}"/> -->
 					<mesh filename="file://$(find wheelchair2_description)/meshes/d435.dae" />
-					<!--<mesh filename="file://$(find realsense2_description)/meshes/d435/d435.dae" />-->
+					<!--<mesh
+					filename="file://$(find realsense2_description)/meshes/d435/d435.dae" />-->
 				</geometry>
 				<material name="${name}_aluminum" />

File: wheelchair2_description/urdf/unused/wheelchair2_real_parth.urdf.xacro (robot description, xacro)
@@ -32,20 +32,25 @@
 				<box size="0.75 0.60 0.60" />
 			</geometry>
-			<material name="black" />
+			<!-- <material name="black" /> -->
 		</collision>
 		<visual>
 			<origin xyz="0 0 0" rpy=" 0 0 3.14" />
 			<geometry>
-				<mesh filename="package://wheelchair2_description/meshes/wheelchair2.dae" scale="0.01 0.01 0.01" />
+				<mesh filename="package://wheelchair2_description/meshes/wheelchair2.dae"
+					scale="0.01 0.01 0.01" />
 			</geometry>
-			<material name="black" />
+			<!-- <material name="black" /> -->
 		</visual>
 	</link>
 	<!--Left
 	Wheel-->
-	<xacro:m1_link_cylinder name="left_wheel" origin_rpy="0 0 0" origin_xyz="0 0 0.027" mass="0.10441" ixx="0.1000000042" ixy="0" ixz="0" iyy="0.1000000042" iyz="0" izz="0.1000000040" radius="0.155" length="0.06" radius_2="0.0028" length_2="0.005" material="grey" />
+	<xacro:m1_link_cylinder name="left_wheel" origin_rpy="0 0 0" origin_xyz="0 0 0.027" mass="0.10441"
+		ixx="0.1000000042" ixy="0" ixz="0" iyy="0.1000000042" iyz="0" izz="0.1000000040" radius="0.155"
+		length="0.06" radius_2="0.0028" length_2="0.005" material="grey" />
 	<!--joint
 	between chassis and Left wheel-->
-	<xacro:w_joint name="chassis_to_left_wheel" type="continuous" axis_xyz="0 0 1" axis_rpy="0 0 0" limit_e="100" limit_v="20" damping="1.0" friction="200000.0" origin_rpy="-1.57 0 0" origin_xyz="-0.22 0.28 -0.285" parent="chassis" child="left_wheel" />
+	<xacro:w_joint name="chassis_to_left_wheel" type="continuous" axis_xyz="0 0 1" axis_rpy="0 0 0"
+		limit_e="100" limit_v="20" damping="1.0" friction="200000.0" origin_rpy="-1.57 0 0"
+		origin_xyz="-0.22 0.28 -0.285" parent="chassis" child="left_wheel" />
 	<!-- inertia values are added by 0.1 in both left and right wheel to avoid collapsing of model in
 	gazebo-->
@@ -54,33 +59,60 @@
 	<!--Right
 	Wheel-->
-	<xacro:m1_link_cylinder name="right_wheel" origin_rpy="0 0 0" origin_xyz="0 0 0.027" mass="0.10441" ixx="0.1000000042" ixy="0" ixz="0" iyy="0.1000000042" iyz="0" izz="0.1000000040" radius="0.155" length="0.06" radius_2="0.0028" length_2="0.005" material="grey" />
-	<xacro:w_joint name="chassis_to_right_wheel" type="continuous" axis_xyz="0 0 1" axis_rpy="0 0 0" limit_e="100" limit_v="20" damping="1.0" friction="200000.0" origin_rpy="-1.57 0 0" origin_xyz="-0.22 -0.32 -0.285" parent="chassis" child="right_wheel" />
+	<xacro:m1_link_cylinder name="right_wheel" origin_rpy="0 0 0" origin_xyz="0 0 0.027"
+		mass="0.10441" ixx="0.1000000042" ixy="0" ixz="0" iyy="0.1000000042" iyz="0" izz="0.1000000040"
+		radius="0.155" length="0.06" radius_2="0.0028" length_2="0.005" material="grey" />
+	<xacro:w_joint name="chassis_to_right_wheel" type="continuous" axis_xyz="0 0 1" axis_rpy="0 0 0"
+		limit_e="100" limit_v="20" damping="1.0" friction="200000.0" origin_rpy="-1.57 0 0"
+		origin_xyz="-0.22 -0.32 -0.285" parent="chassis" child="right_wheel" />
 	<!--Caster
 	1,2 and there joints with Base Link-->
-	<xacro:m_link_sphere name="caster1" origin_rpy="0 0 0" origin_xyz="0 0 0" mass="0.45164" ixx="0.100000005621" ixy="0.100000001310" ixz="0.100000001649" iyy="0.100000004345" iyz="0.100000002360" izz="0.100000003315" material="black" radius="0.1" radius_2="0.001" />
-	<xacro:f_joint name="chassis_to_caster1" type="fixed" axis_xyz="0 0 0" origin_rpy="0 0 0" origin_xyz="0.2 -0.25 -0.33" parent="chassis" child="caster1" />
-	<xacro:m_link_sphere name="caster2" origin_rpy="0 0 0" origin_xyz="0 0 0" mass="0.45164" ixx="0.100000005621" ixy="0.100000001310" ixz="0.100000001649" iyy="0.100000004345" iyz="0.100000002360" izz="0.100000003315" material="black" radius="0.1" radius_2="0.001" />
-	<xacro:f_joint name="chassis_to_caster2" type="fixed" axis_xyz="0 0 0" origin_rpy="0 0 0" origin_xyz="0.2 0.25 -0.33" parent="chassis" child="caster2" />
-	<xacro:f_link_box name="rod1" origin_rpy="0 0 0" origin_xyz="0 0 0" mass="0.45164" ixx="0.100000005621" ixy="0.100000001310" ixz="0.100000001649" iyy="0.100000004345" iyz="0.100000002360" izz="0.100000003315" material="black" size="0.016 0.016 0.6" />
-	<xacro:f_joint name="chassis_to_rod1" type="fixed" axis_xyz="0 0 0" origin_rpy="0 0 0" origin_xyz="-0.23 0.24 0.65" parent="chassis" child="rod1" />
-	<xacro:f_link_box name="rod2" origin_rpy="0 0 0" origin_xyz="0 0 0" mass="0.45164" ixx="0.100000005621" ixy="0.100000001310" ixz="0.100000001649" iyy="0.100000004345" iyz="0.100000002360" izz="0.100000003315" material="black" size="0.016 0.016 0.6" />
-	<xacro:f_joint name="chassis_to_rod2" type="fixed" axis_xyz="0 0 0" origin_rpy="0 0 0" origin_xyz="-0.23 -0.24 0.65" parent="chassis" child="rod2" />
-	<xacro:f_link_box name="camera_base_rod" origin_rpy="0 0 0" origin_xyz="0 0 0" mass="0.45164" ixx="0.100000005621" ixy="0.100000001310" ixz="0.100000001649" iyy="0.100000004345" iyz="0.100000002360" izz="0.100000003315" material="black" size="0.016 0.48 0.016" />
-	<xacro:f_joint name="chassis_to_camera_base_rod" type="fixed" axis_xyz="0 0 0" origin_rpy="0 0 0" origin_xyz="-0.23 0 0.650" parent="chassis" child="camera_base_rod" />
-	<xacro:f_link_box name="lidar_base_rod" origin_rpy="0 0 0" origin_xyz="0 0 0" mass="0.45164" ixx="0.100000005621" ixy="0.100000001310" ixz="0.100000001649" iyy="0.100000004345" iyz="0.100000002360" izz="0.100000003315" material="black" size="0.016 0.48 0.016" />
-	<xacro:f_joint name="chassis_to_lidar_base_rod" type="fixed" axis_xyz="0 0 0" origin_rpy="0 0 0" origin_xyz="0.23 0 -0.15" parent="chassis" child="lidar_base_rod" />
+	<xacro:m_link_sphere name="caster1" origin_rpy="0 0 0" origin_xyz="0 0 0" mass="0.45164"
+		ixx="0.100000005621" ixy="0.100000001310" ixz="0.100000001649" iyy="0.100000004345"
+		iyz="0.100000002360" izz="0.100000003315" material="black" radius="0.1" radius_2="0.001" />
+	<xacro:f_joint name="chassis_to_caster1" type="fixed" axis_xyz="0 0 0" origin_rpy="0 0 0"
+		origin_xyz="0.2 -0.25 -0.33" parent="chassis" child="caster1" />
+	<xacro:m_link_sphere name="caster2" origin_rpy="0 0 0" origin_xyz="0 0 0" mass="0.45164"
+		ixx="0.100000005621" ixy="0.100000001310" ixz="0.100000001649" iyy="0.100000004345"
+		iyz="0.100000002360" izz="0.100000003315" material="black" radius="0.1" radius_2="0.001" />
+	<xacro:f_joint name="chassis_to_caster2" type="fixed" axis_xyz="0 0 0" origin_rpy="0 0 0"
+		origin_xyz="0.2 0.25 -0.33" parent="chassis" child="caster2" />
+	<xacro:f_link_box name="rod1" origin_rpy="0 0 0" origin_xyz="0 0 0" mass="0.45164"
+		ixx="0.100000005621" ixy="0.100000001310" ixz="0.100000001649" iyy="0.100000004345"
+		iyz="0.100000002360" izz="0.100000003315" material="black" size="0.016 0.016 0.6" />
+	<xacro:f_joint name="chassis_to_rod1" type="fixed" axis_xyz="0 0 0" origin_rpy="0 0 0"
+		origin_xyz="-0.23 0.24 0.65" parent="chassis" child="rod1" />
+	<xacro:f_link_box name="rod2" origin_rpy="0 0 0" origin_xyz="0 0 0" mass="0.45164"
+		ixx="0.100000005621" ixy="0.100000001310" ixz="0.100000001649" iyy="0.100000004345"
+		iyz="0.100000002360" izz="0.100000003315" material="black" size="0.016 0.016 0.6" />
+	<xacro:f_joint name="chassis_to_rod2" type="fixed" axis_xyz="0 0 0" origin_rpy="0 0 0"
+		origin_xyz="-0.23 -0.24 0.65" parent="chassis" child="rod2" />
+	<xacro:f_link_box name="camera_base_rod" origin_rpy="0 0 0" origin_xyz="0 0 0" mass="0.45164"
+		ixx="0.100000005621" ixy="0.100000001310" ixz="0.100000001649" iyy="0.100000004345"
+		iyz="0.100000002360" izz="0.100000003315" material="black" size="0.016 0.48 0.016" />
+	<xacro:f_joint name="chassis_to_camera_base_rod" type="fixed" axis_xyz="0 0 0" origin_rpy="0 0 0"
+		origin_xyz="-0.23 0 0.650" parent="chassis" child="camera_base_rod" />
+	<xacro:f_link_box name="lidar_base_rod" origin_rpy="0 0 0" origin_xyz="0 0 0" mass="0.45164"
+		ixx="0.100000005621" ixy="0.100000001310" ixz="0.100000001649" iyy="0.100000004345"
+		iyz="0.100000002360" izz="0.100000003315" material="black" size="0.016 0.48 0.016" />
+	<xacro:f_joint name="chassis_to_lidar_base_rod" type="fixed" axis_xyz="0 0 0" origin_rpy="0 0 0"
+		origin_xyz="0.23 0 -0.15" parent="chassis" child="lidar_base_rod" />
 	<!--Lidar-->
-	<xacro:m_link_cylinder name="rplidar" origin_rpy="0 0 0" origin_xyz="0 0 0" mass="0.10441" ixx="0.1000000042" ixy="0" ixz="0" iyy="0.1000000042" iyz="0" izz="0.1000000040" material="black" filename="package://wheelchair2_description/meshes/rplidar.dae" scale="1 1 1" />
+	<xacro:m_link_cylinder name="rplidar" origin_rpy="0 0 0" origin_xyz="0 0 0" mass="0.10441"
+		ixx="0.1000000042" ixy="0" ixz="0" iyy="0.1000000042" iyz="0" izz="0.1000000040"
+		material="black" filename="package://wheelchair2_description/meshes/rplidar.dae" scale="1 1 1" />
 	<!-- joint between chassis and lidar -->
-	<xacro:f_joint name="chassis_to_rplidar" type="fixed" axis_xyz="0 0 0" origin_rpy="0 0 -1.57" origin_xyz="0.51 0 -0.15" parent="chassis" child="rplidar" />
+	<xacro:f_joint name="chassis_to_rplidar" type="fixed" axis_xyz="0 0 0" origin_rpy="0 0 -1.57"
+		origin_xyz="0.51 0 -0.15" parent="chassis" child="rplidar" />
 	<!--Real_Sense-->
 	<!--D435
 	with tilted angle as in real wheelchair2-->
-	<!--xacro:sensor_d435 parent="base_link">
+	<!--xacro:sensor_d435
+	parent="base_link">
         <origin xyz="-0.23 0 0.860" rpy="0 -0.24 0"/>
       </xacro:sensor_d435-->
 	<!--Labtest
 	3, decent alignment-->
-	<!--xacro:sensor_d455 parent="base_link" name="camera2">
+	<!--xacro:sensor_d455
+	parent="base_link" name="camera2">
         <origin xyz="-0.23 0 0.860" rpy="0 0 0"/>
       </xacro:sensor_d455>
@@ -91,8 +123,10 @@
 		<origin xyz="0.20 -0.24 0.50" rpy="0 -0.01 0" />
 	</xacro:sensor_d435>
-	<!--xacro:sensor_d455 parent="camera_base_rod" name="camera1">
+	<!--xacro:sensor_d455
+	parent="camera_base_rod" name="camera1">
         <origin xyz="0.60 -0.34 -0.50" rpy="0 -0.01 0"/>
       </xacro:sensor_d455-->
-	<!--xacro:sensor_d455 parent="camera2_link" name="camera1">
+	<!--xacro:sensor_d455
+	parent="camera2_link" name="camera1">
         <origin xyz="0.60 -0.34 -0.50" rpy="0 -0.01 0"/>
       </xacro:sensor_d455-->
