Commit message: robot is being spawned, sensor not working

File: wheelchair2_description/urdf/gz_sim/common_properties.urdf.xacro (robot description, xacro)
@@ -1,15 +1,15 @@
-<?xml version="1.0" encoding="UTF-8"?>
+<?xml version="1.0"?>
 <robot name="xacro_properties" xmlns:xacro="http://www.ros.org/wiki/xacro">
-  <material name="grey">
-    <color rgba="0.5 0.5 0.5 1.0"/>
-  </material>
-  <material name="black">
-    <color rgba="0.0 0.0 0.0 1.0"/>
-  </material>
-  <material name="red">
-    <color rgba="1.0 0.0 0.0 1.0"/>
-  </material>
-  <material name="green">
-    <color rgba="0.0 1.0 0.0 1.0"/>
-  </material>
+	<material name="grey">
+		<color rgba="0.5 0.5 0.5 1.0" />
+	</material>
+	<material name="black">
+		<color rgba="0.0 0.0 0.0 1.0" />
+	</material>
+	<material name="red">
+		<color rgba="1.0 0.0 0.0 1.0" />
+	</material>
+	<material name="green">
+		<color rgba="0.0 1.0 0.0 1.0" />
+	</material>
 </robot>

File: wheelchair2_description/urdf/gz_sim/links_joints.urdf.xacro (robot description, xacro)
@@ -9,11 +9,8 @@
 		params="name origin_xyz origin_rpy mass ixx ixy ixz iyy iyz izz filename scale material ">
 		<link name="${name}">
-			<inertial>				<!--Inertial
-				valuse include origin, mass and inertias as per CAD model-->
+			<inertial>
 				<mass value="${mass}" />
 				<origin rpy="${origin_rpy}" xyz="${origin_xyz}" />
 				<inertia ixx="${ixx}" ixy="${ixy}" ixz="${ixz}" iyy="${iyy}" iyz="${iyz}" izz="${izz}" />
-				<!--
-				Taken at the output coordinate system-->
 			</inertial>
 			<collision>				<!-- Collision values include dimensions and origin-->
@@ -23,6 +20,5 @@
 				</geometry>
 			</collision>
-			<visual>				<!-- Visual valuse include origin, material and mesh to make model look similar to
-				real robot-->
+			<visual>
 				<origin rpy="${origin_rpy}" xyz="${origin_xyz}" />
 				<geometry>
@@ -38,11 +34,8 @@
 		params="name origin_xyz origin_rpy mass radius length radius_2 length_2 ixx ixy ixz iyy iyz izz material ">
 		<link name="${name}">
-			<inertial>				<!--Inertial
-				valuse include origin, mass and inertias as per CAD model-->
-				<mass value="${mass}" />
+			<inertial> l <mass value="${mass}" />
 				<origin rpy="${origin_rpy}" xyz="${origin_xyz}" />
-				<inertia ixx="${ixx}" ixy="${ixy}" ixz="${ixz}" iyy="${iyy}" iyz="${iyz}" izz="${izz}" />
-				<!--
-				Taken at the output coordinate system-->
+				<inertia
+					ixx="${ixx}" ixy="${ixy}" ixz="${ixz}" iyy="${iyy}" iyz="${iyz}" izz="${izz}" />
 			</inertial>
 			<collision>				<!-- Collision values include dimensions and origin-->
@@ -52,6 +45,5 @@
 				</geometry>
 			</collision>
-			<visual>				<!-- Visual valuse include origin, material and mesh to make model look similar to
-				real robot-->
+			<visual>
 				<origin rpy="${origin_rpy}" xyz="${origin_xyz}" />
 				<geometry>
@@ -68,11 +60,8 @@
 		params="name origin_xyz origin_rpy size mass ixx ixy ixz iyy iyz izz v_origin_xyz v_origin_rpy filename scale material ">
 		<link name="${name}">
-			<inertial>				<!--Inertial
-				valuse include origin, mass and inertias as per CAD model-->
-				<mass value="${mass}" />
+			<inertial>l <mass value="${mass}" />
 				<origin rpy="${origin_rpy}" xyz="${origin_xyz}" />
-				<inertia ixx="${ixx}" ixy="${ixy}" ixz="${ixz}" iyy="${iyy}" iyz="${iyz}" izz="${izz}" />
-				<!--
-				Taken at the output coordinate system-->
+				<inertia
+					ixx="${ixx}" ixy="${ixy}" ixz="${ixz}" iyy="${iyy}" iyz="${iyz}" izz="${izz}" />
 			</inertial>
 			<collision>				<!-- Collision values include dimensions and origin-->
@@ -82,6 +71,5 @@
 				</geometry>
 			</collision>
-			<visual>				<!-- Visual valuse include origin, material and mesh 0.057 0.083 0.29to make model
-				look similar to real robot-->
+			<visual>
 				<origin rpy="${v_origin_rpy}" xyz="${v_origin_xyz}" />
 				<geometry>
@@ -95,11 +83,8 @@
 		params="name origin_xyz origin_rpy size mass ixx ixy ixz iyy iyz izz material ">
 		<link name="${name}">
-			<inertial>				<!--Inertial
-				valuse include origin, mass and inertias as per CAD model-->
-				<mass value="${mass}" />
+			<inertial> l <mass value="${mass}" />
 				<origin rpy="${origin_rpy}" xyz="${origin_xyz}" />
-				<inertia ixx="${ixx}" ixy="${ixy}" ixz="${ixz}" iyy="${iyy}" iyz="${iyz}" izz="${izz}" />
-				<!--
-				Taken at the output coordinate system-->
+				<inertia
+					ixx="${ixx}" ixy="${ixy}" ixz="${ixz}" iyy="${iyy}" iyz="${iyz}" izz="${izz}" />
 			</inertial>
 			<collision>				<!-- Collision values include dimensions and origin-->
@@ -109,6 +94,5 @@
 				</geometry>
 			</collision>
-			<visual>				<!-- Visual valuse include origin, material and mesh to make model look similar to
-				real robot-->
+			<visual>
 				<origin rpy="${origin_rpy}" xyz="${origin_xyz}" />
 				<geometry>
@@ -122,9 +106,8 @@
 		params="name origin_xyz origin_rpy radius radius_2 mass ixx ixy ixz iyy iyz izz material">
 		<link name="${name}">
-			<inertial>				<!--Inertial
-				valuse include origin, mass and inertias as per CAD model-->
-				<mass value="${mass}" />
+			<inertial> l <mass value="${mass}" />
 				<origin rpy="${origin_rpy}" xyz="${origin_xyz}" />
-				<inertia ixx="${ixx}" ixy="${ixy}" ixz="${ixz}" iyy="${iyy}" iyz="${iyz}" izz="${izz}" />
+				<inertia
+					ixx="${ixx}" ixy="${ixy}" ixz="${ixz}" iyy="${iyy}" iyz="${iyz}" izz="${izz}" />
 			</inertial>
 			<collision>				<!-- Collision values include dimensions and origin-->
@@ -134,6 +117,5 @@
 				</geometry>
 			</collision>
-			<visual>				<!-- Visual valuse include origin, material and mesh to make model look similar to
-				real robot-->
+			<visual>
 				<origin rpy="${origin_rpy}" xyz="${origin_xyz}" />
 				<geometry>
@@ -158,14 +140,4 @@
 			<child link="${child}" />
 		</joint>
-		<!-- <transmission name="trans_${name}"> -->
-		<!-- 	<type>transmission_interface/SimpleTransmission</type> -->
-		<!-- 	<joint name="${name}"> -->
-		<!-- 		<hardwareInterface>hardware_interface/EffortJointInterface</hardwareInterface> -->
-		<!-- 	</joint> -->
-		<!-- 	<actuator name="motor_${name}"> -->
-		<!-- 		<hardwareInterface>hardware_interface/EffortJointInterface</hardwareInterface> -->
-		<!-- 		<mechanicalReduction>1</mechanicalReduction> -->
-		<!-- 	</actuator> -->
-		<!-- </transmission> -->
 	</xacro:macro>
 	<xacro:macro name="w_joint"
@@ -179,14 +151,4 @@
 			<child link="${child}" />
 		</joint>
-		<!-- <transmission name="trans_${name}"> -->
-		<!-- 	<type>transmission_interface/SimpleTransmission</type> -->
-		<!-- 	<joint name="${name}"> -->
-		<!-- 		<hardwareInterface>hardware_interface/EffortJointInterface</hardwareInterface> -->
-		<!-- 	</joint> -->
-		<!-- 	<actuator name="motor_${name}"> -->
-		<!-- 		<hardwareInterface>hardware_interface/EffortJointInterface</hardwareInterface> -->
-		<!-- 		<mechanicalReduction>1</mechanicalReduction> -->
-		<!-- 	</actuator> -->
-		<!-- </transmission> -->
 	</xacro:macro>
 	<xacro:macro name="m2_joint"

File: wheelchair2_description/urdf/gz_sim/realsense.urdf.xacro (robot description, xacro)
@@ -44,6 +44,4 @@
 					<!-- <box size="${d435_cam_width} ${d435_cam_height} ${d435_cam_depth}"/> -->
 					<mesh filename="file://$(find wheelchair2_description)/meshes/d435.dae" />
-					<!--<mesh
-					filename="file://$(find realsense2_description)/meshes/d435/d435.dae" />-->
 				</geometry>
 				<material name="${name}_aluminum" />
@@ -136,30 +134,4 @@
 				</camera>
 			</sensor>
-			<!-- <sensor name="depth" type="depth"> -->
-			<!-- 	<camera> -->
-			<!-- 		<horizontal_fov>${85.2*0.01745329251994329577}</horizontal_fov> -->
-			<!-- 		<image> -->
-			<!-- 			<width>1280</width> -->
-			<!-- 			<height>720</height> -->
-			<!-- 		</image> -->
-			<!-- 		<clip> -->
-			<!-- 			<near>0.1</near> -->
-			<!-- 			<far>100</far> -->
-			<!-- 		</clip> -->
-			<!-- 		<noise> -->
-			<!-- 			<type>gaussian</type> -->
-			<!-- 			<mean>0.0</mean> -->
-			<!-- 			<stddev>0.100</stddev> -->
-			<!-- 		</noise> -->
-			<!-- 	</camera> -->
-			<!-- 	<always_on>1</always_on> -->
-			<!-- 	<update_rate>90</update_rate> -->
-			<!-- 	<visualize>0</visualize> -->
-			<!-- 	<plugin name="color_controller" filename="libgazebo_ros_camera.so"> -->
-			<!-- 		<camera_name>camera</camera_name> -->
-			<!-- 		<min_depth>0.1</min_depth> -->
-			<!-- 		<max_depth>500</max_depth> -->
-			<!-- 	</plugin> -->
-			<!-- </sensor> -->
 		</gazebo>
 	</xacro:macro>

File: wheelchair2_description/urdf/gz_sim/wheelchair2_camera_lidar.urdf.xacro (robot description, xacro)
@@ -1,3 +1,3 @@
-<?xml version="1.0" encoding="UTF-8"?>
+<?xml version="1.0"?>
 <robot name="wheelchair2"
 	xmlns:xacro="http://www.ros.org/wiki/xacro">
@@ -22,5 +22,4 @@
 			<origin xyz="0 0 0" rpy=" 0 0 0" />
 			<!-- ALL INERTIA VALUES IN KILOGRAM PER SQUARE METER-->
-			<!-- NOTE: z=c x=b y=a -->
 			<inertia ixx="6.47" ixy="-0.12" ixz="-1.17" iyy="8.54" iyz="0.29" izz="8.54" />
 		</inertial>
@@ -49,6 +48,4 @@
 		limit_e="100" limit_v="20" damping="1.0" friction="200000.0" origin_rpy="-1.57 0 0"
 		origin_xyz="-0.22 0.28 -0.285" parent="chassis" child="left_wheel" />
-	<!--  inertia values are added by 0.1 in both left and right wheel to avoid collapsing of model in
-	gazebo-->
 	<!-- joint between chassis and Right Wheel-->
 	<!-- Right Wheel-->
@@ -101,9 +98,3 @@
 		<origin xyz="0.20 -0.24 0.50" rpy="0 -0.01 0" />
 	</xacro:realsense>
-	<!-- Gazebo Plugin-->
-	<!-- <gazebo> -->
-	<!-- 	<plugin name="gazebo_ros2_control" filename="libgazebo_ros2_control.so"> -->
-	<!-- 		<legacyModeNS>true</legacyModeNS> -->
-	<!-- 	</plugin> -->
-	<!-- </gazebo> -->
 </robot>

File: wheelchair2_description/urdf/gz_sim/wheelchair2_camera_lidar_gz.urdf.xacro (robot description, xacro)
@@ -3,18 +3,4 @@
 	xmlns:xacro="http://www.ros.org/wiki/xacro">
 	<gazebo>
-		<!-- 	<plugin name='diff_drive' filename='libgazebo_ros_diff_drive.so'> -->
-		<!-- 		<left_joint>chassis_to_left_wheel</left_joint> -->
-		<!-- 		<right_joint>chassis_to_right_wheel</right_joint> -->
-		<!-- 		<wheel_separation>0.48</wheel_separation> -->
-		<!-- 		<wheel_diameter>0.31</wheel_diameter> -->
-		<!-- 		<max_wheel_torque>40</max_wheel_torque> -->
-		<!-- 		<max_wheel_acceleration>1.0</max_wheel_acceleration> -->
-		<!-- 		<odometry_frame>odom</odometry_frame> -->
-		<!-- 		<robot_base_frame>base_link</robot_base_frame> -->
-		<!-- 		<publish_odom>true</publish_odom> -->
-		<!-- 		<publish_odom_tf>true</publish_odom_tf> -->
-		<!-- 		<publish_wheel_tf>false</publish_wheel_tf> -->
-		<!-- 	</plugin> -->
-		<!-- </gazebo> -->
 		<plugin filename="gz-sim-diff-drive-system" name="gz::sim::systems::DiffDrive">
 			<!-- Remove <ros> tag. -->
@@ -24,10 +10,9 @@
 			<!-- kinematics -->
 			<wheel_separation>0.48</wheel_separation>
-			<wheel_radius>0.155</wheel_radius> <!-- computed from <wheel_diameter> in the original
-			plugin-->
+			<wheel_radius>0.155</wheel_radius>
+			<!-- computed from <wheel_diameter> in the original plugin -->
 			<!-- limits -->
-			<max_linear_acceleration>0.155</max_linear_acceleration> <!-- computed from
-		<max_linear_acceleration> in the original plugin-->
-			<topic>cmd_vel</topic> <!-- from <commant_topic> -->
+			<max_linear_acceleration>0.155</max_linear_acceleration>
+			<topic>cmd_vel</topic>
 			<odom_topic>odom</odom_topic> <!-- from <odometry_topic> -->
 			<frame_id>odom</frame_id> <!-- from <odometry_frame> -->
@@ -37,6 +22,4 @@
 		</plugin>
 	</gazebo>
-	<!--Gazebo
-	related physics values of left wheel joint-->
 	<gazebo reference="chassis_to_left_wheel">
 		<mu1 value="10000.0" />
@@ -51,5 +34,4 @@
 		<minDepth value="0.0001" />
 	</gazebo>
-	<!-- Gazebo related physics values of right wheel joint-->
 	<gazebo reference="chassis_to_right_wheel">
 		<mu1 value="10000.0" />

File: wheelchair2_description/urdf/links_joints.urdf.xacro (robot description, xacro)
@@ -23,6 +23,5 @@
 				</geometry>
 			</collision>
-			<visual>				<!-- Visual valuse include origin, material and mesh to make model look similar to
-				real robot-->
+			<visual>
 				<origin rpy="${origin_rpy}" xyz="${origin_xyz}" />
 				<geometry>

File: wheelchair2_description/urdf/wheelchair2.urdf.xacro (robot description, xacro)
@@ -7,6 +7,8 @@
 	<xacro:include filename="$(find wheelchair2_description)/urdf/wheelchair2_gazebo.urdf.xacro" />
 	<xacro:include filename="$(find wheelchair2_description)/urdf/_d435.urdf.xacro" />
-	<!--xacro:include filename="$(find wheelchair2_description)/urdf/_d455.urdf.xacro" /-->
-	<!--xacro:arg name="use_nominal_extrinsics" default="false"/>
+	<!--xacro:include
+	filename="$(find wheelchair2_description)/urdf/_d455.urdf.xacro" /-->
+	<!--xacro:arg
+	name="use_nominal_extrinsics" default="false"/>
   <xacro:arg name="add_plug" default="false" />
   <xacro:arg name="use_mesh" default="true" /-->
@@ -38,5 +40,6 @@
 			<origin xyz="0 0 0" rpy=" 0 0 3.14" />
 			<geometry>
-				<mesh filename="file://$(find wheelchair2_description)/wheelchair2.dae" scale="0.01 0.01 0.01" />
+				<mesh filename="file://$(find wheelchair2_description)/wheelchair2.dae"
+					scale="0.01 0.01 0.01" />
 			</geometry>
 			<material name="black" />
@@ -45,8 +48,12 @@
 	<!--Left
 	Wheel-->
-	<xacro:m1_link_cylinder name="left_wheel" origin_rpy="0 0 0" origin_xyz="0 0 0.027" mass="0.10441" ixx="0.1000000042" ixy="0" ixz="0" iyy="0.1000000042" iyz="0" izz="0.1000000040" radius="0.155" length="0.06" radius_2="0.0028" length_2="0.005" material="grey" />
+	<xacro:m1_link_cylinder name="left_wheel" origin_rpy="0 0 0" origin_xyz="0 0 0.027" mass="0.10441"
+		ixx="0.1000000042" ixy="0" ixz="0" iyy="0.1000000042" iyz="0" izz="0.1000000040" radius="0.155"
+		length="0.06" radius_2="0.0028" length_2="0.005" material="grey" />
 	<!--joint
 	between chassis and Left wheel-->
-	<xacro:w_joint name="chassis_to_left_wheel" type="continuous" axis_xyz="0 0 1" axis_rpy="0 0 0" limit_e="100" limit_v="20" damping="1.0" friction="200000.0" origin_rpy="-1.57 0 0" origin_xyz="-0.22 0.28 -0.285" parent="chassis" child="left_wheel" />
+	<xacro:w_joint name="chassis_to_left_wheel" type="continuous" axis_xyz="0 0 1" axis_rpy="0 0 0"
+		limit_e="100" limit_v="20" damping="1.0" friction="200000.0" origin_rpy="-1.57 0 0"
+		origin_xyz="-0.22 0.28 -0.285" parent="chassis" child="left_wheel" />
 	<!-- inertia values are added by 0.1 in both left and right wheel to avoid collapsing of model in
 	gazebo-->
@@ -55,24 +62,52 @@
 	<!--Right
 	Wheel-->
-	<xacro:m1_link_cylinder name="right_wheel" origin_rpy="0 0 0" origin_xyz="0 0 0.027" mass="0.10441" ixx="0.1000000042" ixy="0" ixz="0" iyy="0.1000000042" iyz="0" izz="0.1000000040" radius="0.155" length="0.06" radius_2="0.0028" length_2="0.005" material="grey" />
-	<xacro:w_joint name="chassis_to_right_wheel" type="continuous" axis_xyz="0 0 1" axis_rpy="0 0 0" limit_e="100" limit_v="20" damping="1.0" friction="200000.0" origin_rpy="-1.57 0 0" origin_xyz="-0.22 -0.32 -0.285" parent="chassis" child="right_wheel" />
+	<xacro:m1_link_cylinder name="right_wheel" origin_rpy="0 0 0" origin_xyz="0 0 0.027"
+		mass="0.10441" ixx="0.1000000042" ixy="0" ixz="0" iyy="0.1000000042" iyz="0" izz="0.1000000040"
+		radius="0.155" length="0.06" radius_2="0.0028" length_2="0.005" material="grey" />
+	<xacro:w_joint name="chassis_to_right_wheel" type="continuous" axis_xyz="0 0 1" axis_rpy="0 0 0"
+		limit_e="100" limit_v="20" damping="1.0" friction="200000.0" origin_rpy="-1.57 0 0"
+		origin_xyz="-0.22 -0.32 -0.285" parent="chassis" child="right_wheel" />
 	<!--Caster
 	1,2 and there joints with Base Link-->
-	<xacro:m_link_sphere name="caster1" origin_rpy="0 0 0" origin_xyz="0 0 0" mass="0.45164" ixx="0.100000005621" ixy="0.100000001310" ixz="0.100000001649" iyy="0.100000004345" iyz="0.100000002360" izz="0.100000003315" material="black" radius="0.1" radius_2="0.001" />
-	<xacro:f_joint name="chassis_to_caster1" type="fixed" axis_xyz="0 0 0" origin_rpy="0 0 0" origin_xyz="0.2 -0.25 -0.33" parent="chassis" child="caster1" />
-	<xacro:m_link_sphere name="caster2" origin_rpy="0 0 0" origin_xyz="0 0 0" mass="0.45164" ixx="0.100000005621" ixy="0.100000001310" ixz="0.100000001649" iyy="0.100000004345" iyz="0.100000002360" izz="0.100000003315" material="black" radius="0.1" radius_2="0.001" />
-	<xacro:f_joint name="chassis_to_caster2" type="fixed" axis_xyz="0 0 0" origin_rpy="0 0 0" origin_xyz="0.2 0.25 -0.33" parent="chassis" child="caster2" />
-	<xacro:f_link_box name="rod1" origin_rpy="0 0 0" origin_xyz="0 0 0" mass="0.45164" ixx="0.100000005621" ixy="0.100000001310" ixz="0.100000001649" iyy="0.100000004345" iyz="0.100000002360" izz="0.100000003315" material="black" size="0.016 0.016 0.6" />
-	<xacro:f_joint name="chassis_to_rod1" type="fixed" axis_xyz="0 0 0" origin_rpy="0 0 0" origin_xyz="-0.23 0.24 0.65" parent="chassis" child="rod1" />
-	<xacro:f_link_box name="rod2" origin_rpy="0 0 0" origin_xyz="0 0 0" mass="0.45164" ixx="0.100000005621" ixy="0.100000001310" ixz="0.100000001649" iyy="0.100000004345" iyz="0.100000002360" izz="0.100000003315" material="black" size="0.016 0.016 0.6" />
-	<xacro:f_joint name="chassis_to_rod2" type="fixed" axis_xyz="0 0 0" origin_rpy="0 0 0" origin_xyz="-0.23 -0.24 0.65" parent="chassis" child="rod2" />
-	<xacro:f_link_box name="camera_base_rod" origin_rpy="0 0 0" origin_xyz="0 0 0" mass="0.45164" ixx="0.100000005621" ixy="0.100000001310" ixz="0.100000001649" iyy="0.100000004345" iyz="0.100000002360" izz="0.100000003315" material="black" size="0.016 0.48 0.016" />
-	<xacro:f_joint name="chassis_to_camera_base_rod" type="fixed" axis_xyz="0 0 0" origin_rpy="0 0 0" origin_xyz="-0.23 0 0.650" parent="chassis" child="camera_base_rod" />
-	<!--xacro:f_link_box name="lidar_base_rod" origin_rpy="0 0 0" origin_xyz="0 0 0" mass="0.45164" ixx="0.100000005621" ixy="0.100000001310" ixz="0.100000001649" iyy="0.100000004345" iyz="0.100000002360" izz="0.100000003315" material="black" size="0.016 0.48 0.016"/>
-    <xacro:f_joint name="chassis_to_lidar_base_rod" type="fixed" axis_xyz="0 0 0" origin_rpy="0 0 0" origin_xyz="0.23 0 -0.15" parent="chassis" child="lidar_base_rod" /-->
+	<xacro:m_link_sphere name="caster1" origin_rpy="0 0 0" origin_xyz="0 0 0" mass="0.45164"
+		ixx="0.100000005621" ixy="0.100000001310" ixz="0.100000001649" iyy="0.100000004345"
+		iyz="0.100000002360" izz="0.100000003315" material="black" radius="0.1" radius_2="0.001" />
+	<xacro:f_joint name="chassis_to_caster1" type="fixed" axis_xyz="0 0 0" origin_rpy="0 0 0"
+		origin_xyz="0.2 -0.25 -0.33" parent="chassis" child="caster1" />
+	<xacro:m_link_sphere name="caster2" origin_rpy="0 0 0" origin_xyz="0 0 0" mass="0.45164"
+		ixx="0.100000005621" ixy="0.100000001310" ixz="0.100000001649" iyy="0.100000004345"
+		iyz="0.100000002360" izz="0.100000003315" material="black" radius="0.1" radius_2="0.001" />
+	<xacro:f_joint name="chassis_to_caster2" type="fixed" axis_xyz="0 0 0" origin_rpy="0 0 0"
+		origin_xyz="0.2 0.25 -0.33" parent="chassis" child="caster2" />
+	<xacro:f_link_box name="rod1" origin_rpy="0 0 0" origin_xyz="0 0 0" mass="0.45164"
+		ixx="0.100000005621" ixy="0.100000001310" ixz="0.100000001649" iyy="0.100000004345"
+		iyz="0.100000002360" izz="0.100000003315" material="black" size="0.016 0.016 0.6" />
+	<xacro:f_joint name="chassis_to_rod1" type="fixed" axis_xyz="0 0 0" origin_rpy="0 0 0"
+		origin_xyz="-0.23 0.24 0.65" parent="chassis" child="rod1" />
+	<xacro:f_link_box name="rod2" origin_rpy="0 0 0" origin_xyz="0 0 0" mass="0.45164"
+		ixx="0.100000005621" ixy="0.100000001310" ixz="0.100000001649" iyy="0.100000004345"
+		iyz="0.100000002360" izz="0.100000003315" material="black" size="0.016 0.016 0.6" />
+	<xacro:f_joint name="chassis_to_rod2" type="fixed" axis_xyz="0 0 0" origin_rpy="0 0 0"
+		origin_xyz="-0.23 -0.24 0.65" parent="chassis" child="rod2" />
+	<xacro:f_link_box name="camera_base_rod" origin_rpy="0 0 0" origin_xyz="0 0 0" mass="0.45164"
+		ixx="0.100000005621" ixy="0.100000001310" ixz="0.100000001649" iyy="0.100000004345"
+		iyz="0.100000002360" izz="0.100000003315" material="black" size="0.016 0.48 0.016" />
+	<xacro:f_joint name="chassis_to_camera_base_rod" type="fixed" axis_xyz="0 0 0" origin_rpy="0 0 0"
+		origin_xyz="-0.23 0 0.650" parent="chassis" child="camera_base_rod" />
+	<!--xacro:f_link_box
+	name="lidar_base_rod" origin_rpy="0 0 0" origin_xyz="0 0 0" mass="0.45164" ixx="0.100000005621"
+	ixy="0.100000001310" ixz="0.100000001649" iyy="0.100000004345" iyz="0.100000002360"
+	izz="0.100000003315" material="black" size="0.016 0.48 0.016"/>
+    <xacro:f_joint name="chassis_to_lidar_base_rod" type="fixed" axis_xyz="0 0 0" origin_rpy="0 0 0"
+	origin_xyz="0.23 0 -0.15" parent="chassis" child="lidar_base_rod" /-->
 	<!--Lidar-->
-	<!--xacro:m_link_cylinder name="rplidar" origin_rpy="0 0 0" origin_xyz="0 0 0" mass="0.10441" ixx="0.1000000042" ixy="0" ixz="0" iyy="0.1000000042" iyz="0" izz="0.1000000040" material="black" filename="package://wheelchair2_description/meshes/rplidar.dae" scale="1 1 1"/-->
+	<!--xacro:m_link_cylinder
+	name="rplidar" origin_rpy="0 0 0" origin_xyz="0 0 0" mass="0.10441" ixx="0.1000000042" ixy="0"
+	ixz="0" iyy="0.1000000042" iyz="0" izz="0.1000000040" material="black"
+	filename="package://wheelchair2_description/meshes/rplidar.dae" scale="1 1 1"/-->
 	<!-- joint between chassis and lidar -->
-	<!--xacro:f_joint name="chassis_to_rplidar" type="fixed" axis_xyz="0 0 0" origin_rpy="0 0 3.14" origin_xyz="0.23 0 -0.15" parent="chassis" child="rplidar" /-->
+	<!--xacro:f_joint
+	name="chassis_to_rplidar" type="fixed" axis_xyz="0 0 0" origin_rpy="0 0 3.14" origin_xyz="0.23 0
+	-0.15" parent="chassis" child="rplidar" /-->
 	<!--Real_Sense-->
 	<xacro:sensor_d435 parent="base_link" name="camera2" topics_ns="camera2" pointcloud="true">
@@ -82,6 +117,4 @@
 		<origin xyz="0.60 -0.34 -0.50" rpy="0 -0.01 0" />
 	</xacro:sensor_d435>
-	<!--Gazebo
-	Plugin-->
 	<gazebo>
 		<plugin name="gazebo_ros_control" filename="libgazebo_ros_control.so">

File: wheelchair2_description/urdf/wheelchair2_livox.urdf.xacro (robot description, xacro)
@@ -106,5 +106,4 @@
 	</xacro:mid360>
 	<xacro:kangaroo_x2_driver name="kangaroo_ros2_control" prefix="" is_sim="$(arg is_sim)"></xacro:kangaroo_x2_driver>
-	<!-- Gazebo Plugin-->
 	<xacro:if value="$(arg is_sim)">
 		<gazebo>
