Commit message: Added the wheelchair model, as now gazebo uses GPU

File: wheelchair2_gazebo/urdf/wheelchair2_camera_livox_gazebo.urdf.xacro (robot description, xacro)
@@ -36,5 +36,5 @@
             <material name="black" />
         </collision>
-        <!-- <visual>
+        <visual>
             <origin xyz="0 0 0" rpy=" 0 0 3.14" />
             <geometry>
@@ -42,5 +42,5 @@
             </geometry>
             <material name="black" />
-        </visual> -->
+        </visual>
     </link>
     <!-- Left Wheel-->
