Commit message: added use_sim_time arg

File: wheelchair2_gazebo/urdf/realsense.urdf.xacro (robot description, xacro)
@@ -2,5 +2,5 @@
 <robot name="realsense"
 	xmlns:xacro="http://ros.org/wiki/xacro">
-	<xacro:macro name="realsense" params="name:=camera topics_ns:=camera pointcloud:=false parent *origin">
+	<xacro:macro name="realsense" params="name:=camera topics_ns:=camera pointcloud:=false parent *origin use_sim_time">
 		<xacro:property name="M_PI" value="3.1415926535897931" />
 		<!-- The following values are approximate, and the camera node
@@ -110,30 +110,30 @@
 		</joint>
 		<link name="${name}_color_optical_frame" />
-		<!-- Realsense Gazebo Plugin -->
-		<gazebo reference="camera_link">
-			<material>Gazebo/Red</material>
-			<sensor name="camera" type="depth">
-				<pose> 0 0 0 0 0 0 </pose>
-				<visualize>true</visualize>
-				<update_rate>10</update_rate>
-				<camera>
-					<horizontal_fov>1.089</horizontal_fov>
-					<image>
-						<format>B8G8R8</format>
-						<width>640</width>
-						<height>480</height>
-					</image>
-					<clip>
-						<near>0.05</near>
-						<far>8.0</far>
-					</clip>
-				</camera>
-				<plugin name="camera_controller" filename="libgazebo_ros_camera.so">
-					<frame_name>camera_link_optical</frame_name>
-					<min_depth>0.1</min_depth>
-					<max_depth>100.0</max_depth>
-				</plugin>
-			</sensor>
-		</gazebo>
+		<xacro:if value="${use_sim_time}">
+			<!-- Realsense Gazebo Plugin -->
+			<gazebo reference="camera_link">
+				<material>Gazebo/Black</material>
+				<sensor name="camera" type="camera">
+					<pose> 0 0 0 0 0 0 </pose>
+					<visualize>true</visualize>
+					<update_rate>10</update_rate>
+					<camera>
+						<camera_info_topic>camera/camera_info</camera_info_topic>
+						<horizontal_fov>1.089</horizontal_fov>
+						<image>
+							<format>R8G8B8</format>
+							<width>640</width>
+							<height>480</height>
+						</image>
+						<clip>
+							<near>0.05</near>
+							<far>8.0</far>
+						</clip>
+					</camera>
+					<topic>camera/image_raw</topic>
+					<gz_frame_id>camera_link</gz_frame_id>
+				</sensor>
+			</gazebo>
+		</xacro:if>
 	</xacro:macro>
 </robot>

File: wheelchair2_gazebo/urdf/wheelchair2_camera_livox_gazebo.urdf.xacro (robot description, xacro)
@@ -2,17 +2,12 @@
 <robot name="wheelchair2"
     xmlns:xacro="http://www.ros.org/wiki/xacro">
-    <!-- Include Files-->
-    <xacro:include filename="$(find wheelchair2_description)/urdf/links_joints.urdf.xacro" />
-    <!-- <xacro:include filename="$(find wheelchair2_description)/urdf/kangaroo_ros2_control.urdf.xacro" /> -->
-    <xacro:include filename="$(find wheelchair2_gazebo)/urdf/realsense.urdf.xacro" />
-    <xacro:include filename="$(find wheelchair2_description)/urdf/mid360.xacro" />
-    <xacro:include filename="$(find wheelchair2_gazebo)/urdf/gz_ros2_control.urdf.xacro" />
-    <xacro:include filename="$(find wheelchair2_gazebo)/urdf/wheelchair2_gazebo.urdf.xacro" />
-    <xacro:include filename="$(find wheelchair2_gazebo)/urdf/livox.urdf.xacro" />
+    <xacro:arg name="use_sim_time" default="false" />
     <xacro:arg name="use_nominal_extrinsics" default="false" />
     <xacro:arg name="add_plug" default="false" />
     <xacro:arg name="use_mesh" default="true" />
+    <xacro:include filename="$(find wheelchair2_description)/urdf/links_joints.urdf.xacro" />
+    <xacro:include filename="$(find wheelchair2_description)/urdf/kangaroo_ros2_control.urdf.xacro" />
+    <xacro:include filename="$(find wheelchair2_gazebo)/urdf/realsense.urdf.xacro" />
     <link name="base_footprint" />
-    <!-- Add Base Footprint -->
     <joint name="base_footprint_joint" type="fixed">
         <parent link="base_footprint" />
@@ -20,26 +15,24 @@
         <origin xyz="0.22 0 0.2" rpy="0 0 0" />
     </joint>
-    <link name='base_link'>
+    <link name="base_link">
         <pose>0 0 0.1 0 0 0</pose>
         <inertial>
-            <!-- ALL MASSES IN KILOGRAM-->
-            <mass value="8.96" />
-            <origin xyz="0 0 0" rpy=" 0 0 0" />
-            <!-- ALL INERTIA VALUES IN KILOGRAM PER SQUARE METER-->
-            <inertia ixx="2.83" ixy="-0.12" ixz="-1.17" iyy="3.47" iyz="0.29" izz="0.73" />
+            <mass value="8.96"/>
+            <origin xyz="0 0 0" rpy="0 0 0"/>
+            <inertia ixx="2.83" ixy="-0.12" ixz="-1.17" iyy="3.47" iyz="0.29" izz="0.73"/>
         </inertial>
         <collision>
-            <origin xyz="0.1 0 0" rpy=" 0 0 0" />
+            <origin xyz="0.1 0 0" rpy="0 0 0"/>
             <geometry>
-                <box size="0.75 0.60 0.60" />
+                <box size="0.75 0.60 0.60"/>
             </geometry>
-            <material name="black" />
+            <material name="black"/>
         </collision>
         <visual>
-            <origin xyz="0 0 0" rpy=" 0 0 3.14" />
+            <origin xyz="0 0 0" rpy="0 0 3.14"/>
             <geometry>
-                <mesh filename="file://$(find wheelchair2_description)/meshes/wheelchair2.dae" scale="0.01 0.01 0.01" />
+                <mesh filename="file://$(find wheelchair2_description)/meshes/wheelchair2.dae" scale="0.01 0.01 0.01"/>
             </geometry>
-            <material name="black" />
+            <material name="black"/>
         </visual>
     </link>
@@ -65,16 +58,33 @@
     <xacro:f_link_box name="camera_base_rod" origin_rpy="0 0 0" origin_xyz="0 0 0" mass="0.45164" ixx="0.100000005621" ixy="0.100000001310" ixz="0.100000001649" iyy="0.100000004345" iyz="0.100000002360" izz="0.100000003315" material="black" size="0.016 0.48 0.016" />
     <xacro:f_joint name="base_link_to_camera_base_rod" type="fixed" axis_xyz="0 0 0" origin_rpy="0 0 0" origin_xyz="-0.23 0 0.650" parent="base_link" child="camera_base_rod" />
-    <!-- <xacro:f_link_box name="lidar_base_rod" origin_rpy="0 0 0" origin_xyz="0 0 0" mass="0.45164" ixx="0.100000005621" ixy="0.100000001310" ixz="0.100000001649" iyy="0.100000004345" iyz="0.100000002360" izz="0.100000003315" material="black" size="0.016 0.48 0.016" /> -->
-    <!-- <xacro:f_joint name="base_link_to_lidar_base_rod" type="fixed" axis_xyz="0 0 0" origin_rpy="0 0 0" origin_xyz="0.23 0 -0.15" parent="base_link" child="lidar_base_rod" /> -->
-    <!--Lidar-->
-    <!-- <xacro:m_link_cylinder name="laser_frame" origin_rpy="0 0 0" origin_xyz="0 0 0" mass="0.10441" ixx="0.1000000042" ixy="0" ixz="0" iyy="0.1000000042" iyz="0" izz="0.1000000040" material="black" filename="file://$(find wheelchair2_description)/meshes/rplidar.dae" scale="1 1 1" /> -->
-    <!-- joint between base_link and lidar -->
-    <!-- <xacro:f_joint name="base_link_to_laser" type="fixed" axis_xyz="0 0 0" origin_rpy="0 0 0" origin_xyz="0.53 0 -0.15" parent="base_link" child="laser_frame" /> -->
-    <xacro:realsense parent="base_link" name="camera_link">
-        <origin xyz="0 0 1.25" rpy="0 0 0" />
+    <!-- 3D Printed Mount -->
+    <link name="camera_mount_link"/>
+    <joint name="base_to_camera_mount" type="fixed">
+        <origin xyz="-0.19159 0 1.2144" rpy="0 0 0" />
+        <parent link="base_link"/>
+        <child link="camera_mount_link"/>
+    </joint>
+    <!-- Realsense mounted to 3D printed mount -->
+    <xacro:realsense name="camera" parent="camera_mount_link" use_sim_time="$(arg use_sim_time)">
+        <origin xyz="0 0 0" rpy="0 0 0"/>
     </xacro:realsense>
-    <!-- MID-360 -->
-    <xacro:mid360 name="livox_frame" parent="base_link" topic="mid360">
-        <origin xyz="-0.05 0 -0.05" rpy="3.14 0 0" />
-    </xacro:mid360>
+    <!-- livox link w.r.t camera_link -->
+    <link name="livox_frame"/>
+    <joint name="camera_link_to_livox_frame" type="fixed">
+        <origin xyz="-0.064156 0 -0.064846" rpy="-3.1416 -0.0131 0" />
+        <parent link="camera_link" />
+        <child link="livox_frame" />
+        <axis xyz="0 0 0" />
+    </joint>
+    <xacro:kangaroo_x2_driver name="kangaroo_ros2_control" prefix="" use_sim_time="$(arg use_sim_time)"></xacro:kangaroo_x2_driver>
+    <!-- Gazebo Plugin-->
+    <xacro:if value="$(arg use_sim_time)">
+        <gazebo>
+            <plugin name="gz_ros2_control::GazeboSimROS2ControlPlugin" filename="libgz_ros2_control-system.so">
+                <parameters>$(find wheelchair2_bringup)/config/wheelchair2_controllers.yaml</parameters>
+            </plugin>
+        </gazebo>
+        <xacro:include filename="$(find wheelchair2_gazebo)/urdf/wheelchair2_gazebo.urdf.xacro" />
+        <xacro:include filename="$(find wheelchair2_gazebo)/urdf/livox.urdf.xacro" />
+    </xacro:if>
 </robot>
