Commit message: 3dbbs + gicp submodule tested

File: install/wheelchair2_description/share/wheelchair2_description/urdf/common_properties.urdf.xacro (robot description, xacro)
@@ -1,15 +1 @@
-<?xml version="1.0" encoding="UTF-8"?>
-<robot name="xacro_properties" xmlns:xacro="http://www.ros.org/wiki/xacro">
-  <material name="grey">
-    <color rgba="0.5 0.5 0.5 1.0"/>
-  </material>
-  <material name="black">
-    <color rgba="0.0 0.0 0.0 1.0"/>
-  </material>
-  <material name="red">
-    <color rgba="1.0 0.0 0.0 1.0"/>
-  </material>
-  <material name="green">
-    <color rgba="0.0 1.0 0.0 1.0"/>
-  </material>
-</robot>
+/home/container_user/wheelchair2/src/build/wheelchair2_description/urdf/common_properties.urdf.xacro

File: install/wheelchair2_description/share/wheelchair2_description/urdf/kangaroo_ros2_control.urdf.xacro (robot description, xacro)
@@ -1,40 +1 @@
-<?xml version="1.0" encoding="UTF-8"?>
-<robot xmlns:xacro="http://www.ros.org/wiki/xacro">
-	<xacro:macro name="kangaroo_x2_driver" params="name prefix use_sim_time">
-		<ros2_control name="${name}" type="system">
-			<hardware>
-				<xacro:if value="${use_sim_time}">
-					<plugin>gz_ros2_control/GazeboSimSystem</plugin>
-				</xacro:if>
-				<xacro:unless value="${use_sim_time}">
-					<plugin>wheelchair2_kangaroo_x2_driver/Kangaroo</plugin>
-					<!-- <plugin>mock_components/GenericSystem</plugin> -->
-					<param name="left_wheel_name">base_link_to_left_wheel</param>
-					<param name="right_wheel_name">base_link_to_right_wheel</param>
-					<param name="wheel_diameter">0.32</param>
-					<param name="wheel_center_distance">0.55</param>
-					<param name="encoder_lines_per_revolution">65536</param>
-					<param name="hz">50</param>
-					<param name="port">/dev/ttyACM0</param>
-					<param name="mixed_mode">true</param>
-				</xacro:unless>
-			</hardware>
-			<joint name="${prefix}base_link_to_left_wheel">
-				<command_interface name="velocity">
-					<param name="min">-1</param>
-					<param name="max">1</param>
-				</command_interface>
-				<state_interface name="position"/>
-				<state_interface name="velocity"/>
-			</joint>
-			<joint name="${prefix}base_link_to_right_wheel">
-				<command_interface name="velocity">
-					<param name="min">-1</param>
-					<param name="max">1</param>
-				</command_interface>
-				<state_interface name="position"/>
-				<state_interface name="velocity"/>
-			</joint>
-		</ros2_control>
-	</xacro:macro>
-</robot>
+/home/container_user/wheelchair2/src/build/wheelchair2_description/urdf/kangaroo_ros2_control.urdf.xacro

File: install/wheelchair2_description/share/wheelchair2_description/urdf/links_joints.urdf.xacro (robot description, xacro)
@@ -1,224 +1 @@
-<?xml version="1.0"?>
-<robot xmlns:xacro="http://www.ros.org/wiki/xacro">
-	<!--Include
-	Files-->
-	<xacro:include filename="$(find wheelchair2_description)/urdf/common_properties.urdf.xacro" />
-	<!--macro
-	for cylinder shaped links(r,lwheels and lidar)-->
-	<xacro:macro name="m_link_cylinder"
-		params="name origin_xyz origin_rpy mass ixx ixy ixz iyy iyz izz filename scale material ">
-		<link name="${name}">
-			<inertial>				<!--Inertial
-				valuse include origin, mass and inertias as per CAD model-->
-				<mass value="${mass}" />
-				<origin rpy="${origin_rpy}" xyz="${origin_xyz}" />
-				<inertia ixx="${ixx}" ixy="${ixy}" ixz="${ixz}" iyy="${iyy}" iyz="${iyz}" izz="${izz}" />
-				<!--
-				Taken at the output coordinate system-->
-			</inertial>
-			<collision>				<!-- Collision values include dimensions and origin-->
-				<origin rpy="${origin_rpy}" xyz="${origin_xyz}" />
-				<geometry>
-					<mesh filename="${filename}" scale="${scale}" />
-				</geometry>
-			</collision>
-			<visual>
-				<origin rpy="${origin_rpy}" xyz="${origin_xyz}" />
-				<geometry>
-					<mesh filename="${filename}" scale="${scale}" />
-				</geometry>
-				<material name="${material}" />
-			</visual>
-		</link>
-	</xacro:macro>
-	<!--macro
-	for cylinder shaped links(r,lwheels and lidar)-->
-	<xacro:macro name="m1_link_cylinder"
-		params="name origin_xyz origin_rpy mass radius length radius_2 length_2 ixx ixy ixz iyy iyz izz material ">
-		<link name="${name}">
-			<inertial>				<!--Inertial
-				valuse include origin, mass and inertias as per CAD model-->
-				<mass value="${mass}" />
-				<origin rpy="${origin_rpy}" xyz="${origin_xyz}" />
-				<inertia ixx="${ixx}" ixy="${ixy}" ixz="${ixz}" iyy="${iyy}" iyz="${iyz}" izz="${izz}" />
-				<!--
-				Taken at the output coordinate system-->
-			</inertial>
-			<collision>				<!-- Collision values include dimensions and origin-->
-				<origin rpy="${origin_rpy}" xyz="${origin_xyz}" />
-				<geometry>
-					<cylinder radius="${radius}" length="${length}" />
-				</geometry>
-			</collision>
-			<visual>				<!-- Visual valuse include origin, material and mesh to make model look similar to
-				real robot-->
-				<origin rpy="${origin_rpy}" xyz="${origin_xyz}" />
-				<geometry>
-					<cylinder radius="${radius_2}" length="${length_2}" />
-					<!-- <mesh filename="${filename}" scale="${scale}"/> -->
-				</geometry>
-				<material name="${material}" />
-			</visual>
-		</link>
-	</xacro:macro>
-	<!--macro
-	for box shaped links(r,lwheels and lidar)-->
-	<xacro:macro name="m_link_box"
-		params="name origin_xyz origin_rpy size mass ixx ixy ixz iyy iyz izz v_origin_xyz v_origin_rpy filename scale material ">
-		<link name="${name}">
-			<inertial>				<!--Inertial
-				valuse include origin, mass and inertias as per CAD model-->
-				<mass value="${mass}" />
-				<origin rpy="${origin_rpy}" xyz="${origin_xyz}" />
-				<inertia ixx="${ixx}" ixy="${ixy}" ixz="${ixz}" iyy="${iyy}" iyz="${iyz}" izz="${izz}" />
-				<!--
-				Taken at the output coordinate system-->
-			</inertial>
-			<collision>				<!-- Collision values include dimensions and origin-->
-				<origin rpy="${origin_rpy}" xyz="${origin_xyz}" />
-				<geometry>
-					<box size="${size}" />
-				</geometry>
-			</collision>
-			<visual>				<!-- Visual valuse include origin, material and mesh 0.057 0.083 0.29to make model
-				look similar to real robot-->
-				<origin rpy="${v_origin_rpy}" xyz="${v_origin_xyz}" />
-				<geometry>
-					<!-- <mesh filename="${filename}" scale="${scale}"/> -->
-				</geometry>
-				<material name="${material}" />
-			</visual>
-		</link>
-	</xacro:macro>
-	<xacro:macro name="f_link_box"
-		params="name origin_xyz origin_rpy size mass ixx ixy ixz iyy iyz izz material ">
-		<link name="${name}">
-			<inertial>				<!--Inertial
-				valuse include origin, mass and inertias as per CAD model-->
-				<mass value="${mass}" />
-				<origin rpy="${origin_rpy}" xyz="${origin_xyz}" />
-				<inertia ixx="${ixx}" ixy="${ixy}" ixz="${ixz}" iyy="${iyy}" iyz="${iyz}" izz="${izz}" />
-				<!--
-				Taken at the output coordinate system-->
-			</inertial>
-			<collision>				<!-- Collision values include dimensions and origin-->
-				<origin rpy="${origin_rpy}" xyz="${origin_xyz}" />
-				<geometry>
-					<box size="${size}" />
-				</geometry>
-			</collision>
-			<visual>				<!-- Visual valuse include origin, material and mesh to make model look similar to
-				real robot-->
-				<origin rpy="${origin_rpy}" xyz="${origin_xyz}" />
-				<geometry>
-					<box size="${size}" />
-				</geometry>
-				<material name="${material}" />
-			</visual>
-		</link>
-	</xacro:macro>
-	<xacro:macro name="m_link_sphere"
-		params="name origin_xyz origin_rpy radius radius_2 mass ixx ixy ixz iyy iyz izz material">
-		<link name="${name}">
-			<inertial>				<!--Inertial
-				valuse include origin, mass and inertias as per CAD model-->
-				<mass value="${mass}" />
-				<origin rpy="${origin_rpy}" xyz="${origin_xyz}" />
-				<inertia ixx="${ixx}" ixy="${ixy}" ixz="${ixz}" iyy="${iyy}" iyz="${iyz}" izz="${izz}" />
-			</inertial>
-			<collision>				<!-- Collision values include dimensions and origin-->
-				<origin rpy="${origin_rpy}" xyz="${origin_xyz}" />
-				<geometry>
-					<sphere radius="${radius}" />
-				</geometry>
-			</collision>
-			<visual>				<!-- Visual valuse include origin, material and mesh to make model look similar to
-				real robot-->
-				<origin rpy="${origin_rpy}" xyz="${origin_xyz}" />
-				<geometry>
-					<sphere radius="${radius_2}" />
-					<!-- <mesh filename="${filename}" scale="${scale}"/> -->
-				</geometry>
-				<material name="${material}" />
-			</visual>
-		</link>
-	</xacro:macro>
-	<!-- macro of moving joints like l,rwheels-->
-	<!-- It includes parent link, child link, limits, axis, origin, dynamics and transmission of the
-	robot-->
-	<xacro:macro name="m_joint"
-		params="name type axis_xyz axis_rpy origin_rpy origin_xyz parent limit_e limit_v lower upper child damping friction ">
-		<joint name="${name}" type="${type}">
-			<axis xyz="${axis_xyz}" rpy="${axis_rpy}" />
-			<limit effort="${limit_e}" velocity="${limit_v}" lower="${lower}" upper="${upper}" />
-			<origin rpy="${origin_rpy}" xyz="${origin_xyz}" />
-			<dynamics damping="${damping}" friction="${friction}" />
-			<parent link="${parent}" />
-			<child link="${child}" />
-		</joint>
-		<!-- <transmission name="trans_${name}"> -->
-		<!-- 	<type>transmission_interface/SimpleTransmission</type> -->
-		<!-- 	<joint name="${name}"> -->
-		<!-- 		<hardwareInterface>hardware_interface/EffortJointInterface</hardwareInterface> -->
-		<!-- 	</joint> -->
-		<!-- 	<actuator name="motor_${name}"> -->
-		<!-- 		<hardwareInterface>hardware_interface/EffortJointInterface</hardwareInterface> -->
-		<!-- 		<mechanicalReduction>1</mechanicalReduction> -->
-		<!-- 	</actuator> -->
-		<!-- </transmission> -->
-	</xacro:macro>
-	<xacro:macro name="w_joint"
-		params="name type axis_xyz axis_rpy origin_rpy origin_xyz parent limit_e limit_v child damping friction ">
-		<joint name="${name}" type="${type}">
-			<axis xyz="${axis_xyz}" rpy="${axis_rpy}" />
-			<limit effort="${limit_e}" velocity="${limit_v}" />
-			<origin rpy="${origin_rpy}" xyz="${origin_xyz}" />
-			<dynamics damping="${damping}" friction="${friction}" />
-			<parent link="${parent}" />
-			<child link="${child}" />
-		</joint>
-		<!-- <transmission name="trans_${name}"> -->
-		<!-- 	<type>transmission_interface/SimpleTransmission</type> -->
-		<!-- 	<joint name="${name}"> -->
-		<!-- 		<hardwareInterface>hardware_interface/EffortJointInterface</hardwareInterface> -->
-		<!-- 	</joint> -->
-		<!-- 	<actuator name="motor_${name}"> -->
-		<!-- 		<hardwareInterface>hardware_interface/EffortJointInterface</hardwareInterface> -->
-		<!-- 		<mechanicalReduction>1</mechanicalReduction> -->
-		<!-- 	</actuator> -->
-		<!-- </transmission> -->
-	</xacro:macro>
-	<xacro:macro name="m2_joint"
-		params="name type axis_xyz axis_rpy origin_rpy origin_xyz parent limit_e limit_v lower upper child damping friction ">
-		<joint name="${name}" type="${type}">
-			<axis xyz="${axis_xyz}" rpy="${axis_rpy}" />
-			<limit effort="${limit_e}" velocity="${limit_v}" lower="${lower}" upper="${upper}" />
-			<origin rpy="${origin_rpy}" xyz="${origin_xyz}" />
-			<dynamics damping="${damping}" friction="${friction}" />
-			<parent link="${parent}" />
-			<child link="${child}" />
-		</joint>
-	</xacro:macro>
-	<xacro:macro name="mimic_joint"
-		params="name type axis_xyz axis_rpy origin_rpy origin_xyz parent joint multiplier offset limit_e limit_v lower upper child damping friction ">
-		<joint name="${name}" type="${type}">
-			<axis xyz="${axis_xyz}" rpy="${axis_rpy}" />
-			<limit effort="${limit_e}" velocity="${limit_v}" lower="${lower}" upper="${upper}" />
-			<origin rpy="${origin_rpy}" xyz="${origin_xyz}" />
-			<dynamics damping="${damping}" friction="${friction}" />
-			<parent link="${parent}" />
-			<child link="${child}" />
-			<mimic joint="${joint}" multiplier="${multiplier}" offset="${offset}" />
-		</joint>
-	</xacro:macro>
-	<!-- macro of fixed joints like casters and rplidar-->
-	<!-- It includes parent link, child link, axis and origin of the robot-->
-	<xacro:macro name="f_joint" params="name type axis_xyz origin_rpy origin_xyz parent child">
-		<joint name="${name}" type="${type}">
-			<axis xyz="${axis_xyz}" />
-			<origin rpy="${origin_rpy}" xyz="${origin_xyz}" />
-			<parent link="${parent}" />
-			<child link="${child}" />
-		</joint>
-	</xacro:macro>
-</robot>
+/home/container_user/wheelchair2/src/build/wheelchair2_description/urdf/links_joints.urdf.xacro

File: install/wheelchair2_description/share/wheelchair2_description/urdf/realsense.urdf.xacro (robot description, xacro)
@@ -1,144 +1 @@
-<?xml version="1.0"?>
-<robot name="realsense"
-	xmlns:xacro="http://ros.org/wiki/xacro">
-	<xacro:macro name="realsense" params="name:=camera topics_ns:=camera pointcloud:=false parent *origin use_sim_time">
-		<xacro:property name="M_PI" value="3.1415926535897931" />
-		<!-- The following values are approximate, and the camera node
-     publishing TF values with actual calibrated camera extrinsic values -->
-		<xacro:property name="d435_cam_depth_to_left_ir_offset" value="0.0" />
-		<xacro:property name="d435_cam_depth_to_right_ir_offset" value="-0.050" />
-		<xacro:property name="d435_cam_depth_to_color_offset" value="0.015" />
-		<!-- The following values model the aluminum peripherial case for the
-  	D435 camera, with the camera joint represented by the actual
-  	peripherial camera tripod mount -->
-		<xacro:property name="d435_cam_width" value="0.090" />
-		<xacro:property name="d435_cam_height" value="0.025" />
-		<xacro:property name="d435_cam_depth" value="0.02505" />
-		<xacro:property name="d435_cam_mount_from_center_offset" value="0.0149" />
-		<!-- The following offset is relative the the physical D435 camera peripherial
-  	camera tripod mount -->
-		<xacro:property name="d435_cam_depth_px" value="${d435_cam_mount_from_center_offset}" />
-		<xacro:property name="d435_cam_depth_py" value="0.0175" />
-		<xacro:property name="d435_cam_depth_pz" value="${d435_cam_height/2}" />
-		<material name="${name}_aluminum">
-			<color rgba="0.5 0.5 0.5 1" />
-		</material>
-		<!-- camera body, with origin at bottom screw mount -->
-		<joint name="${name}_joint" type="fixed">
-			<xacro:insert_block name="origin" />
-			<parent link="${parent}" />
-			<child link="${name}_bottom_screw_frame" />
-		</joint>
-		<link name="${name}_bottom_screw_frame" />
-		<joint name="${name}_link_joint" type="fixed">
-			<origin xyz="0.1 ${d435_cam_depth_py} ${d435_cam_depth_pz}" rpy="0 0 0" />
-			<parent link="${name}_bottom_screw_frame" />
-			<child link="${name}_link" />
-		</joint>
-		<link name="${name}_link">
-			<visual>
-				<origin xyz="${d435_cam_mount_from_center_offset} ${-d435_cam_depth_py} 0" rpy="${M_PI/2} 0 ${M_PI/2}" />
-				<geometry>
-					<!-- <box size="${d435_cam_width} ${d435_cam_height} ${d435_cam_depth}"/> -->
-					<mesh filename="file://$(find wheelchair2_description)/meshes/d435.dae" />
-				</geometry>
-				<material name="${name}_aluminum" />
-			</visual>
-			<collision>
-				<origin xyz="0 ${-d435_cam_depth_py} 0" rpy="0 0 0" />
-				<geometry>
-					<box size="${d435_cam_depth} ${d435_cam_width} ${d435_cam_height}" />
-				</geometry>
-			</collision>
-			<inertial>
-				<!-- The following are not reliable values, and should not be used for modeling -->
-				<mass value="0.564" />
-				<origin xyz="0 0 0" />
-				<inertia ixx="0.003881243" ixy="0.0" ixz="0.0" iyy="0.000498940" iyz="0.0" izz="0.003879257" />
-			</inertial>
-		</link>
-		<!-- camera depth joints and links -->
-		<joint name="${name}_depth_joint" type="fixed">
-			<origin xyz="0 0 0" rpy="0 0 0" />
-			<parent link="${name}_link" />
-			<child link="${name}_depth_frame" />
-		</joint>
-		<link name="${name}_depth_frame" />
-		<joint name="${name}_depth_optical_joint" type="fixed">
-			<origin xyz="0 0 0" rpy="${-M_PI/2} 0 ${-M_PI/2}" />
-			<parent link="${name}_depth_frame" />
-			<child link="${name}_depth_optical_frame" />
-		</joint>
-		<link name="${name}_depth_optical_frame" />
-		<!-- camera left IR joints and links -->
-		<joint name="${name}_left_ir_joint" type="fixed">
-			<origin xyz="0 ${d435_cam_depth_to_left_ir_offset} 0" rpy="0 0 0" />
-			<parent link="${name}_depth_frame" />
-			<child link="${name}_left_ir_frame" />
-		</joint>
-		<link name="${name}_left_ir_frame" />
-		<joint name="${name}_left_ir_optical_joint" type="fixed">
-			<origin xyz="0 0 0" rpy="${-M_PI/2} 0 ${-M_PI/2}" />
-			<parent link="${name}_left_ir_frame" />
-			<child link="${name}_left_ir_optical_frame" />
-		</joint>
-		<link name="${name}_left_ir_optical_frame" />
-		<!-- camera right IR joints and links -->
-		<joint name="${name}_right_ir_joint" type="fixed">
-			<origin xyz="0 ${d435_cam_depth_to_right_ir_offset} 0" rpy="0 0 0" />
-			<parent link="${name}_depth_frame" />
-			<child link="${name}_right_ir_frame" />
-		</joint>
-		<link name="${name}_right_ir_frame" />
-		<joint name="${name}_right_ir_optical_joint" type="fixed">
-			<origin xyz="0 0 0" rpy="${-M_PI/2} 0 ${-M_PI/2}" />
-			<parent link="${name}_right_ir_frame" />
-			<child link="${name}_right_ir_optical_frame" />
-		</joint>
-		<link name="${name}_right_ir_optical_frame" />
-		<!-- camera color joints and links -->
-		<joint name="${name}_color_joint" type="fixed">
-			<origin xyz="0 ${d435_cam_depth_to_color_offset} 0" rpy="0 0 0" />
-			<parent link="${name}_depth_frame" />
-			<child link="${name}_color_frame" />
-		</joint>
-		<link name="${name}_color_frame" />
-		<joint name="${name}_color_optical_joint" type="fixed">
-			<origin xyz="0 0 0" rpy="${-M_PI/2} 0 ${-M_PI/2}" />
-			<parent link="${name}_color_frame" />
-			<child link="${name}_color_optical_frame" />
-		</joint>
-		<link name="${name}_color_optical_frame" />
-		<xacro:if value="${use_sim_time}">
-			<gazebo reference="${name}_link">
-				<material>Gazebo/Black</material>
-				<sensor name="${name}_camera_sensor" type="camera"> <pose> 0 0 0 0 0 0 </pose>
-					<visualize>true</visualize>
-					<update_rate>10</update_rate>
-					<camera>
-						<camera_info_topic>${topics_ns}/color/camera_info</camera_info_topic>
-						<horizontal_fov>1.089</horizontal_fov>
-						<image>
-							<format>R8G8B8</format>
-							<width>640</width>
-							<height>480</height>
-						</image>
-						<clip>
-							<near>0.05</near>
-							<far>8.0</far>
-						</clip>
-					</camera>
-					<plugin name="camera_controller" filename="libgazebo_ros_camera.so">
-						<ros>
-							<namespace>${topics_ns}</namespace>
-							<remapping>image_raw:=color/image_raw</remapping>
-							<remapping>camera_info:=color/camera_info</remapping>
-						</ros>
-						<camera_name>${name}_color</camera_name>
-						<frame_name>${name}_color_optical_frame</frame_name>
-					</plugin>
-				</sensor>
-			</gazebo>
-		</xacro:if>
-	</xacro:macro>
-</robot>
+/home/container_user/wheelchair2/src/build/wheelchair2_description/urdf/realsense.urdf.xacro
