Commit message: working now

File: wheelchair2_description/urdf/wheelchairs/blacky.urdf.xacro (robot description, xacro)
@@ -62,5 +62,5 @@
         <parent link="base_footprint"/>
         <child link="livox_mount_link"/>
-        <origin xyz="0.0 0 1.24" rpy="0 0 0" />
+        <origin xyz="0.0 0 0.8" rpy="0 0 0" />
     </joint>
     <link name="livox_frame"/>

File: wheelchair2_gazebo/urdf/livox.urdf.xacro (robot description, xacro)
@@ -1,19 +1,35 @@
 <?xml version="1.0"?>
-<robot name="wheelchair2"
-    xmlns:xacro="http://www.ros.org/wiki/xacro">
+<robot name="wheelchair2" xmlns:xacro="http://www.ros.org/wiki/xacro">
     <gazebo reference="livox_frame">
         <material>Gazebo/Black</material>
-        <sensor name="Livox" type="custom">
-            <plugin filename="RGLServerPluginInstance" name="rgl::RGLServerPluginInstance">
+        <sensor name="laser" type="gpu_lidar">
+            <pose>0 0 0 0 0 0</pose>
+            <topic>scan</topic>
+            <update_rate>10</update_rate>
+            <lidar>
+                <scan>
+                    <horizontal>
+                        <samples>640</samples>
+                        <resolution>1</resolution>
+                        <min_angle>-3.14159</min_angle>
+                        <max_angle>3.14159</max_angle>
+                    </horizontal>
+                    <vertical>
+                        <samples>1</samples>
+                        <resolution>1</resolution>
+                        <min_angle>0</min_angle>
+                        <max_angle>0</max_angle>
+                    </vertical>
+                </scan>
                 <range>
-                    <min>0</min>
-                    <max>10</max>
+                    <min>0.1</min>
+                    <max>10.0</max>
+                    <resolution>0.01</resolution>
                 </range>
-                <update_rate>10</update_rate>
-                <update_on_paused_sim>false</update_on_paused_sim>
-                <topic>rgl_lidar</topic>
-                <frame>livox_frame</frame>
-                <pattern_preset>Livox Mid360</pattern_preset>
-            </plugin>
+                <frame_id>livox_frame</frame_id>
+            </lidar>
+            <always_on>1</always_on>
+            <visualize>true</visualize>
+            <gz_frame_id>livox_frame</gz_frame_id>
         </sensor>
     </gazebo>
